Commit message: [fix] fix allegro hand collision mesh and reduce the number of visual mesh by removing duplicates

File: robots/allegro_hand/allegro_hand_right.urdf (robot description, URDF)
Before this commit: robot allegro_right, 23 links, 22 joints
Links:
- link base_link: geometry collision box size=0.0414 0.0538 0.0428; collision box size=0.0414 0.0720 0.013
- link link_11.0_tip: geometry collision mesh filename=meshes/collision/link_tip.obj; visual mesh filename=meshes/visual/link_tip.obj
- link link_15.0_tip: geometry collision mesh filename=meshes/collision/link_tip.obj; visual mesh filename=meshes/visual/link_tip.obj
- link link_3.0_tip: geometry collision mesh filename=meshes/collision/link_tip.obj; visual mesh filename=meshes/visual/link_tip.obj
- link link_7.0_tip: geometry collision mesh filename=meshes/collision/link_tip.obj; visual mesh filename=meshes/visual/link_tip.obj
