Commit message: [init] add shadow hand

File: robots/allegro_hand/allegro_hand_left.urdf (robot description, URDF)
Before this commit: robot allegro_left, 23 links, 22 joints
Links:
- link wrist: mass 0.01 -> None

Commit message: [update] update left and right allegro model with both version

File: robots/allegro_hand/allegro_hand_left.urdf (robot description, URDF)
Before this commit: robot allegro_left, 23 links, 22 joints
Links:
- link base_link: geometry collision box size=0.0414 0.0538 0.0428; collision box size=0.0414 0.0720 0.013
- link link_11.0: geometry collision box size=0.0196 0.0269 0.022; visual mesh filename=meshes/visual/link_3.0.obj
- link link_11.0_tip: geometry collision mesh filename=meshes/collision/link_tip.obj; visual mesh filename=meshes/visual/link_tip.obj
- link link_15.0: geometry collision box size=0.0196 0.0269 0.04; visual mesh filename=meshes/visual/link_15.0.obj
- link link_15.0_tip: geometry collision mesh filename=meshes/collision/link_tip.obj; visual mesh filename=meshes/visual/link_tip.obj
- link link_3.0: geometry collision box size=0.0196 0.0269 0.022; visual mesh filename=meshes/visual/link_3.0.obj
- link link_3.0_tip: geometry collision mesh filename=meshes/collision/link_tip.obj; visual mesh filename=meshes/visual/link_tip.obj
- link link_7.0: geometry collision box size=0.0196 0.0269 0.022; visual mesh filename=meshes/visual/link_3.0.obj
- link link_7.0_tip: geometry collision mesh filename=meshes/collision/link_tip.obj; visual mesh filename=meshes/visual/link_tip.obj

File: robots/allegro_hand/allegro_hand_left_glb.urdf (robot description, URDF)
Before this commit: robot allegro_right, 23 links, 22 joints
Links:
- link base_link: geometry collision box size=0.0414 0.0538 0.0428; collision box size=0.0414 0.0720 0.013
- link link_0.0: geometry collision box size=0.0196 0.0275 0.0164; visual mesh filename=meshes/visual/link_0.0.glb
- link link_1.0: geometry collision box size=0.0196 0.0275 0.054; visual mesh filename=meshes/visual/link_1.0.glb
- link link_10.0: geometry collision box size=0.0196 0.0275 0.0384; visual mesh filename=meshes/visual/link_2.0.glb
- link link_11.0: geometry collision box size=0.0196 0.0269 0.022; visual mesh filename=meshes/visual/link_3.0.glb
- link link_11.0_tip: geometry collision mesh filename=meshes/collision/link_tip.obj; visual mesh filename=meshes/visual/link_tip.glb
- link link_12.0: geometry collision box size=0.0358 0.034 0.0455; visual mesh filename=meshes/visual/link_12.0_left.glb
- link link_13.0: geometry collision box size=0.0196 0.0275 0.0177; visual mesh filename=meshes/visual/link_13.0.glb
- link link_14.0: geometry collision box size=0.0196 0.0275 0.0514; visual mesh filename=meshes/visual/link_14.0.glb
- link link_15.0: geometry collision box size=0.0196 0.0269 0.04; visual mesh filename=meshes/visual/link_15.0.glb
- link link_15.0_tip: geometry collision mesh filename=meshes/collision/link_tip.obj; visual mesh filename=meshes/visual/link_tip.glb
- link link_2.0: geometry collision box size=0.0196 0.0275 0.0384; visual mesh filename=meshes/visual/link_2.0.glb
- link link_3.0: geometry collision box size=0.0196 0.0269 0.022; visual mesh filename=meshes/visual/link_3.0.glb
- link link_3.0_tip: geometry collision mesh filename=meshes/collision/link_tip.obj; visual mesh filename=meshes/visual/link_tip.glb
- link link_4.0: geometry collision box size=0.0196 0.0275 0.0164; visual mesh filename=meshes/visual/link_0.0.glb
- link link_5.0: geometry collision box size=0.0196 0.0275 0.054; visual mesh filename=meshes/visual/link_1.0.glb
- link link_6.0: geometry collision box size=0.0196 0.0275 0.0384; visual mesh filename=meshes/visual/link_2.0.glb
- link link_7.0: geometry collision box size=0.0196 0.0269 0.022; visual mesh filename=meshes/visual/link_3.0.glb
- link link_7.0_tip: geometry collision mesh filename=meshes/collision/link_tip.obj; visual mesh filename=meshes/visual/link_tip.glb
- link link_8.0: geometry collision box size=0.0196 0.0275 0.0164; visual mesh filename=meshes/visual/link_0.0.glb
- link link_9.0: geometry collision box size=0.0196 0.0275 0.054; visual mesh filename=meshes/visual/link_1.0.glb
Joints:
- joint joint_12.0: axis -1 0 0 -> 1 0 0; origin xyz=-0.0182 0.019333 -0.045987 rpy=0 -1.65806278845 -1.5707963259 -> xyz=-0.0182 -0.019333 -0.045987 rpy=0 -1.65806278845 1.5707963259
- joint joint_13.0: axis 0 0 1 -> 0 0 -1

File: robots/allegro_hand/allegro_hand_right_glb.urdf (robot description, URDF)
Before this commit: robot allegro_right, 23 links, 22 joints
Links:
- link wrist: mass 0.01 -> None

Commit message: [fix] fix allegro velocity limit issue and update isaacgym checking code

File: robots/allegro_hand/allegro_hand_left.urdf (robot description, URDF)
Before this commit: robot allegro_left, 23 links, 22 joints
Joints:
- joint joint_0.0: limit lower=-0.47 upper=0.47 effort=10 velocity=0 -> lower=-0.47 upper=0.47 effort=10 velocity=3.14
- joint joint_1.0: limit lower=-0.196 upper=1.61 effort=10 velocity=0 -> lower=-0.196 upper=1.61 effort=10 velocity=3.14
- joint joint_10.0: limit lower=-0.174 upper=1.709 effort=10 velocity=0 -> lower=-0.174 upper=1.709 effort=10 velocity=3.14
- joint joint_11.0: limit lower=-0.227 upper=1.618 effort=10 velocity=0 -> lower=-0.227 upper=1.618 effort=10 velocity=3.14
- joint joint_12.0: limit lower=0.263 upper=1.396 effort=10 velocity=0 -> lower=0.263 upper=1.396 effort=10 velocity=3.14
- joint joint_13.0: limit lower=-0.105 upper=1.163 effort=10 velocity=0 -> lower=-0.105 upper=1.163 effort=10 velocity=3.14
- joint joint_14.0: limit lower=-0.189 upper=1.644 effort=10 velocity=0 -> lower=-0.189 upper=1.644 effort=10 velocity=3.14
- joint joint_15.0: limit lower=-0.162 upper=1.719 effort=10 velocity=0 -> lower=-0.162 upper=1.719 effort=10 velocity=3.14
- joint joint_2.0: limit lower=-0.174 upper=1.709 effort=10 velocity=0 -> lower=-0.174 upper=1.709 effort=10 velocity=3.14
- joint joint_3.0: limit lower=-0.227 upper=1.618 effort=10 velocity=0 -> lower=-0.227 upper=1.618 effort=10 velocity=3.14
- joint joint_4.0: limit lower=-0.47 upper=0.47 effort=10 velocity=0 -> lower=-0.47 upper=0.47 effort=10 velocity=3.14
- joint joint_5.0: limit lower=-0.196 upper=1.61 effort=10 velocity=0 -> lower=-0.196 upper=1.61 effort=10 velocity=3.14
- joint joint_6.0: limit lower=-0.174 upper=1.709 effort=10 velocity=0 -> lower=-0.174 upper=1.709 effort=10 velocity=3.14
- joint joint_7.0: limit lower=-0.227 upper=1.618 effort=10 velocity=0 -> lower=-0.227 upper=1.618 effort=10 velocity=3.14
- joint joint_8.0: limit lower=-0.47 upper=0.47 effort=10 velocity=0 -> lower=-0.47 upper=0.47 effort=10 velocity=3.14
- joint joint_9.0: limit lower=-0.196 upper=1.61 effort=10 velocity=0 -> lower=-0.196 upper=1.61 effort=10 velocity=3.14

File: robots/allegro_hand/allegro_hand_left_glb.urdf (robot description, URDF)
Before this commit: robot allegro_left, 23 links, 22 joints
Joints:
- joint joint_0.0: limit lower=-0.47 upper=0.47 effort=10 velocity=0 -> lower=-0.47 upper=0.47 effort=10 velocity=3.14
- joint joint_1.0: limit lower=-0.196 upper=1.61 effort=10 velocity=0 -> lower=-0.196 upper=1.61 effort=10 velocity=3.14
- joint joint_10.0: limit lower=-0.174 upper=1.709 effort=10 velocity=0 -> lower=-0.174 upper=1.709 effort=10 velocity=3.14
- joint joint_11.0: limit lower=-0.227 upper=1.618 effort=10 velocity=0 -> lower=-0.227 upper=1.618 effort=10 velocity=3.14
- joint joint_12.0: limit lower=0.263 upper=1.396 effort=10 velocity=0 -> lower=0.263 upper=1.396 effort=10 velocity=3.14
- joint joint_13.0: limit lower=-0.105 upper=1.163 effort=10 velocity=0 -> lower=-0.105 upper=1.163 effort=10 velocity=3.14
- joint joint_14.0: limit lower=-0.189 upper=1.644 effort=10 velocity=0 -> lower=-0.189 upper=1.644 effort=10 velocity=3.14
- joint joint_15.0: limit lower=-0.162 upper=1.719 effort=10 velocity=0 -> lower=-0.162 upper=1.719 effort=10 velocity=3.14
- joint joint_2.0: limit lower=-0.174 upper=1.709 effort=10 velocity=0 -> lower=-0.174 upper=1.709 effort=10 velocity=3.14
- joint joint_3.0: limit lower=-0.227 upper=1.618 effort=10 velocity=0 -> lower=-0.227 upper=1.618 effort=10 velocity=3.14
- joint joint_4.0: limit lower=-0.47 upper=0.47 effort=10 velocity=0 -> lower=-0.47 upper=0.47 effort=10 velocity=3.14
- joint joint_5.0: limit lower=-0.196 upper=1.61 effort=10 velocity=0 -> lower=-0.196 upper=1.61 effort=10 velocity=3.14
- joint joint_6.0: limit lower=-0.174 upper=1.709 effort=10 velocity=0 -> lower=-0.174 upper=1.709 effort=10 velocity=3.14
- joint joint_7.0: limit lower=-0.227 upper=1.618 effort=10 velocity=0 -> lower=-0.227 upper=1.618 effort=10 velocity=3.14
- joint joint_8.0: limit lower=-0.47 upper=0.47 effort=10 velocity=0 -> lower=-0.47 upper=0.47 effort=10 velocity=3.14
- joint joint_9.0: limit lower=-0.196 upper=1.61 effort=10 velocity=0 -> lower=-0.196 upper=1.61 effort=10 velocity=3.14

File: robots/allegro_hand/allegro_hand_right.urdf (robot description, URDF)
Before this commit: robot allegro_right, 23 links, 22 joints
Joints:
- joint joint_0.0: limit lower=-0.47 upper=0.47 effort=10 velocity=0 -> lower=-0.47 upper=0.47 effort=10 velocity=3.14
- joint joint_1.0: limit lower=-0.196 upper=1.61 effort=10 velocity=0 -> lower=-0.196 upper=1.61 effort=10 velocity=3.14
- joint joint_10.0: limit lower=-0.174 upper=1.709 effort=10 velocity=0 -> lower=-0.174 upper=1.709 effort=10 velocity=3.14
- joint joint_11.0: limit lower=-0.227 upper=1.618 effort=10 velocity=0 -> lower=-0.227 upper=1.618 effort=10 velocity=3.14
- joint joint_12.0: limit lower=0.263 upper=1.396 effort=10 velocity=0 -> lower=0.263 upper=1.396 effort=10 velocity=3.14
- joint joint_13.0: limit lower=-0.105 upper=1.163 effort=10 velocity=0 -> lower=-0.105 upper=1.163 effort=10 velocity=3.14
- joint joint_14.0: limit lower=-0.189 upper=1.644 effort=10 velocity=0 -> lower=-0.189 upper=1.644 effort=10 velocity=3.14
- joint joint_15.0: limit lower=-0.162 upper=1.719 effort=10 velocity=0 -> lower=-0.162 upper=1.719 effort=10 velocity=3.14
- joint joint_2.0: limit lower=-0.174 upper=1.709 effort=10 velocity=0 -> lower=-0.174 upper=1.709 effort=10 velocity=3.14
- joint joint_3.0: limit lower=-0.227 upper=1.618 effort=10 velocity=0 -> lower=-0.227 upper=1.618 effort=10 velocity=3.14
- joint joint_4.0: limit lower=-0.47 upper=0.47 effort=10 velocity=0 -> lower=-0.47 upper=0.47 effort=10 velocity=3.14
- joint joint_5.0: limit lower=-0.196 upper=1.61 effort=10 velocity=0 -> lower=-0.196 upper=1.61 effort=10 velocity=3.14
- joint joint_6.0: limit lower=-0.174 upper=1.709 effort=10 velocity=0 -> lower=-0.174 upper=1.709 effort=10 velocity=3.14
- joint joint_7.0: limit lower=-0.227 upper=1.618 effort=10 velocity=0 -> lower=-0.227 upper=1.618 effort=10 velocity=3.14
- joint joint_8.0: limit lower=-0.47 upper=0.47 effort=10 velocity=0 -> lower=-0.47 upper=0.47 effort=10 velocity=3.14
- joint joint_9.0: limit lower=-0.196 upper=1.61 effort=10 velocity=0 -> lower=-0.196 upper=1.61 effort=10 velocity=3.14

File: robots/allegro_hand/allegro_hand_right_glb.urdf (robot description, URDF)
Before this commit: robot allegro_right, 23 links, 22 joints
Joints:
- joint joint_0.0: limit lower=-0.47 upper=0.47 effort=10 velocity=0 -> lower=-0.47 upper=0.47 effort=10 velocity=3.14
- joint joint_1.0: limit lower=-0.196 upper=1.61 effort=10 velocity=0 -> lower=-0.196 upper=1.61 effort=10 velocity=3.14
- joint joint_10.0: limit lower=-0.174 upper=1.709 effort=10 velocity=0 -> lower=-0.174 upper=1.709 effort=10 velocity=3.14
- joint joint_11.0: limit lower=-0.227 upper=1.618 effort=10 velocity=0 -> lower=-0.227 upper=1.618 effort=10 velocity=3.14
- joint joint_12.0: limit lower=0.263 upper=1.396 effort=10 velocity=0 -> lower=0.263 upper=1.396 effort=10 velocity=3.14
- joint joint_13.0: limit lower=-0.105 upper=1.163 effort=10 velocity=0 -> lower=-0.105 upper=1.163 effort=10 velocity=3.14
- joint joint_14.0: limit lower=-0.189 upper=1.644 effort=10 velocity=0 -> lower=-0.189 upper=1.644 effort=10 velocity=3.14
- joint joint_15.0: limit lower=-0.162 upper=1.719 effort=10 velocity=0 -> lower=-0.162 upper=1.719 effort=10 velocity=3.14
- joint joint_2.0: limit lower=-0.174 upper=1.709 effort=10 velocity=0 -> lower=-0.174 upper=1.709 effort=10 velocity=3.14
- joint joint_3.0: limit lower=-0.227 upper=1.618 effort=10 velocity=0 -> lower=-0.227 upper=1.618 effort=10 velocity=3.14
- joint joint_4.0: limit lower=-0.47 upper=0.47 effort=10 velocity=0 -> lower=-0.47 upper=0.47 effort=10 velocity=3.14
- joint joint_5.0: limit lower=-0.196 upper=1.61 effort=10 velocity=0 -> lower=-0.196 upper=1.61 effort=10 velocity=3.14
- joint joint_6.0: limit lower=-0.174 upper=1.709 effort=10 velocity=0 -> lower=-0.174 upper=1.709 effort=10 velocity=3.14
- joint joint_7.0: limit lower=-0.227 upper=1.618 effort=10 velocity=0 -> lower=-0.227 upper=1.618 effort=10 velocity=3.14
- joint joint_8.0: limit lower=-0.47 upper=0.47 effort=10 velocity=0 -> lower=-0.47 upper=0.47 effort=10 velocity=3.14
- joint joint_9.0: limit lower=-0.196 upper=1.61 effort=10 velocity=0 -> lower=-0.196 upper=1.61 effort=10 velocity=3.14

Commit message: [fix] fix allegro internal

File: robots/allegro_hand/allegro_hand_left.urdf (robot description, URDF)
Before this commit: robot allegro_left, 23 links, 22 joints
Links:
- link link_0.0: mass 0.005 -> 0.0119
- link link_1.0: mass 0.125164 -> 0.065
- link link_10.0: mass 0.131691 -> 0.0355
- link link_11.0: mass 0.0388 -> 0.0096
- link link_11.0_tip: mass None -> 0.0168
- link link_12.0: mass 0.005 -> 0.0176
- link link_13.0: mass 0.125164 -> 0.0119
- link link_14.0: mass 0.131691 -> 0.038
- link link_15.0_tip: mass None -> 0.0168
- link link_2.0: mass 0.131691 -> 0.0355
- link link_3.0: mass 0.0388 -> 0.0096
- link link_3.0_tip: mass None -> 0.0168
- link link_5.0: mass 0.125164 -> 0.065
- link link_6.0: mass 0.131691 -> 0.0355
- link link_7.0_tip: mass None -> 0.0096
- link link_9.0: mass 0.125164 -> 0.065

File: robots/allegro_hand/allegro_hand_left_glb.urdf (robot description, URDF)
Before this commit: robot allegro_left, 23 links, 22 joints
Links:
- link link_0.0: mass 0.005 -> 0.0119
- link link_1.0: mass 0.125164 -> 0.065
- link link_10.0: mass 0.131691 -> 0.0355
- link link_11.0: mass 0.0388 -> 0.0096
- link link_11.0_tip: mass None -> 0.0168
- link link_12.0: mass 0.005 -> 0.0176
- link link_13.0: mass 0.125164 -> 0.0119
- link link_14.0: mass 0.131691 -> 0.038
- link link_15.0_tip: mass None -> 0.0168
- link link_2.0: mass 0.131691 -> 0.0355
- link link_3.0: mass 0.0388 -> 0.0096
- link link_3.0_tip: mass None -> 0.0168
- link link_5.0: mass 0.125164 -> 0.065
- link link_6.0: mass 0.131691 -> 0.0355
- link link_7.0_tip: mass None -> 0.0096
- link link_9.0: mass 0.125164 -> 0.065

File: robots/allegro_hand/allegro_hand_right.urdf (robot description, URDF)
Before this commit: robot allegro_right, 23 links, 22 joints
Links:
- link link_0.0: mass 0.005 -> 0.0119
- link link_1.0: mass 0.125164 -> 0.065
- link link_10.0: mass 0.131691 -> 0.0355
- link link_11.0: mass 0.0388 -> 0.0096
- link link_11.0_tip: mass None -> 0.0168
- link link_12.0: mass 0.005 -> 0.0176
- link link_13.0: mass 0.125164 -> 0.0119
- link link_14.0: mass 0.131691 -> 0.038
- link link_15.0_tip: mass None -> 0.0168
- link link_2.0: mass 0.131691 -> 0.0355
- link link_3.0: mass 0.0388 -> 0.0096
- link link_3.0_tip: mass None -> 0.0168
- link link_5.0: mass 0.125164 -> 0.065
- link link_6.0: mass 0.131691 -> 0.0355
- link link_7.0_tip: mass None -> 0.0096
- link link_9.0: mass 0.125164 -> 0.065

File: robots/allegro_hand/allegro_hand_right_glb.urdf (robot description, URDF)
Before this commit: robot allegro_right, 23 links, 22 joints
Links:
- link link_0.0: mass 0.005 -> 0.0119
- link link_1.0: mass 0.125164 -> 0.065
- link link_10.0: mass 0.131691 -> 0.0355
- link link_11.0: mass 0.0388 -> 0.0096
- link link_11.0_tip: mass None -> 0.0168
- link link_12.0: mass 0.005 -> 0.0176
- link link_13.0: mass 0.125164 -> 0.0119
- link link_14.0: mass 0.131691 -> 0.038
- link link_15.0_tip: mass None -> 0.0168
- link link_2.0: mass 0.131691 -> 0.0355
- link link_3.0: mass 0.0388 -> 0.0096
- link link_3.0_tip: mass None -> 0.0168
- link link_5.0: mass 0.125164 -> 0.065
- link link_6.0: mass 0.131691 -> 0.0355
- link link_7.0_tip: mass None -> 0.0096
- link link_9.0: mass 0.125164 -> 0.065
