Commit message: [fix] fix sapien rendering and dclaw inertia

File: robots/dclaw_gripper/dclaw.urdf (robot description, URDF)
Before this commit: robot DClaw, 10 links, 9 joints
Links:
- link Link1_1: mass 0.0500997884947533 -> None
- link Link1_2: mass 0.0500997884944988 -> None
- link Link1_3: mass 0 -> None
- link Link2_1: mass 0.0500997884947319 -> None
- link Link2_2: mass 0.050099788494456 -> None
- link Link2_3: mass 0.0500997884940055 -> None
- link Link3_1: mass 0.0260028886170262 -> None
- link Link3_2: mass 0.0260028959491832 -> None
- link Link3_3: mass 0.0260028939266903 -> None

File: robots/dclaw_gripper/dclaw_glb.urdf (robot description, URDF)
Before this commit: robot DClaw, 10 links, 9 joints
Links:
- link Link1_1: mass 0.0500997884947533 -> None
- link Link1_2: mass 0.0500997884944988 -> None
- link Link1_3: mass 0 -> None
- link Link2_1: mass 0.0500997884947319 -> None
- link Link2_2: mass 0.050099788494456 -> None
- link Link2_3: mass 0.0500997884940055 -> None
- link Link3_1: mass 0.0260028886170262 -> None
- link Link3_2: mass 0.0260028959491832 -> None
- link Link3_3: mass 0.0260028939266903 -> None
