Commit message: [update] major update for readme and hand models

File: robots/dclaw_gripper/dclaw_gripper.urdf (robot description, URDF)
Before this commit: robot dclaw_gripper, 10 links, 9 joints
Links:
- added link base
Joints:
- added joint base_joint: type fixed, parent base, child base_link, origin xyz=0 0 0 rpy=0 -1.57079 0

File: robots/dclaw_gripper/dclaw_gripper_glb.urdf (robot description, URDF)
Before this commit: robot dclaw_gripper, 10 links, 9 joints
Links:
- added link base
Joints:
- added joint base_joint: type fixed, parent base, child base_link, origin xyz=0 0 0 rpy=0 -1.57079 0
