Commit message: [update] update shadow hand model for better wrist link definition

File: robots/shadow_hand/shadow_hand_right.urdf (robot description, URDF)
Before this commit: robot bimanual_shadowhand_motor, 33 links, 32 joints
Links:
- removed link manipulator
- added link ee_link
Joints:
- joint ee_fixed_joint: child manipulator -> ee_link; origin xyz=0.0 0.0 0.05 rpy=0.0 0.0 0.0 -> xyz=0.0 0.0 0.0 rpy=0.0 0.0 -1.57079

Commit message: [update] update shadow hand model

File: robots/shadow_hand/shadow_hand_right.urdf (robot description, URDF)
Before this commit: robot bimanual_shadowhand_motor, 33 links, 32 joints
Links:
- link ffdistal: mass 0.012 -> 0.12; geometry collision mesh filename=meshes/visual/f_distal_pst.obj scale=0.001 0.001 0.001; visual mesh filename=meshes/visual/f_distal_pst.obj scale=0.001 0.001 0.001
- link ffknuckle: geometry collision mesh filename=meshes/collision/f_knuckle_E3M5.obj; visual mesh filename=meshes/visual/f_knuckle_E3M5.obj scale=0.001 0.001 0.001
- link ffmiddle: geometry collision cylinder length=0.025 radius=0.007; collision sphere radius=0.007
- link ffproximal: geometry collision cylinder length=0.040 radius=0.007; visual mesh filename=meshes/visual/f_proximal_E3M5.obj scale=0.001 0.001 0.001
- link forearm: geometry collision box size=0.07 0.07 0.07; collision mesh filename=meshes/collision/forearm_E3M5.obj scale=0.001 0.001 0.001
- link lfdistal: mass 0.012 -> 0.12; geometry collision mesh filename=meshes/visual/f_distal_pst.obj scale=0.001 0.001 0.001; visual mesh filename=meshes/visual/f_distal_pst.obj scale=0.001 0.001 0.001
- link lfknuckle: geometry collision mesh filename=meshes/collision/f_knuckle_E3M5.obj; visual mesh filename=meshes/visual/f_knuckle_E3M5.obj scale=0.001 0.001 0.001
- link lfmetacarpal: geometry collision box size=0.018 0.024 0.040; visual mesh filename=meshes/visual/lf_metacarpal_E3M5.obj scale=0.001 0.001 0.001
- link lfmiddle: geometry collision cylinder length=0.025 radius=0.007; collision sphere radius=0.007
- link lfproximal: geometry collision cylinder length=0.040 radius=0.007; visual mesh filename=meshes/visual/f_proximal_E3M5.obj scale=0.001 0.001 0.001
- link mfdistal: mass 0.012 -> 0.12; geometry collision mesh filename=meshes/visual/f_distal_pst.obj scale=0.001 0.001 0.001; visual mesh filename=meshes/visual/f_distal_pst.obj scale=0.001 0.001 0.001
- link mfknuckle: geometry collision mesh filename=meshes/collision/f_knuckle_E3M5.obj; visual mesh filename=meshes/visual/f_knuckle_E3M5.obj scale=0.001 0.001 0.001
- link mfmiddle: geometry collision cylinder length=0.025 radius=0.007; collision sphere radius=0.007
- link mfproximal: geometry collision cylinder length=0.040 radius=0.007; visual mesh filename=meshes/visual/f_proximal_E3M5.obj scale=0.001 0.001 0.001
- link palm: geometry collision box size=0.018 0.024 0.004; collision box size=0.020 0.024 0.032
- link rfdistal: mass 0.012 -> 0.12; geometry collision mesh filename=meshes/visual/f_distal_pst.obj scale=0.001 0.001 0.001; visual mesh filename=meshes/visual/f_distal_pst.obj scale=0.001 0.001 0.001
- link rfknuckle: geometry collision mesh filename=meshes/collision/f_knuckle_E3M5.obj; visual mesh filename=meshes/visual/f_knuckle_E3M5.obj scale=0.001 0.001 0.001
- link rfmiddle: geometry collision cylinder length=0.025 radius=0.007; collision sphere radius=0.007
- link rfproximal: geometry collision cylinder length=0.040 radius=0.007; visual mesh filename=meshes/visual/f_proximal_E3M5.obj scale=0.001 0.001 0.001
- link thdistal: mass 0.016 -> 0.16; geometry collision mesh filename=meshes/visual/th_distal_pst.obj scale=0.001 0.001 0.001; visual mesh filename=meshes/visual/th_distal_pst.obj scale=0.001 0.001 0.001
- link thhub: geometry collision sphere radius=0.010
- link thmiddle: geometry collision mesh filename=meshes/collision/th_middle_E3M5.obj scale=0.001 0.001 0.001; visual mesh filename=meshes/visual/th_middle_E3M5.obj scale=0.001 0.001 0.001
- link thproximal: geometry collision mesh filename=meshes/collision/th_proximal_E3M5.obj scale=0.001 0.001 0.001; visual mesh filename=meshes/visual/th_proximal_E3M5.obj scale=0.001 0.001 0.001
- link wrist: geometry collision box size=0.027 0.018 0.010; collision box size=0.027 0.018 0.010
