Commit message: [update] fix shadow urdf and update left hand

File: robots/shadow_hand/shadow_hand_left.urdf (robot description, URDF)
Before this commit: robot shadow_right, 33 links, 32 joints
Links:
- removed link ee_link
- removed link ffdistal
- removed link ffknuckle
- removed link ffmiddle
- removed link ffproximal
- removed link fftip
- removed link imu
- removed link lfdistal
- removed link lfknuckle
- removed link lfmetacarpal
- removed link lfmiddle
- removed link lfproximal
- removed link lftip
- removed link mfdistal
- removed link mfknuckle
- removed link mfmiddle
- removed link mfproximal
- removed link mftip
- removed link palm
- removed link rfdistal
- removed link rfknuckle
- removed link rfmiddle
- removed link rfproximal
- removed link rftip
- removed link thbase
- removed link thdistal
- removed link thhub
- removed link thmiddle
- removed link thproximal
- removed link thtip
- added link lh_ffdistal, mass 0.012; collision mesh filename=meshes/visual/f_distal/pst/f_distal_pst.dae scale=0.001 0.001 0.001; visual mesh filename=meshes/visual/f_distal/pst/f_distal_pst.dae scale=0.001 0.001 0.001
- added link lh_ffknuckle, mass 0.008; collision cylinder length=0.014 radius=0.007; visual mesh filename=meshes/visual/f_knuckle/f_knuckle_E3M5.dae scale=0.001 0.001 0.001
- added link lh_ffmiddle, mass 0.017; collision cylinder length=0.025 radius=0.007; collision sphere radius=0.007
- added link lh_ffproximal, mass 0.030; collision cylinder length=0.040 radius=0.007; visual mesh filename=meshes/visual/f_proximal/f_proximal_E3M5.dae scale=0.001 0.001 0.001
- added link lh_fftip, mass 0.001
- added link lh_imu
- added link lh_lfdistal, mass 0.012; collision mesh filename=meshes/visual/f_distal/pst/f_distal_pst.dae scale=0.001 0.001 0.001; visual mesh filename=meshes/visual/f_distal/pst/f_distal_pst.dae scale=0.001 0.001 0.001
- added link lh_lfknuckle, mass 0.008; collision cylinder length=0.014 radius=0.007; visual mesh filename=meshes/visual/f_knuckle/f_knuckle_E3M5.dae scale=0.001 0.001 0.001
- added link lh_lfmetacarpal, mass 0.030; collision box size=0.018 0.024 0.040; visual mesh filename=meshes/visual/lf_metacarpal/lf_metacarpal_E3M5.dae scale=-0.001 0.001 0.001
- added link lh_lfmiddle, mass 0.017; collision cylinder length=0.025 radius=0.007; collision sphere radius=0.007
- added link lh_lfproximal, mass 0.030; collision cylinder length=0.040 radius=0.007; visual mesh filename=meshes/visual/f_proximal/f_proximal_E3M5.dae scale=0.001 0.001 0.001
- added link lh_lftip, mass 0.001
- added link lh_manipulator
- added link lh_mfdistal, mass 0.012; collision mesh filename=meshes/visual/f_distal/pst/f_distal_pst.dae scale=0.001 0.001 0.001; visual mesh filename=meshes/visual/f_distal/pst/f_distal_pst.dae scale=0.001 0.001 0.001
- added link lh_mfknuckle, mass 0.008; collision cylinder length=0.014 radius=0.007; visual mesh filename=meshes/visual/f_knuckle/f_knuckle_E3M5.dae scale=0.001 0.001 0.001
- added link lh_mfmiddle, mass 0.017; collision cylinder length=0.025 radius=0.007; collision sphere radius=0.007
- added link lh_mfproximal, mass 0.030; collision cylinder length=0.040 radius=0.007; visual mesh filename=meshes/visual/f_proximal/f_proximal_E3M5.dae scale=0.001 0.001 0.001
- added link lh_mftip, mass 0.001
- added link lh_palm, mass 0.3; collision box size=0.018 0.024 0.004; collision box size=0.020 0.024 0.040
- added link lh_rfdistal, mass 0.012; collision mesh filename=meshes/visual/f_distal/pst/f_distal_pst.dae scale=0.001 0.001 0.001; visual mesh filename=meshes/visual/f_distal/pst/f_distal_pst.dae scale=0.001 0.001 0.001
- added link lh_rfknuckle, mass 0.008; collision cylinder length=0.014 radius=0.007; visual mesh filename=meshes/visual/f_knuckle/f_knuckle_E3M5.dae scale=0.001 0.001 0.001
- added link lh_rfmiddle, mass 0.017; collision cylinder length=0.025 radius=0.007; collision sphere radius=0.007
- added link lh_rfproximal, mass 0.030; collision cylinder length=0.040 radius=0.007; visual mesh filename=meshes/visual/f_proximal/f_proximal_E3M5.dae scale=0.001 0.001 0.001
- added link lh_rftip, mass 0.001
- added link lh_thbase, mass 0.010; collision sphere radius=0.011; visual box size=0.001 0.001 0.001
- added link lh_thdistal, mass 0.016; collision mesh filename=meshes/visual/th_distal/pst/th_distal_pst.dae scale=0.001 0.001 0.001; visual mesh filename=meshes/visual/th_distal/pst/th_distal_pst.dae scale=0.001 0.001 0.001
- added link lh_thhub, mass 0.005; collision sphere radius=0.010; visual box size=0.001 0.001 0.001
- added link lh_thmiddle, mass 0.020; collision cylinder length=0.014 radius=0.010; collision cylinder length=0.018 radius=0.011
- added link lh_thproximal, mass 0.040; collision cylinder length=0.018 radius=0.012; visual mesh filename=meshes/visual/th_proximal/th_proximal_E3M5.dae scale=0.001 0.001 0.001
- added link lh_thtip, mass 0.001
- link forearm: geometry collision box size=0.07 0.07 0.07; collision mesh filename=meshes/collision/forearm_E3M5.obj scale=0.001 0.001 0.001
- link wrist: geometry collision box size=0.027 0.018 0.010; collision box size=0.027 0.018 0.010
Joints:
- removed joint FFJ1
- removed joint FFJ2
- removed joint FFJ3
- removed joint FFJ4
- removed joint FFtip
- removed joint LFJ1
- removed joint LFJ2
- removed joint LFJ3
- removed joint LFJ4
- removed joint LFJ5
- removed joint LFtip
- removed joint MFJ1
- removed joint MFJ2
- removed joint MFJ3
- removed joint MFJ4
- removed joint MFtip
- removed joint RFJ1
- removed joint RFJ2
- removed joint RFJ3
- removed joint RFJ4
- removed joint RFtip
- removed joint THJ1
- removed joint THJ2
- removed joint THJ3
- removed joint THJ4
- removed joint THJ5
- removed joint WRJ1
- removed joint WRJ2
- removed joint ee_fixed_joint
- removed joint palm_to_imu
- removed joint thtip
- added joint lh_FFJ1: type revolute, parent lh_ffmiddle, child lh_ffdistal, origin xyz=0 0 0.025 rpy=0 0 0, axis 1 0 0, limit lower=0 upper=1.57079632679 effort=2 velocity=2.0
- added joint lh_FFJ2: type revolute, parent lh_ffproximal, child lh_ffmiddle, origin xyz=0 0 0.045 rpy=0 0 0, axis 1 0 0, limit lower=0 upper=1.57079632679 effort=2 velocity=2.0
- added joint lh_FFJ3: type revolute, parent lh_ffknuckle, child lh_ffproximal, origin xyz=0 0 0 rpy=0 0 0, axis 1 0 0, limit lower=-0.261799387799 upper=1.57079632679 effort=2 velocity=2.0
- added joint lh_FFJ4: type revolute, parent lh_palm, child lh_ffknuckle, origin xyz=-0.033 0 0.095 rpy=0 0 0, axis 0 1 0, limit lower=-0.349065850399 upper=0.349065850399 effort=2 velocity=2.0
- added joint lh_FFtip: type fixed, parent lh_ffdistal, child lh_fftip, origin xyz=0 0 0.026 rpy=0 0 0
- added joint lh_LFJ1: type revolute, parent lh_lfmiddle, child lh_lfdistal, origin xyz=0 0 0.025 rpy=0 0 0, axis 1 0 0, limit lower=0 upper=1.57079632679 effort=2 velocity=2.0
- added joint lh_LFJ2: type revolute, parent lh_lfproximal, child lh_lfmiddle, origin xyz=0 0 0.045 rpy=0 0 0, axis 1 0 0, limit lower=0 upper=1.57079632679 effort=2 velocity=2.0
- added joint lh_LFJ3: type revolute, parent lh_lfknuckle, child lh_lfproximal, origin xyz=0 0 0 rpy=0 0 0, axis 1 0 0, limit lower=-0.261799387799 upper=1.57079632679 effort=2 velocity=2.0
- added joint lh_LFJ4: type revolute, parent lh_lfmetacarpal, child lh_lfknuckle, origin xyz=-0.05397275 0 0.03779463 rpy=0 -0.9599 0, axis 0 -1 0, limit lower=-0.349065850399 upper=0.349065850399 effort=2 velocity=2.0
- added joint lh_LFJ5: type revolute, parent lh_palm, child lh_lfmetacarpal, origin xyz=0.033 0 0.02071 rpy=0 0.9599 0, axis 1 0 0, limit lower=0 upper=0.785398163397 effort=2 velocity=2.0
- added joint lh_LFtip: type fixed, parent lh_lfdistal, child lh_lftip, origin xyz=0 0 0.026 rpy=0 0 0
- added joint lh_MFJ1: type revolute, parent lh_mfmiddle, child lh_mfdistal, origin xyz=0 0 0.025 rpy=0 0 0, axis 1 0 0, limit lower=0 upper=1.57079632679 effort=2 velocity=2.0
- added joint lh_MFJ2: type revolute, parent lh_mfproximal, child lh_mfmiddle, origin xyz=0 0 0.045 rpy=0 0 0, axis 1 0 0, limit lower=0 upper=1.57079632679 effort=2 velocity=2.0
- added joint lh_MFJ3: type revolute, parent lh_mfknuckle, child lh_mfproximal, origin xyz=0 0 0 rpy=0 0 0, axis 1 0 0, limit lower=-0.261799387799 upper=1.57079632679 effort=2 velocity=2.0
- added joint lh_MFJ4: type revolute, parent lh_palm, child lh_mfknuckle, origin xyz=-0.011 0 0.099 rpy=0 0 0, axis 0 1 0, limit lower=-0.349065850399 upper=0.349065850399 effort=2 velocity=2.0
- added joint lh_MFtip: type fixed, parent lh_mfdistal, child lh_mftip, origin xyz=0 0 0.026 rpy=0 0 0
- added joint lh_RFJ1: type revolute, parent lh_rfmiddle, child lh_rfdistal, origin xyz=0 0 0.025 rpy=0 0 0, axis 1 0 0, limit lower=0 upper=1.57079632679 effort=2 velocity=2.0
- added joint lh_RFJ2: type revolute, parent lh_rfproximal, child lh_rfmiddle, origin xyz=0 0 0.045 rpy=0 0 0, axis 1 0 0, limit lower=0 upper=1.57079632679 effort=2 velocity=2.0
- added joint lh_RFJ3: type revolute, parent lh_rfknuckle, child lh_rfproximal, origin xyz=0 0 0 rpy=0 0 0, axis 1 0 0, limit lower=-0.261799387799 upper=1.57079632679 effort=2 velocity=2.0
- added joint lh_RFJ4: type revolute, parent lh_palm, child lh_rfknuckle, origin xyz=0.011 0 0.095 rpy=0 0 0, axis 0 -1 0, limit lower=-0.349065850399 upper=0.349065850399 effort=2 velocity=2.0
- added joint lh_RFtip: type fixed, parent lh_rfdistal, child lh_rftip, origin xyz=0 0 0.026 rpy=0 0 0
- added joint lh_THJ1: type revolute, parent lh_thmiddle, child lh_thdistal, origin xyz=0 0 0.032 rpy=0 0 0, axis 1 0 0, limit lower=-0.261799387799 upper=1.57079632679 effort=1.0 velocity=4.0
- added joint lh_THJ2: type revolute, parent lh_thhub, child lh_thmiddle, origin xyz=0 0 0 rpy=0 0 0, axis 1 0 0, limit lower=-0.698131700798 upper=0.698131700798 effort=2.0 velocity=2.0
- added joint lh_THJ3: type revolute, parent lh_thproximal, child lh_thhub, origin xyz=0 0 0.038 rpy=0 0 0, axis 0 -1 0, limit lower=-0.209439510239 upper=0.209439510239 effort=2.0 velocity=4.0
- added joint lh_THJ4: type revolute, parent lh_thbase, child lh_thproximal, origin xyz=0 0 0 rpy=0 0 0, axis 0 -1 0, limit lower=0.0 upper=1.2217304764 effort=3 velocity=4.0
- added joint lh_THJ5: type revolute, parent lh_palm, child lh_thbase, origin xyz=-0.034 -0.00858 0.029 rpy=-0.785398163397 0 1.57079632679, axis 0 0 1, limit lower=-1.0471975512 upper=1.0471975512 effort=5.0 velocity=4.0
- added joint lh_WRJ1: type revolute, parent lh_wrist, child lh_palm, origin xyz=0 0 0.034 rpy=0 0 0, axis 1 0 0, limit lower=-0.698131700798 upper=0.488692190558 effort=30 velocity=2.0
- added joint lh_WRJ2: type revolute, parent lh_forearm, child lh_wrist, origin xyz=0 -0.010 0.21301 rpy=0 0 0, axis 0 -1 0, limit lower=-0.523598775598 upper=0.174532925199 effort=10 velocity=2.0
- added joint lh_ee_fixed_joint: type fixed, parent lh_palm, child lh_manipulator, origin xyz=0.0 0.0 0.05 rpy=0.0 0.0 0.0
- added joint lh_palm_to_imu: type fixed, parent lh_palm, child lh_imu, origin xyz=0.01785 0.00765 0.049125 rpy=-1.5707963 3.141592 0.0
- added joint lh_thtip: type fixed, parent lh_thdistal, child lh_thtip, origin xyz=0 0 0.0275 rpy=0 0 0
- added joint right_hand_to_left_hand: type fixed, parent rh_forearm, child lh_forearm, origin xyz=-0.4 0.0 0.0 rpy=0.0 0.0 0.0

File: robots/shadow_hand/shadow_hand_left_new.urdf (robot description, URDF)
Before this commit: robot shadow_right, 33 links, 32 joints
Links:
- link ffdistal: geometry collision mesh filename=meshes/visual/f_distal_pst.obj scale=0.001 0.001 0.001; visual mesh filename=meshes/visual/f_distal_pst.obj scale=0.001 0.001 0.001
- link ffknuckle: geometry collision mesh filename=meshes/collision/f_knuckle_E3M5.obj; visual mesh filename=meshes/visual/f_knuckle_E3M5.obj scale=0.001 0.001 0.001
- link ffmiddle: geometry collision cylinder length=0.025 radius=0.007; collision sphere radius=0.007
- link ffproximal: geometry collision cylinder length=0.040 radius=0.007; visual mesh filename=meshes/visual/f_proximal_E3M5.obj scale=0.001 0.001 0.001
- link forearm: geometry collision box size=0.07 0.07 0.07; collision mesh filename=meshes/collision/forearm_E3M5.obj scale=0.001 0.001 0.001
- link lfdistal: geometry collision mesh filename=meshes/visual/f_distal_pst.obj scale=0.001 0.001 0.001; visual mesh filename=meshes/visual/f_distal_pst.obj scale=0.001 0.001 0.001
- link lfknuckle: geometry collision mesh filename=meshes/collision/f_knuckle_E3M5.obj; visual mesh filename=meshes/visual/f_knuckle_E3M5.obj scale=0.001 0.001 0.001
- link lfmetacarpal: geometry collision box size=0.018 0.024 0.040; visual mesh filename=meshes/visual/lf_metacarpal_E3M5.obj scale=-0.001 0.001 0.001
- link lfmiddle: geometry collision cylinder length=0.025 radius=0.007; collision sphere radius=0.007
- link lfproximal: geometry collision cylinder length=0.040 radius=0.007; visual mesh filename=meshes/visual/f_proximal_E3M5.obj scale=0.001 0.001 0.001
- link mfdistal: geometry collision mesh filename=meshes/visual/f_distal_pst.obj scale=0.001 0.001 0.001; visual mesh filename=meshes/visual/f_distal_pst.obj scale=0.001 0.001 0.001
- link mfknuckle: geometry collision mesh filename=meshes/collision/f_knuckle_E3M5.obj; visual mesh filename=meshes/visual/f_knuckle_E3M5.obj scale=0.001 0.001 0.001
- link mfmiddle: geometry collision cylinder length=0.025 radius=0.007; collision sphere radius=0.007
- link mfproximal: geometry collision cylinder length=0.040 radius=0.007; visual mesh filename=meshes/visual/f_proximal_E3M5.obj scale=0.001 0.001 0.001
- link palm: geometry collision box size=0.018 0.024 0.004; collision box size=0.020 0.024 0.032
- link rfdistal: geometry collision mesh filename=meshes/visual/f_distal_pst.obj scale=0.001 0.001 0.001; visual mesh filename=meshes/visual/f_distal_pst.obj scale=0.001 0.001 0.001
- link rfknuckle: geometry collision mesh filename=meshes/collision/f_knuckle_E3M5.obj; visual mesh filename=meshes/visual/f_knuckle_E3M5.obj scale=0.001 0.001 0.001
- link rfmiddle: geometry collision cylinder length=0.025 radius=0.007; collision sphere radius=0.007
- link rfproximal: geometry collision cylinder length=0.040 radius=0.007; visual mesh filename=meshes/visual/f_proximal_E3M5.obj scale=0.001 0.001 0.001
- link thdistal: geometry collision mesh filename=meshes/visual/th_distal_pst.obj scale=0.001 0.001 0.001; visual mesh filename=meshes/visual/th_distal_pst.obj scale=0.001 0.001 0.001
- link thmiddle: geometry collision mesh filename=meshes/collision/th_middle_E3M5.obj scale=0.001 0.001 0.001; visual mesh filename=meshes/visual/th_middle_E3M5.obj scale=0.001 0.001 0.001
- link thproximal: geometry collision mesh filename=meshes/collision/th_proximal_E3M5.obj scale=0.001 0.001 0.001; visual mesh filename=meshes/visual/th_proximal_E3M5.obj scale=0.001 0.001 0.001
- link wrist: geometry collision box size=0.027 0.018 0.010; collision box size=0.027 0.018 0.010
Joints:
- joint FFJ4: axis 0 -1 0 -> 0 1 0; origin xyz=0.033 0 0.095 rpy=0 0 0 -> xyz=-0.033 0 0.095 rpy=0 0 0
- joint LFJ4: axis 0 1 0 -> 0 -1 0; origin xyz=0.05397275 0 0.03779463 rpy=0 0.9599 0 -> xyz=-0.05397275 0 0.03779463 rpy=0 -0.9599 0
- joint LFJ5: origin xyz=-0.033 0 0.02071 rpy=0 -0.9599 0 -> xyz=0.033 0 0.02071 rpy=0 0.9599 0
- joint MFJ4: axis 0 -1 0 -> 0 1 0; origin xyz=0.011 0 0.099 rpy=0 0 0 -> xyz=-0.011 0 0.099 rpy=0 0 0
- joint RFJ4: axis 0 1 0 -> 0 -1 0; origin xyz=-0.011 0 0.095 rpy=0 0 0 -> xyz=0.011 0 0.095 rpy=0 0 0
- joint THJ3: axis 0 1 0 -> 0 -1 0
- joint THJ4: axis 0 1 0 -> 0 -1 0
- joint THJ5: axis 0 0 -1 -> 0 0 1; origin xyz=0.034 -0.00858 0.029 rpy=-0.785398163397 0 -1.57079632679 -> xyz=-0.034 -0.00858 0.029 rpy=-0.785398163397 0 1.57079632679
- joint WRJ2: axis 0 1 0 -> 0 -1 0
- joint ee_fixed_joint: origin xyz=0.0 0.0 0.0 rpy=0.0 0.0 -1.57079 -> xyz=0.0 0.0 0.00 rpy=0.0 0.0 0.0
