Commit message: [refactor] fix visual problem of shadow_hand_left and upload .glb version

File: robots/shadow_hand/shadow_hand_left.urdf (robot description, URDF)
Before this commit: robot shadow_left, 33 links, 33 joints
Links:
- removed link lh_ffdistal
- removed link lh_ffknuckle
- removed link lh_ffmiddle
- removed link lh_ffproximal
- removed link lh_fftip
- removed link lh_imu
- removed link lh_lfdistal
- removed link lh_lfknuckle
- removed link lh_lfmetacarpal
- removed link lh_lfmiddle
- removed link lh_lfproximal
- removed link lh_lftip
- removed link lh_manipulator
- removed link lh_mfdistal
- removed link lh_mfknuckle
- removed link lh_mfmiddle
- removed link lh_mfproximal
- removed link lh_mftip
- removed link lh_palm
- removed link lh_rfdistal
- removed link lh_rfknuckle
- removed link lh_rfmiddle
- removed link lh_rfproximal
- removed link lh_rftip
- removed link lh_thbase
- removed link lh_thdistal
- removed link lh_thhub
- removed link lh_thmiddle
- removed link lh_thproximal
- removed link lh_thtip
- added link ee_link
- added link ffdistal, mass 0.12; collision mesh filename=meshes/visual/f_distal_pst.obj scale=0.001 0.001 0.001; visual mesh filename=meshes/visual/f_distal_pst.obj scale=0.001 0.001 0.001
- added link ffknuckle, mass 0.008; collision mesh filename=meshes/collision/f_knuckle_E3M5.obj; visual mesh filename=meshes/visual/f_knuckle_E3M5.obj scale=0.001 0.001 0.001
- added link ffmiddle, mass 0.017; collision cylinder length=0.025 radius=0.007; collision sphere radius=0.007
- added link ffproximal, mass 0.030; collision cylinder length=0.040 radius=0.007; visual mesh filename=meshes/visual/f_proximal_E3M5.obj scale=0.001 0.001 0.001
- added link fftip, mass 0.001
- added link imu
- added link lfdistal, mass 0.12; collision mesh filename=meshes/visual/f_distal_pst.obj scale=0.001 0.001 0.001; visual mesh filename=meshes/visual/f_distal_pst.obj scale=0.001 0.001 0.001
- added link lfknuckle, mass 0.008; collision mesh filename=meshes/collision/f_knuckle_E3M5.obj; visual mesh filename=meshes/visual/f_knuckle_E3M5.obj scale=0.001 0.001 0.001
- added link lfmetacarpal, mass 0.030; collision box size=0.018 0.024 0.040; visual mesh filename=meshes/visual/lf_metacarpal_E3M5_left.obj scale=0.001 0.001 0.001
- added link lfmiddle, mass 0.017; collision cylinder length=0.025 radius=0.007; collision sphere radius=0.007
- added link lfproximal, mass 0.030; collision cylinder length=0.040 radius=0.007; visual mesh filename=meshes/visual/f_proximal_E3M5.obj scale=0.001 0.001 0.001
- added link lftip, mass 0.001
- added link mfdistal, mass 0.12; collision mesh filename=meshes/visual/f_distal_pst.obj scale=0.001 0.001 0.001; visual mesh filename=meshes/visual/f_distal_pst.obj scale=0.001 0.001 0.001
- added link mfknuckle, mass 0.008; collision mesh filename=meshes/collision/f_knuckle_E3M5.obj; visual mesh filename=meshes/visual/f_knuckle_E3M5.obj scale=0.001 0.001 0.001
- added link mfmiddle, mass 0.017; collision cylinder length=0.025 radius=0.007; collision sphere radius=0.007
- added link mfproximal, mass 0.030; collision cylinder length=0.040 radius=0.007; visual mesh filename=meshes/visual/f_proximal_E3M5.obj scale=0.001 0.001 0.001
- added link mftip, mass 0.001
- added link palm, mass 0.3; collision box size=0.018 0.024 0.004; collision box size=0.020 0.024 0.032
- added link rfdistal, mass 0.12; collision mesh filename=meshes/visual/f_distal_pst.obj scale=0.001 0.001 0.001; visual mesh filename=meshes/visual/f_distal_pst.obj scale=0.001 0.001 0.001
- added link rfknuckle, mass 0.008; collision mesh filename=meshes/collision/f_knuckle_E3M5.obj; visual mesh filename=meshes/visual/f_knuckle_E3M5.obj scale=0.001 0.001 0.001
- added link rfmiddle, mass 0.017; collision cylinder length=0.025 radius=0.007; collision sphere radius=0.007
- added link rfproximal, mass 0.030; collision cylinder length=0.040 radius=0.007; visual mesh filename=meshes/visual/f_proximal_E3M5.obj scale=0.001 0.001 0.001
- added link rftip, mass 0.001
- added link thbase, mass 0.010; collision sphere radius=0.011; visual box size=0.001 0.001 0.001
- added link thdistal, mass 0.16; collision mesh filename=meshes/visual/th_distal_pst.obj scale=0.001 0.001 0.001; visual mesh filename=meshes/visual/th_distal_pst.obj scale=0.001 0.001 0.001
- added link thhub, mass 0.005; collision sphere radius=0.010
- added link thmiddle, mass 0.020; collision mesh filename=meshes/collision/th_middle_E3M5.obj scale=0.001 0.001 0.001; visual mesh filename=meshes/visual/th_middle_E3M5.obj scale=0.001 0.001 0.001
- added link thproximal, mass 0.040; collision mesh filename=meshes/collision/th_proximal_E3M5.obj scale=0.001 0.001 0.001; visual mesh filename=meshes/visual/th_proximal_E3M5.obj scale=0.001 0.001 0.001
- added link thtip, mass 0.001
Joints:
- removed joint lh_FFJ1
- removed joint lh_FFJ2
- removed joint lh_FFJ3
- removed joint lh_FFJ4
- removed joint lh_FFtip
- removed joint lh_LFJ1
- removed joint lh_LFJ2
- removed joint lh_LFJ3
- removed joint lh_LFJ4
- removed joint lh_LFJ5
- removed joint lh_LFtip
- removed joint lh_MFJ1
- removed joint lh_MFJ2
- removed joint lh_MFJ3
- removed joint lh_MFJ4
- removed joint lh_MFtip
- removed joint lh_RFJ1
- removed joint lh_RFJ2
- removed joint lh_RFJ3
- removed joint lh_RFJ4
- removed joint lh_RFtip
- removed joint lh_THJ1
- removed joint lh_THJ2
- removed joint lh_THJ3
- removed joint lh_THJ4
- removed joint lh_THJ5
- removed joint lh_WRJ1
- removed joint lh_WRJ2
- removed joint lh_ee_fixed_joint
- removed joint lh_palm_to_imu
- removed joint lh_thtip
- removed joint right_hand_to_left_hand
- added joint FFJ1: type revolute, parent ffmiddle, child ffdistal, origin xyz=0 0 0.025 rpy=0 0 0, axis 1 0 0, limit lower=0 upper=1.57079632679 effort=2 velocity=2.0
- added joint FFJ2: type revolute, parent ffproximal, child ffmiddle, origin xyz=0 0 0.045 rpy=0 0 0, axis 1 0 0, limit lower=0 upper=1.57079632679 effort=2 velocity=2.0
- added joint FFJ3: type revolute, parent ffknuckle, child ffproximal, origin xyz=0 0 0 rpy=0 0 0, axis 1 0 0, limit lower=-0.261799387799 upper=1.57079632679 effort=2 velocity=2.0
- added joint FFJ4: type revolute, parent palm, child ffknuckle, origin xyz=-0.033 0 0.095 rpy=0 0 0, axis 0 1 0, limit lower=-0.349065850399 upper=0.349065850399 effort=2 velocity=2.0
- added joint FFtip: type fixed, parent ffdistal, child fftip, origin xyz=0 0 0.026 rpy=0 0 0
- added joint LFJ1: type revolute, parent lfmiddle, child lfdistal, origin xyz=0 0 0.025 rpy=0 0 0, axis 1 0 0, limit lower=0 upper=1.57079632679 effort=2 velocity=2.0
- added joint LFJ2: type revolute, parent lfproximal, child lfmiddle, origin xyz=0 0 0.045 rpy=0 0 0, axis 1 0 0, limit lower=0 upper=1.57079632679 effort=2 velocity=2.0
- added joint LFJ3: type revolute, parent lfknuckle, child lfproximal, origin xyz=0 0 0 rpy=0 0 0, axis 1 0 0, limit lower=-0.261799387799 upper=1.57079632679 effort=2 velocity=2.0
- added joint LFJ4: type revolute, parent lfmetacarpal, child lfknuckle, origin xyz=-0.05397275 0 0.03779463 rpy=0 -0.9599 0, axis 0 -1 0, limit lower=-0.349065850399 upper=0.349065850399 effort=2 velocity=2.0
- added joint LFJ5: type revolute, parent palm, child lfmetacarpal, origin xyz=0.033 0 0.02071 rpy=0 0.9599 0, axis 1 0 0, limit lower=0 upper=0.785398163397 effort=2 velocity=2.0
- added joint LFtip: type fixed, parent lfdistal, child lftip, origin xyz=0 0 0.026 rpy=0 0 0
- added joint MFJ1: type revolute, parent mfmiddle, child mfdistal, origin xyz=0 0 0.025 rpy=0 0 0, axis 1 0 0, limit lower=0 upper=1.57079632679 effort=2 velocity=2.0
- added joint MFJ2: type revolute, parent mfproximal, child mfmiddle, origin xyz=0 0 0.045 rpy=0 0 0, axis 1 0 0, limit lower=0 upper=1.57079632679 effort=2 velocity=2.0
- added joint MFJ3: type revolute, parent mfknuckle, child mfproximal, origin xyz=0 0 0 rpy=0 0 0, axis 1 0 0, limit lower=-0.261799387799 upper=1.57079632679 effort=2 velocity=2.0
- added joint MFJ4: type revolute, parent palm, child mfknuckle, origin xyz=-0.011 0 0.099 rpy=0 0 0, axis 0 1 0, limit lower=-0.349065850399 upper=0.349065850399 effort=2 velocity=2.0
- added joint MFtip: type fixed, parent mfdistal, child mftip, origin xyz=0 0 0.026 rpy=0 0 0
- added joint RFJ1: type revolute, parent rfmiddle, child rfdistal, origin xyz=0 0 0.025 rpy=0 0 0, axis 1 0 0, limit lower=0 upper=1.57079632679 effort=2 velocity=2.0
- added joint RFJ2: type revolute, parent rfproximal, child rfmiddle, origin xyz=0 0 0.045 rpy=0 0 0, axis 1 0 0, limit lower=0 upper=1.57079632679 effort=2 velocity=2.0
- added joint RFJ3: type revolute, parent rfknuckle, child rfproximal, origin xyz=0 0 0 rpy=0 0 0, axis 1 0 0, limit lower=-0.261799387799 upper=1.57079632679 effort=2 velocity=2.0
- added joint RFJ4: type revolute, parent palm, child rfknuckle, origin xyz=0.011 0 0.095 rpy=0 0 0, axis 0 -1 0, limit lower=-0.349065850399 upper=0.349065850399 effort=2 velocity=2.0
- added joint RFtip: type fixed, parent rfdistal, child rftip, origin xyz=0 0 0.026 rpy=0 0 0
- added joint THJ1: type revolute, parent thmiddle, child thdistal, origin xyz=0 0 0.032 rpy=0 0 0, axis 1 0 0, limit lower=-0.261799387799 upper=1.57079632679 effort=1.0 velocity=4.0
- added joint THJ2: type revolute, parent thhub, child thmiddle, origin xyz=0 0 0 rpy=0 0 0, axis 1 0 0, limit lower=-0.698131700798 upper=0.698131700798 effort=2.0 velocity=2.0
- added joint THJ3: type revolute, parent thproximal, child thhub, origin xyz=0 0 0.038 rpy=0 0 0, axis 0 -1 0, limit lower=-0.209439510239 upper=0.209439510239 effort=2.0 velocity=4.0
- added joint THJ4: type revolute, parent thbase, child thproximal, origin xyz=0 0 0 rpy=0 0 0, axis 0 -1 0, limit lower=0.0 upper=1.2217304764 effort=3 velocity=4.0
- added joint THJ5: type revolute, parent palm, child thbase, origin xyz=-0.034 -0.00858 0.029 rpy=-0.785398163397 0 1.57079632679, axis 0 0 1, limit lower=-1.0471975512 upper=1.0471975512 effort=5.0 velocity=4.0
- added joint WRJ1: type revolute, parent wrist, child palm, origin xyz=0 0 0.034 rpy=0 0 0, axis 1 0 0, limit lower=-0.698131700798 upper=0.488692190558 effort=30 velocity=2.0
- added joint WRJ2: type revolute, parent forearm, child wrist, origin xyz=0 -0.010 0.21301 rpy=0 0 0, axis 0 -1 0, limit lower=-0.523598775598 upper=0.174532925199 effort=10 velocity=2.0
- added joint ee_fixed_joint: type fixed, parent palm, child ee_link, origin xyz=0.0 0.0 0.00 rpy=0.0 0.0 0.0
- added joint palm_to_imu: type fixed, parent palm, child imu, origin xyz=0.01785 0.00765 0.049125 rpy=-1.5707963 3.141592 0.0
- added joint thtip: type fixed, parent thdistal, child thtip, origin xyz=0 0 0.0275 rpy=0 0 0

File: robots/shadow_hand/shadow_hand_left_glb.urdf (robot description, URDF)
Before this commit: robot shadow_left, 33 links, 32 joints
Links:
- link ffdistal: geometry collision mesh filename=meshes/visual/f_distal_pst.glb scale=0.001 0.001 0.001; visual mesh filename=meshes/visual/f_distal_pst.glb scale=0.001 0.001 0.001
- link ffknuckle: geometry collision mesh filename=meshes/collision/f_knuckle_E3M5.obj; visual mesh filename=meshes/visual/f_knuckle_E3M5.glb scale=0.001 0.001 0.001
- link ffproximal: geometry collision cylinder length=0.040 radius=0.007; visual mesh filename=meshes/visual/f_proximal_E3M5.glb scale=0.001 0.001 0.001
- link forearm: geometry collision box size=0.07 0.07 0.07; collision mesh filename=meshes/collision/forearm_E3M5.obj scale=0.001 0.001 0.001
- link lfdistal: geometry collision mesh filename=meshes/visual/f_distal_pst.glb scale=0.001 0.001 0.001; visual mesh filename=meshes/visual/f_distal_pst.glb scale=0.001 0.001 0.001
- link lfknuckle: geometry collision mesh filename=meshes/collision/f_knuckle_E3M5.obj; visual mesh filename=meshes/visual/f_knuckle_E3M5.glb scale=0.001 0.001 0.001
- link lfmetacarpal: geometry collision box size=0.018 0.024 0.040; visual mesh filename=meshes/visual/lf_metacarpal_E3M5_left.glb scale=0.001 0.001 0.001
- link lfmiddle: geometry collision cylinder length=0.025 radius=0.007; collision sphere radius=0.007
- link lfproximal: geometry collision cylinder length=0.040 radius=0.007; visual mesh filename=meshes/visual/f_proximal_E3M5.glb scale=0.001 0.001 0.001
- link mfdistal: geometry collision mesh filename=meshes/visual/f_distal_pst.glb scale=0.001 0.001 0.001; visual mesh filename=meshes/visual/f_distal_pst.glb scale=0.001 0.001 0.001
- link mfknuckle: geometry collision mesh filename=meshes/collision/f_knuckle_E3M5.obj; visual mesh filename=meshes/visual/f_knuckle_E3M5.glb scale=0.001 0.001 0.001
- link mfmiddle: geometry collision cylinder length=0.025 radius=0.007; collision sphere radius=0.007
- link mfproximal: geometry collision cylinder length=0.040 radius=0.007; visual mesh filename=meshes/visual/f_proximal_E3M5.glb scale=0.001 0.001 0.001
- link palm: geometry collision box size=0.018 0.024 0.004; collision box size=0.020 0.024 0.032
- link rfdistal: geometry collision mesh filename=meshes/visual/f_distal_pst.glb scale=0.001 0.001 0.001; visual mesh filename=meshes/visual/f_distal_pst.glb scale=0.001 0.001 0.001
- link rfknuckle: geometry collision mesh filename=meshes/collision/f_knuckle_E3M5.obj; visual mesh filename=meshes/visual/f_knuckle_E3M5.glb scale=0.001 0.001 0.001
- link rfmiddle: geometry collision cylinder length=0.025 radius=0.007; collision sphere radius=0.007
- link rfproximal: geometry collision cylinder length=0.040 radius=0.007; visual mesh filename=meshes/visual/f_proximal_E3M5.glb scale=0.001 0.001 0.001
- link thdistal: geometry collision mesh filename=meshes/visual/th_distal_pst.glb scale=0.001 0.001 0.001; visual mesh filename=meshes/visual/th_distal_pst.glb scale=0.001 0.001 0.001
- link thmiddle: geometry collision mesh filename=meshes/collision/th_middle_E3M5.obj scale=0.001 0.001 0.001; visual mesh filename=meshes/visual/th_middle_E3M5.glb scale=0.001 0.001 0.001
- link thproximal: geometry collision mesh filename=meshes/collision/th_proximal_E3M5.obj scale=0.001 0.001 0.001; visual mesh filename=meshes/visual/th_proximal_E3M5.glb scale=0.001 0.001 0.001
- link wrist: geometry collision box size=0.027 0.018 0.010; collision box size=0.027 0.018 0.010

Commit message: [fix] fix shadow hand collision mesh

File: robots/shadow_hand/shadow_hand_left.urdf (robot description, URDF)
Before this commit: robot shadow_left, 33 links, 32 joints
Links:
- link ffdistal: geometry collision mesh filename=meshes/collision/f_distal_pst.obj scale=0.001 0.001 0.001; visual mesh filename=meshes/visual/f_distal_pst.obj scale=0.001 0.001 0.001
- link mfdistal: geometry collision mesh filename=meshes/collision/f_distal_pst.obj scale=0.001 0.001 0.001; visual mesh filename=meshes/visual/f_distal_pst.obj scale=0.001 0.001 0.001
- link rfdistal: geometry collision mesh filename=meshes/collision/f_distal_pst.obj scale=0.001 0.001 0.001; visual mesh filename=meshes/visual/f_distal_pst.obj scale=0.001 0.001 0.001

File: robots/shadow_hand/shadow_hand_left_glb.urdf (robot description, URDF)
Before this commit: robot shadow_left, 33 links, 32 joints
Links:
- link ffdistal: geometry collision mesh filename=meshes/collision/f_distal_pst.obj scale=0.001 0.001 0.001; visual mesh filename=meshes/visual/f_distal_pst.glb scale=0.001 0.001 0.001
- link lfdistal: geometry collision mesh filename=meshes/visual/f_distal_pst.obj scale=0.001 0.001 0.001; visual mesh filename=meshes/visual/f_distal_pst.glb scale=0.001 0.001 0.001
- link mfdistal: geometry collision mesh filename=meshes/collision/f_distal_pst.obj scale=0.001 0.001 0.001; visual mesh filename=meshes/visual/f_distal_pst.glb scale=0.001 0.001 0.001
- link rfdistal: geometry collision mesh filename=meshes/collision/f_distal_pst.obj scale=0.001 0.001 0.001; visual mesh filename=meshes/visual/f_distal_pst.glb scale=0.001 0.001 0.001
- link thdistal: geometry collision mesh filename=meshes/visual/th_distal_pst.obj scale=0.001 0.001 0.001; visual mesh filename=meshes/visual/th_distal_pst.glb scale=0.001 0.001 0.001

File: robots/shadow_hand/shadow_hand_right.urdf (robot description, URDF)
Before this commit: robot shadow_right, 33 links, 32 joints
Links:
- link lfdistal: geometry collision mesh filename=meshes/collision/f_distal_pst.obj scale=0.001 0.001 0.001; visual mesh filename=meshes/visual/f_distal_pst.obj scale=0.001 0.001 0.001
- link mfdistal: geometry collision mesh filename=meshes/collision/f_distal_pst.obj scale=0.001 0.001 0.001; visual mesh filename=meshes/visual/f_distal_pst.obj scale=0.001 0.001 0.001
- link rfdistal: geometry collision mesh filename=meshes/collision/f_distal_pst.obj scale=0.001 0.001 0.001; visual mesh filename=meshes/visual/f_distal_pst.obj scale=0.001 0.001 0.001

File: robots/shadow_hand/shadow_hand_right_glb.urdf (robot description, URDF)
Before this commit: robot shadow_right, 33 links, 32 joints
Links:
- link lfdistal: geometry collision mesh filename=meshes/collision/f_distal_pst.obj scale=0.001 0.001 0.001; visual mesh filename=meshes/visual/f_distal_pst.glb scale=0.001 0.001 0.001
- link mfdistal: geometry collision mesh filename=meshes/collision/f_distal_pst.obj scale=0.001 0.001 0.001; visual mesh filename=meshes/visual/f_distal_pst.glb scale=0.001 0.001 0.001
- link rfdistal: geometry collision mesh filename=meshes/collision/f_distal_pst.obj scale=0.001 0.001 0.001; visual mesh filename=meshes/visual/f_distal_pst.glb scale=0.001 0.001 0.001
