Commit message: [refector] rebuild collision meshes and change visual material

File: robots/barrett_hand/bhand_model.urdf (robot description, URDF)
Before this commit: robot bhand_model, 9 links, 8 joints
Links:
- link finger_1_dist_link: geometry collision box size=0.012 0.012 0.02; collision box size=0.014 0.038 0.02
- link finger_1_prox_link: geometry collision box size=0.02 0.026 0.01; collision box size=0.076 0.024 0.026
- link finger_2_dist_link: geometry collision box size=0.012 0.012 0.02; collision box size=0.014 0.038 0.02
- link finger_2_prox_link: geometry collision box size=0.02 0.026 0.01; collision box size=0.076 0.024 0.026
- link finger_3_dist_link: geometry collision box size=0.012 0.012 0.02; collision box size=0.014 0.038 0.02

Commit message: [refector] upload .glb visual meshes, and _glb.urdf

File: robots/barrett_hand/bhand_model.urdf (robot description, URDF)
Before this commit: robot bhand_model, 9 links, 8 joints
Links:
- link base_link: geometry collision box size=0.026 0.02 0.01; collision box size=0.026 0.02 0.01
- link finger_1_dist_link: mass 19342.3312257343 -> 19342.3312257343E-5
- link finger_1_med_liink: mass 31321.1214212939 -> 31321.1214212939E-5
- link finger_1_prox_link: mass 56143.0626955765 -> 56143.0626955765E-5; geometry collision box size=0.02 0.026 0.01; collision box size=0.07 0.024 0.026
- link finger_2_dist_link: mass 19342.3313295693 -> 19342.3313295693E-5
- link finger_2_med_link: mass 31321.1215499126 -> 31321.1215499126E-5
- link finger_2_prox_link: mass 56143.0626955765 -> 56143.0626955765E-5; geometry collision box size=0.02 0.026 0.01; collision box size=0.07 0.024 0.026
- link finger_3_dist_link: mass 19342.3312257343 -> 19342.3312257343E-5
- link finger_3_med_link: mass 31321.121421294 -> 31321.121421294E-5
Joints:
- joint finger_1_dist_joint: limit lower=-0.785 upper=0 effort=0 velocity=0 -> lower=-0.785 upper=0 effort=0 velocity=10
- joint finger_1_med_joint: limit lower=-2.44 upper=0 effort=0 velocity=0 -> lower=-2.44 upper=0 effort=0 velocity=10
- joint finger_1_prox_joint: limit lower=-3.141 upper=0 effort=0 velocity=0 -> lower=-3.14 upper=0 effort=0 velocity=10
- joint finger_2_dist_joint: limit lower=-0.785 upper=0 effort=0 velocity=0 -> lower=-0.785 upper=0 effort=0 velocity=10
- joint finger_2_med_joint: limit lower=-2.44 upper=0 effort=0 velocity=0 -> lower=-2.44 upper=0 effort=0 velocity=10
- joint finger_2_prox_joint: limit lower=0 upper=3.141 effort=0 velocity=0 -> lower=0 upper=3.14 effort=0 velocity=10
- joint finger_3_dist_joint: limit lower=-0.785 upper=0 effort=0 velocity=0 -> lower=-0.785 upper=0 effort=0 velocity=10
- joint finger_3_med_joint: limit lower=-2.44 upper=0 effort=0 velocity=0 -> lower=-2.44 upper=0 effort=0 velocity=10

File: robots/barrett_hand/bhand_model_glb.urdf (robot description, URDF)
Before this commit: robot bhand_model, 9 links, 8 joints
Links:
- link base_link: geometry collision box size=0.026 0.02 0.01; collision box size=0.026 0.02 0.01
- link finger_1_dist_link: geometry collision box size=0.012 0.012 0.02; collision box size=0.014 0.038 0.02
- link finger_1_med_liink: geometry collision box size=0.008 0.022 0.018; collision box size=0.02 0.022 0.01
- link finger_1_prox_link: geometry collision box size=0.02 0.026 0.01; collision box size=0.07 0.024 0.026
- link finger_2_dist_link: geometry collision box size=0.012 0.012 0.02; collision box size=0.014 0.038 0.02
- link finger_2_med_link: geometry collision box size=0.008 0.022 0.018; collision box size=0.02 0.022 0.01
- link finger_2_prox_link: geometry collision box size=0.02 0.026 0.01; collision box size=0.07 0.024 0.026
- link finger_3_dist_link: geometry collision box size=0.012 0.012 0.02; collision box size=0.014 0.038 0.02
- link finger_3_med_link: geometry collision box size=0.008 0.022 0.018; collision box size=0.02 0.022 0.01
Joints:
- joint finger_1_dist_joint: limit lower=-0.785 upper=0 effort=0 velocity=0 -> lower=-0.785 upper=0 effort=0 velocity=10
- joint finger_1_med_joint: limit lower=-2.44 upper=0 effort=0 velocity=0 -> lower=-2.44 upper=0 effort=0 velocity=10
- joint finger_1_prox_joint: limit lower=-3.14 upper=0 effort=0 velocity=0 -> lower=-3.141 upper=0 effort=0 velocity=10
- joint finger_2_dist_joint: limit lower=-0.785 upper=0 effort=0 velocity=0 -> lower=-0.785 upper=0 effort=0 velocity=10
- joint finger_2_med_joint: limit lower=-2.44 upper=0 effort=0 velocity=0 -> lower=-2.44 upper=0 effort=0 velocity=10
- joint finger_2_prox_joint: limit lower=0 upper=3.14 effort=0 velocity=0 -> lower=0 upper=3.141 effort=0 velocity=10
- joint finger_3_dist_joint: limit lower=-0.785 upper=0 effort=0 velocity=0 -> lower=-0.785 upper=0 effort=0 velocity=10
- joint finger_3_med_joint: limit lower=-2.44 upper=0 effort=0 velocity=0 -> lower=-2.44 upper=0 effort=0 velocity=10
