Commit message: [fix] fix ability hand mesh

File: robots/ability_hand/ability_hand_right.urdf (robot description, URDF)
Before this commit: robot ability_hand, 17 links, 16 joints
Links:
- link index_L1: geometry collision box size=0.012 0.012 0.002; collision box size=0.012 0.012 0.002
- link thumb_base: geometry collision mesh filename=meshes/collision/FB_palm_ref_MIR.obj; visual mesh filename=meshes/visual/FB_palm_ref_MIR.obj
