Commit message: [update] clean urdf file for ability hand

File: robots/ability_hand/ability_hand_left.urdf (robot description, URDF)
Before this commit: robot ability_hand, 17 links, 16 joints
Links:
- added link base_link
- link base: geometry collision mesh filename=meshes/collision/wristmesh_C.obj; visual mesh filename=meshes/visual/wristmesh.obj
- link index_L1: geometry collision box size=0.012 0.012 0.002; collision box size=0.012 0.012 0.002
- link thumb_base: geometry collision mesh filename=meshes/collision/FB_palm_ref.obj; visual mesh filename=meshes/visual/FB_palm_ref.obj
Joints:
- added joint base_joint: type fixed, parent base_link, child base, origin xyz=0 0 0 rpy=0 0 -1.57079

File: robots/ability_hand/ability_hand_left_glb.urdf (robot description, URDF)
Before this commit: robot ability_hand, 17 links, 16 joints
Links:
- added link base_link
- link base: geometry collision mesh filename=meshes/collision/wristmesh_C.obj; visual mesh filename=meshes/visual/wristmesh.glb
- link index_L1: geometry collision box size=0.012 0.012 0.002; collision box size=0.012 0.012 0.002
- link thumb_base: geometry collision mesh filename=meshes/collision/FB_palm_ref.obj; visual mesh filename=meshes/visual/FB_palm_ref.glb
Joints:
- added joint base_joint: type fixed, parent base_link, child base, origin xyz=0 0 0 rpy=0 0 -1.57079

File: robots/ability_hand/ability_hand_right.urdf (robot description, URDF)
Before this commit: robot ability_hand, 17 links, 16 joints
Links:
- added link base_link
- link base: geometry collision mesh filename=meshes/collision/wristmesh_C.obj; visual mesh filename=meshes/visual/wristmesh.obj
Joints:
- added joint base_joint: type fixed, parent base_link, child base, origin xyz=0 0 0 rpy=0 0 -1.57079

File: robots/ability_hand/ability_hand_right_glb.urdf (robot description, URDF)
Before this commit: robot ability_hand, 17 links, 16 joints
Links:
- added link base_link
- link base: geometry collision mesh filename=meshes/collision/wristmesh_C.obj; visual mesh filename=meshes/visual/wristmesh.glb
- link index_L1: geometry collision box size=0.012 0.012 0.002; collision box size=0.012 0.012 0.002
- link thumb_base: geometry collision mesh filename=meshes/collision/FB_palm_ref_MIR.obj; visual mesh filename=meshes/visual/FB_palm_ref_MIR.glb
Joints:
- added joint base_joint: type fixed, parent base_link, child base, origin xyz=0 0 0 rpy=0 0 -1.57079
