Commit message: [refactor] revise the mesh of palm_lower and material metallic

File: robots/leap_hand/robot.urdf (robot description, URDF)
Before this commit: robot onshape, 17 links, 16 joints
Links:
- link palm_lower: geometry collision box size=0.004 0.036 0.034; collision box size=0.01 0.12 0.02
