Commit message: [ref] ref urdf format

File: robots/leap_hand/leap_hand_right.urdf (robot description, URDF)
Before this commit: robot onshape, 17 links, 16 joints
Links:
- added link base
Joints:
- added joint base_joint: type fixed, parent base, child palm_lower, origin xyz=0 0.038 0.098 rpy=0 -1.57079 0

File: robots/leap_hand/leap_hand_right_glb.urdf (robot description, URDF)
Before this commit: robot onshape, 17 links, 16 joints
Links:
- added link base
Joints:
- added joint base_joint: type fixed, parent base, child palm_lower, origin xyz=0 0.038 0.098 rpy=0 -1.57079 0
