Commit message: [fix] clean up svh hand directory for the right hand

File: robots/hands/schunk_hand/schunk_svh_hand_right.urdf (robot description, URDF)
Before this commit: robot svh, 31 links, 30 joints
Links:
- removed link right_hand_e
- removed link right_hand_virtual_a
- link right_hand_a: geometry collision mesh filename=meshes/collision/d11.obj scale=1 1 1; visual mesh filename=meshes/visual/d11.obj scale=1 1 1
- link right_hand_b: geometry collision mesh filename=meshes/collision/d12.obj scale=1 1 1; visual mesh filename=meshes/visual/d12.obj scale=1 1 1
- link right_hand_base_link: geometry collision cylinder length=0.045 radius=0.045; visual mesh filename=meshes/visual/base10.obj
- link right_hand_c: geometry collision mesh filename=meshes/collision/d13.obj scale=1 1 1; visual mesh filename=meshes/visual/d13.obj scale=1 1 1
- link right_hand_e2: geometry collision box size=0.012 0.018 0.021; collision box size=0.0246 0.035 0.0564
- link right_hand_i: geometry collision mesh filename=meshes/collision/f41.obj; visual mesh filename=meshes/visual/f41.obj
- link right_hand_j: geometry collision mesh filename=meshes/collision/f31.obj scale=1 1 1; visual mesh filename=meshes/visual/f31.obj
- link right_hand_k: geometry collision mesh filename=meshes/collision/f21.obj scale=1 1 1; visual mesh filename=meshes/visual/f21.obj
- link right_hand_l: geometry collision mesh filename=meshes/collision/f11.obj scale=1 1 1; visual mesh filename=meshes/visual/f11.obj
- link right_hand_m: geometry collision mesh filename=meshes/collision/f42.obj; visual mesh filename=meshes/visual/f42.obj
- link right_hand_n: geometry collision mesh filename=meshes/collision/f22_f32.obj scale=1 1 1; visual mesh filename=meshes/visual/f22_f32.obj
- link right_hand_o: geometry collision mesh filename=meshes/collision/f22_f32.obj scale=1 1 1; visual mesh filename=meshes/visual/f22_f32.obj
- link right_hand_p: geometry collision mesh filename=meshes/collision/f12.obj; visual mesh filename=meshes/visual/f12.obj
- link right_hand_q: geometry collision mesh filename=meshes/collision/finger_tip.obj; visual mesh filename=meshes/visual/finger_tip.obj
- link right_hand_r: geometry collision mesh filename=meshes/collision/finger_tip.obj scale=1 1 1; visual mesh filename=meshes/visual/finger_tip.obj
- link right_hand_s: geometry collision mesh filename=meshes/collision/finger_tip.obj scale=1 1 1; visual mesh filename=meshes/visual/finger_tip.obj
- link right_hand_t: geometry collision mesh filename=meshes/collision/finger_tip.obj scale=1 1 1; visual mesh filename=meshes/visual/finger_tip.obj
- link right_hand_virtual_i: geometry collision sphere radius=0.01; visual mesh filename=meshes/visual/f30_f40.obj
- link right_hand_virtual_j: geometry collision sphere radius=0.01; visual mesh filename=meshes/visual/f30_f40.obj
- link right_hand_virtual_k: geometry collision sphere radius=0.01; visual mesh filename=meshes/visual/f10_f20.obj
- link right_hand_virtual_l: geometry collision sphere radius=0.012; visual mesh filename=meshes/visual/f10_f20.obj
- link right_hand_z: geometry collision box size=0.006 0.024 0.033; collision box size=0.006 0.024 0.033
Joints:
- removed joint right_hand_Thumb_Helper
- removed joint right_hand_f5
- joint right_hand_Finger_Spread: origin xyz=0.025355 0 0.056 rpy=-1.5707 -1.5707 0 -> xyz=0.025355 -0.006 0.056 rpy=-1.5707 -1.5707 0; parent right_hand_e -> right_hand_e2
- joint right_hand_Thumb_Flexion: origin xyz=0 0 0 rpy=0 0 -0.9704 -> xyz=0 0 0.04596 rpy=1.57079 -0.6004 1.57079; parent right_hand_virtual_a -> right_hand_z
- joint right_hand_ring_spread: origin xyz=0.003855 0 0.0655 rpy=-1.5707 -1.5707 0 -> xyz=0.003855 -0.006 0.0655 rpy=-1.5707 -1.5707 0; parent right_hand_e -> right_hand_e2

Commit message: [update] update svh hand right

File: robots/hands/schunk_hand/schunk_svh_hand_right.urdf (robot description, URDF)
Before this commit: robot svh, 29 links, 28 joints
Links:
- link right_hand_e1: geometry collision box size=0.042 0.038 0.015; collision box size=0.05 0.05 0.026

File: robots/hands/schunk_hand/schunk_svh_hand_right_glb.urdf (robot description, URDF)
Before this commit: robot svh, 29 links, 28 joints
Links:
- link right_hand_e1: geometry collision box size=0.042 0.038 0.015; collision box size=0.05 0.05 0.026
