Commit message: [update] update left svh hand

File: robots/hands/schunk_hand/schunk_svh_hand_left.urdf (robot description, URDF)
Before this commit: robot svh, 29 links, 28 joints
Links:
- link right_hand_a: geometry collision mesh filename=meshes/collision/d11_left.obj scale=1 1 1; visual mesh filename=meshes/visual/d11_left.obj scale=1 1 1
- link right_hand_b: geometry collision mesh filename=meshes/collision/d12_left.obj scale=1 1 1; visual mesh filename=meshes/visual/d12_left.obj scale=1 1 1
- link right_hand_c: geometry collision mesh filename=meshes/collision/d13_left.obj scale=1 1 1; visual mesh filename=meshes/visual/d13_left.obj scale=1 1 1
- link right_hand_e1: geometry collision box size=0.05 0.05 0.026; collision box size=0.0584 0.038 0.0641
- link right_hand_e2: geometry collision box size=0.012 0.018 0.021; collision box size=0.0246 0.035 0.0564
- link right_hand_z: geometry collision box size=0.006 0.024 0.033; collision box size=0.006 0.024 0.033
Joints:
- joint right_hand_Finger_Spread: axis 0 0 1 -> 0 0 -1; origin xyz=0.025355 -0.006 0.056 rpy=-1.5707 -1.5707 0 -> xyz=-0.025355 -0.006 0.056 rpy=-1.5707 -1.5707 0
- joint right_hand_Thumb_Flexion: origin xyz=0 0 0.04596 rpy=1.57079 -0.6004 1.57079 -> xyz=0 0 0.04596 rpy=-1.57079 -0.6004 -1.57079
- joint right_hand_Thumb_Opposition: axis 0 0 -1 -> 0 0 1; origin xyz=-0.0169 0.02626 0 rpy=0 0.2618 1.571 -> xyz=0.0169 0.02626 0 rpy=0 0.2618 1.571
- joint right_hand_index_spread: axis 0 0 1 -> 0 0 -1; origin xyz=-0.025 0 0.110 rpy=0 -1.5707 1.5707 -> xyz=0.025 0 0.110 rpy=0 -1.5707 1.5707
- joint right_hand_j3: axis 0 0 1 -> 0 0 -1
- joint right_hand_j4: axis 0 0 1 -> 0 0 -1
- joint right_hand_j5: origin xyz=0.0184 0.006 0.0375 rpy=0 0 0 -> xyz=-0.0184 0.006 0.0375 rpy=0 0 0
- joint right_hand_ring_spread: axis 0 0 1 -> 0 0 -1; origin xyz=0.003855 -0.006 0.0655 rpy=-1.5707 -1.5707 0 -> xyz=-0.003855 -0.006 0.0655 rpy=-1.5707 -1.5707 0

Commit message: [fix] fix svh hand collision and left hand joint

File: robots/hands/schunk_hand/schunk_svh_hand_left.urdf (robot description, URDF)
Before this commit: robot svh, 29 links, 28 joints
Links:
- link right_hand_e1: geometry collision box size=0.042 0.038 0.015; collision box size=0.05 0.05 0.026
- link right_hand_virtual_l: geometry collision sphere radius=0.01; visual mesh filename=meshes/visual/f10_f20.obj
Joints:
- joint right_hand_j5: axis 0 0 1 -> 0 0 -1

File: robots/hands/schunk_hand/schunk_svh_hand_left_glb.urdf (robot description, URDF)
Before this commit: robot svh, 29 links, 28 joints
Links:
- link right_hand_e1: geometry collision box size=0.042 0.038 0.015; collision box size=0.05 0.05 0.026
- link right_hand_virtual_l: geometry collision sphere radius=0.01; visual mesh filename=meshes/visual/f10_f20.glb

File: robots/hands/schunk_hand/schunk_svh_hand_right.urdf (robot description, URDF)
Before this commit: robot svh, 29 links, 28 joints
Links:
- link right_hand_virtual_l: geometry collision sphere radius=0.01; visual mesh filename=meshes/visual/f10_f20.obj

File: robots/hands/schunk_hand/schunk_svh_hand_right_glb.urdf (robot description, URDF)
Before this commit: robot svh, 29 links, 28 joints
Links:
- link right_hand_virtual_l: geometry collision sphere radius=0.01; visual mesh filename=meshes/visual/f10_f20.glb

Commit message: [fix] fix svh left hand

File: robots/hands/schunk_hand/schunk_svh_hand_left.urdf (robot description, URDF)
Before this commit: robot svh, 29 links, 28 joints
Links:
- removed link right_hand_a
- removed link right_hand_b
- removed link right_hand_base_link
- removed link right_hand_c
- removed link right_hand_e1
- removed link right_hand_e2
- removed link right_hand_i
- removed link right_hand_j
- removed link right_hand_k
- removed link right_hand_l
- removed link right_hand_m
- removed link right_hand_n
- removed link right_hand_o
- removed link right_hand_p
- removed link right_hand_q
- removed link right_hand_r
- removed link right_hand_s
- removed link right_hand_t
- removed link right_hand_virtual_i
- removed link right_hand_virtual_j
- removed link right_hand_virtual_k
- removed link right_hand_virtual_l
- removed link right_hand_z
- added link left_hand_a; collision mesh filename=meshes/collision/d11_left.obj scale=1 1 1; visual mesh filename=meshes/visual/d11_left.obj scale=1 1 1
- added link left_hand_b; collision mesh filename=meshes/collision/d12_left.obj scale=1 1 1; visual mesh filename=meshes/visual/d12_left.obj scale=1 1 1
- added link left_hand_base_link; collision cylinder length=0.045 radius=0.045; visual mesh filename=meshes/visual/base10.obj
- added link left_hand_c, mass 0.02; collision mesh filename=meshes/collision/d13_left.obj scale=1 1 1; visual mesh filename=meshes/visual/d13_left.obj scale=1 1 1
- added link left_hand_e1; collision box size=0.042 0.038 0.015; collision box size=0.05 0.05 0.026
- added link left_hand_e2; collision box size=0.012 0.018 0.021; collision box size=0.0246 0.035 0.0564
- added link left_hand_i; collision mesh filename=meshes/collision/f41.obj; visual mesh filename=meshes/visual/f41.obj
- added link left_hand_j; collision mesh filename=meshes/collision/f31.obj scale=1 1 1; visual mesh filename=meshes/visual/f31.obj
- added link left_hand_k; collision mesh filename=meshes/collision/f21.obj scale=1 1 1; visual mesh filename=meshes/visual/f21.obj
- added link left_hand_l; collision mesh filename=meshes/collision/f11.obj scale=1 1 1; visual mesh filename=meshes/visual/f11.obj
- added link left_hand_m, mass 0.02; collision mesh filename=meshes/collision/f42.obj; visual mesh filename=meshes/visual/f42.obj
- added link left_hand_n; collision mesh filename=meshes/collision/f22_f32.obj scale=1 1 1; visual mesh filename=meshes/visual/f22_f32.obj
- added link left_hand_o; collision mesh filename=meshes/collision/f22_f32.obj scale=1 1 1; visual mesh filename=meshes/visual/f22_f32.obj
- added link left_hand_p, mass 0.024; collision mesh filename=meshes/collision/f12.obj; visual mesh filename=meshes/visual/f12.obj
- added link left_hand_q, mass 0.02; collision mesh filename=meshes/collision/finger_tip.obj; visual mesh filename=meshes/visual/finger_tip.obj
- added link left_hand_r, mass 0.02; collision mesh filename=meshes/collision/finger_tip.obj scale=1 1 1; visual mesh filename=meshes/visual/finger_tip.obj
- added link left_hand_s, mass 0.02; collision mesh filename=meshes/collision/finger_tip.obj scale=1 1 1; visual mesh filename=meshes/visual/finger_tip.obj
- added link left_hand_t, mass 0.02; collision mesh filename=meshes/collision/finger_tip.obj scale=1 1 1; visual mesh filename=meshes/visual/finger_tip.obj
- added link left_hand_virtual_i; collision sphere radius=0.01; visual mesh filename=meshes/visual/f30_f40.obj
- added link left_hand_virtual_j; collision sphere radius=0.01; visual mesh filename=meshes/visual/f30_f40.obj
- added link left_hand_virtual_k; collision sphere radius=0.01; visual mesh filename=meshes/visual/f10_f20.obj
- added link left_hand_virtual_l; collision sphere radius=0.01; visual mesh filename=meshes/visual/f10_f20.obj
- added link left_hand_z; collision box size=0.006 0.024 0.033; collision box size=0.006 0.024 0.033
Joints:
- removed joint right_hand_Finger_Spread
- removed joint right_hand_Index_Finger_Distal
- removed joint right_hand_Index_Finger_Proximal
- removed joint right_hand_Middle_Finger_Distal
- removed joint right_hand_Middle_Finger_Proximal
- removed joint right_hand_Pinky
- removed joint right_hand_Ring_Finger
- removed joint right_hand_Thumb_Flexion
- removed joint right_hand_Thumb_Opposition
- removed joint right_hand_f4
- removed joint right_hand_index_spread
- removed joint right_hand_j12
- removed joint right_hand_j13
- removed joint right_hand_j14
- removed joint right_hand_j15
- removed joint right_hand_j16
- removed joint right_hand_j17
- removed joint right_hand_j3
- removed joint right_hand_j4
- removed joint right_hand_j5
- removed joint right_hand_middle_spread_dummy
- removed joint right_hand_ring_spread
- added joint left_hand_Finger_Spread: type revolute, parent left_hand_e2, child left_hand_virtual_i, origin xyz=-0.025355 -0.006 0.056 rpy=-1.5707 -1.5707 0, axis 0 0 1, limit lower=-0.5829 upper=0.0 effort=1000.0 velocity=1
- added joint left_hand_Index_Finger_Distal: type revolute, parent left_hand_l, child left_hand_p, origin xyz=0.04804 0 0 rpy=0 0 0, axis 0 0 1, limit lower=0 upper=1.334 effort=1000.0 velocity=1
- added joint left_hand_Index_Finger_Proximal: type revolute, parent left_hand_virtual_l, child left_hand_l, origin xyz=0 0 0 rpy=-1.5707 0 0, axis 0 0 1, limit lower=0.0 upper=0.79849 effort=1000.0 velocity=1
- added joint left_hand_Middle_Finger_Distal: type revolute, parent left_hand_k, child left_hand_o, origin xyz=0.05004 0 0 rpy=0 0 0, axis 0 0 1, limit lower=0 upper=1.334 effort=1000.0 velocity=1
- added joint left_hand_Middle_Finger_Proximal: type revolute, parent left_hand_virtual_k, child left_hand_k, origin xyz=0 0 0 rpy=-1.5707 0 0, axis 0 0 1, limit lower=0.0 upper=0.79849 effort=1000.0 velocity=1
- added joint left_hand_Pinky: type revolute, parent left_hand_virtual_i, child left_hand_i, origin xyz=0 0 0 rpy=1.5707 0 0, axis 0 0 1, limit lower=0.0 upper=0.98175 effort=1000.0 velocity=1
- added joint left_hand_Ring_Finger: type revolute, parent left_hand_virtual_j, child left_hand_j, origin xyz=0 0 0 rpy=1.5707 0 0, axis 0 0 1, limit lower=0.0 upper=0.98175 effort=1000.0 velocity=1
- added joint left_hand_Thumb_Flexion: type revolute, parent left_hand_z, child left_hand_a, origin xyz=0 0 0.04596 rpy=-1.57079 -0.6004 -1.57079, axis 0 0 1, limit lower=-0.9704 upper=0.0 effort=1000.0 velocity=1
- added joint left_hand_Thumb_Opposition: type revolute, parent left_hand_e1, child left_hand_z, origin xyz=0.0169 0.02626 0 rpy=0 0.2618 1.571, axis 0 0 1, limit lower=0.0 upper=0.9879 effort=1000.0 velocity=1
- added joint left_hand_f4: type fixed, parent left_hand_base_link, child left_hand_e1, origin xyz=0 -0.01313 0 rpy=0 0 0
- added joint left_hand_index_spread: type revolute, parent left_hand_e1, child left_hand_virtual_l, origin xyz=0.025 0 0.110 rpy=0 -1.5707 1.5707, axis 0 0 1, limit lower=-0.28833 upper=0.0 effort=1000.0 velocity=1, mimic joint=left_hand_Finger_Spread multiplier=0.5 offset=0
- added joint left_hand_j12: type revolute, parent left_hand_j, child left_hand_n, origin xyz=0.05004 0 0 rpy=0 0 0, axis 0 0 1, limit lower=0 upper=1.334 effort=1000.0 velocity=1, mimic joint=left_hand_Ring_Finger multiplier=1.3588 offset=0
- added joint left_hand_j13: type revolute, parent left_hand_i, child left_hand_m, origin xyz=0.04454 0 0 rpy=0 0 0, axis 0 0 1, limit lower=0 upper=1.334 effort=1000.0 velocity=1, mimic joint=left_hand_Pinky multiplier=1.35880 offset=0
- added joint left_hand_j14: type revolute, parent left_hand_p, child left_hand_t, origin xyz=0.026 0 0 rpy=0 0 0, axis 0 0 1, limit lower=0 upper=1.394 effort=1000.0 velocity=1, mimic joint=left_hand_Index_Finger_Distal multiplier=1.0450 offset=0
- added joint left_hand_j15: type revolute, parent left_hand_o, child left_hand_s, origin xyz=0.032 0 0 rpy=0 0 0, axis 0 0 1, limit lower=0 upper=1.334 effort=1000.0 velocity=1, mimic joint=left_hand_Middle_Finger_Distal multiplier=1.0454 offset=0
- added joint left_hand_j16: type revolute, parent left_hand_n, child left_hand_r, origin xyz=0.032 0 0 rpy=0 0 0, axis 0 0 1, limit lower=0 upper=1.395 effort=1000.0 velocity=1, mimic joint=left_hand_Ring_Finger multiplier=1.42093 offset=0
- added joint left_hand_j17: type revolute, parent left_hand_m, child left_hand_q, origin xyz=0.022 0 0 rpy=0 0 0, axis 0 0 1, limit lower=0 upper=1.3971 effort=1000.0 velocity=1, mimic joint=left_hand_Pinky multiplier=1.42307 offset=0
- added joint left_hand_j3: type revolute, parent left_hand_a, child left_hand_b, origin xyz=0.0485 0 0 rpy=0 0 0, axis 0 0 1, limit lower=-0.98506 upper=0.0 effort=1000.0 velocity=1, mimic joint=left_hand_Thumb_Flexion multiplier=1.01511 offset=0
- added joint left_hand_j4: type revolute, parent left_hand_b, child left_hand_c, origin xyz=0.030 0 0 rpy=0 0 0, axis 0 0 1, limit lower=-1.406 upper=0 effort=1000.0 velocity=1, mimic joint=left_hand_Thumb_Flexion multiplier=1.44889 offset=0
- added joint left_hand_j5: type revolute, parent left_hand_e1, child left_hand_e2, origin xyz=-0.0184 0.006 0.0375 rpy=0 0 0, axis 0 0 1, limit lower=-0.98786 upper=0.0 effort=1000.0 velocity=1, mimic joint=left_hand_Thumb_Opposition multiplier=1 offset=0
- added joint left_hand_middle_spread_dummy: type fixed, parent left_hand_e1, child left_hand_virtual_k, origin xyz=0 0 0.110 rpy=0 -1.5707 1.5707
- added joint left_hand_ring_spread: type revolute, parent left_hand_e2, child left_hand_virtual_j, origin xyz=-0.003855 -0.006 0.0655 rpy=-1.5707 -1.5707 0, axis 0 0 1, limit lower=-0.28833 upper=0.0 effort=1000.0 velocity=1, mimic joint=left_hand_Finger_Spread multiplier=0.5 offset=0
- joint fftip_joint: parent right_hand_t -> left_hand_t
- joint lftip_joint: parent right_hand_q -> left_hand_q
- joint mftip_joint: parent right_hand_s -> left_hand_s
- joint rftip_joint: parent right_hand_r -> left_hand_r
- joint root_joint: child right_hand_base_link -> left_hand_base_link
- joint thtip_joint: parent right_hand_c -> left_hand_c

File: robots/hands/schunk_hand/schunk_svh_hand_left_glb.urdf (robot description, URDF)
Before this commit: robot svh, 29 links, 28 joints
Links:
- removed link right_hand_a
- removed link right_hand_b
- removed link right_hand_base_link
- removed link right_hand_c
- removed link right_hand_e1
- removed link right_hand_e2
- removed link right_hand_i
- removed link right_hand_j
- removed link right_hand_k
- removed link right_hand_l
- removed link right_hand_m
- removed link right_hand_n
- removed link right_hand_o
- removed link right_hand_p
- removed link right_hand_q
- removed link right_hand_r
- removed link right_hand_s
- removed link right_hand_t
- removed link right_hand_virtual_i
- removed link right_hand_virtual_j
- removed link right_hand_virtual_k
- removed link right_hand_virtual_l
- removed link right_hand_z
- added link left_hand_a; collision mesh filename=meshes/collision/d11_left.obj scale=1 1 1; visual mesh filename=meshes/visual/d11_left.glb scale=1 1 1
- added link left_hand_b; collision mesh filename=meshes/collision/d12_left.obj scale=1 1 1; visual mesh filename=meshes/visual/d12_left.glb scale=1 1 1
- added link left_hand_base_link; collision cylinder length=0.045 radius=0.045; visual mesh filename=meshes/visual/base10.glb
- added link left_hand_c, mass 0.02; collision mesh filename=meshes/collision/d13_left.obj scale=1 1 1; visual mesh filename=meshes/visual/d13_left.glb scale=1 1 1
- added link left_hand_e1; collision box size=0.042 0.038 0.015; collision box size=0.05 0.05 0.026
- added link left_hand_e2; collision box size=0.012 0.018 0.021; collision box size=0.0246 0.035 0.0564
- added link left_hand_i; collision mesh filename=meshes/collision/f41.obj; visual mesh filename=meshes/visual/f41.glb
- added link left_hand_j; collision mesh filename=meshes/collision/f31.obj scale=1 1 1; visual mesh filename=meshes/visual/f31.glb
- added link left_hand_k; collision mesh filename=meshes/collision/f21.obj scale=1 1 1; visual mesh filename=meshes/visual/f21.glb
- added link left_hand_l; collision mesh filename=meshes/collision/f11.obj scale=1 1 1; visual mesh filename=meshes/visual/f11.glb
- added link left_hand_m, mass 0.02; collision mesh filename=meshes/collision/f42.obj; visual mesh filename=meshes/visual/f42.glb
- added link left_hand_n; collision mesh filename=meshes/collision/f22_f32.obj scale=1 1 1; visual mesh filename=meshes/visual/f22_f32.glb
- added link left_hand_o; collision mesh filename=meshes/collision/f22_f32.obj scale=1 1 1; visual mesh filename=meshes/visual/f22_f32.glb
- added link left_hand_p, mass 0.024; collision mesh filename=meshes/collision/f12.obj; visual mesh filename=meshes/visual/f12.glb
- added link left_hand_q, mass 0.02; collision mesh filename=meshes/collision/finger_tip.obj; visual mesh filename=meshes/visual/finger_tip.glb
- added link left_hand_r, mass 0.02; collision mesh filename=meshes/collision/finger_tip.obj scale=1 1 1; visual mesh filename=meshes/visual/finger_tip.glb
- added link left_hand_s, mass 0.02; collision mesh filename=meshes/collision/finger_tip.obj scale=1 1 1; visual mesh filename=meshes/visual/finger_tip.glb
- added link left_hand_t, mass 0.02; collision mesh filename=meshes/collision/finger_tip.obj scale=1 1 1; visual mesh filename=meshes/visual/finger_tip.glb
- added link left_hand_virtual_i; collision sphere radius=0.01; visual mesh filename=meshes/visual/f30_f40.glb
- added link left_hand_virtual_j; collision sphere radius=0.01; visual mesh filename=meshes/visual/f30_f40.glb
- added link left_hand_virtual_k; collision sphere radius=0.01; visual mesh filename=meshes/visual/f10_f20.glb
- added link left_hand_virtual_l; collision sphere radius=0.01; visual mesh filename=meshes/visual/f10_f20.glb
- added link left_hand_z; collision box size=0.006 0.024 0.033; collision box size=0.006 0.024 0.033
Joints:
- removed joint right_hand_Finger_Spread
- removed joint right_hand_Index_Finger_Distal
- removed joint right_hand_Index_Finger_Proximal
- removed joint right_hand_Middle_Finger_Distal
- removed joint right_hand_Middle_Finger_Proximal
- removed joint right_hand_Pinky
- removed joint right_hand_Ring_Finger
- removed joint right_hand_Thumb_Flexion
- removed joint right_hand_Thumb_Opposition
- removed joint right_hand_f4
- removed joint right_hand_index_spread
- removed joint right_hand_j12
- removed joint right_hand_j13
- removed joint right_hand_j14
- removed joint right_hand_j15
- removed joint right_hand_j16
- removed joint right_hand_j17
- removed joint right_hand_j3
- removed joint right_hand_j4
- removed joint right_hand_j5
- removed joint right_hand_middle_spread_dummy
- removed joint right_hand_ring_spread
- added joint left_hand_Finger_Spread: type revolute, parent left_hand_e2, child left_hand_virtual_i, origin xyz=-0.025355 -0.006 0.056 rpy=-1.5707 -1.5707 0, axis 0 0 1, limit lower=-0.5829 upper=0.0 effort=1000.0 velocity=1
- added joint left_hand_Index_Finger_Distal: type revolute, parent left_hand_l, child left_hand_p, origin xyz=0.04804 0 0 rpy=0 0 0, axis 0 0 1, limit lower=0 upper=1.334 effort=1000.0 velocity=1
- added joint left_hand_Index_Finger_Proximal: type revolute, parent left_hand_virtual_l, child left_hand_l, origin xyz=0 0 0 rpy=-1.5707 0 0, axis 0 0 1, limit lower=0.0 upper=0.79849 effort=1000.0 velocity=1
- added joint left_hand_Middle_Finger_Distal: type revolute, parent left_hand_k, child left_hand_o, origin xyz=0.05004 0 0 rpy=0 0 0, axis 0 0 1, limit lower=0 upper=1.334 effort=1000.0 velocity=1
- added joint left_hand_Middle_Finger_Proximal: type revolute, parent left_hand_virtual_k, child left_hand_k, origin xyz=0 0 0 rpy=-1.5707 0 0, axis 0 0 1, limit lower=0.0 upper=0.79849 effort=1000.0 velocity=1
- added joint left_hand_Pinky: type revolute, parent left_hand_virtual_i, child left_hand_i, origin xyz=0 0 0 rpy=1.5707 0 0, axis 0 0 1, limit lower=0.0 upper=0.98175 effort=1000.0 velocity=1
- added joint left_hand_Ring_Finger: type revolute, parent left_hand_virtual_j, child left_hand_j, origin xyz=0 0 0 rpy=1.5707 0 0, axis 0 0 1, limit lower=0.0 upper=0.98175 effort=1000.0 velocity=1
- added joint left_hand_Thumb_Flexion: type revolute, parent left_hand_z, child left_hand_a, origin xyz=0 0 0.04596 rpy=-1.57079 -0.6004 -1.57079, axis 0 0 1, limit lower=-0.9704 upper=0.0 effort=1000.0 velocity=1
- added joint left_hand_Thumb_Opposition: type revolute, parent left_hand_e1, child left_hand_z, origin xyz=0.0169 0.02626 0 rpy=0 0.2618 1.571, axis 0 0 1, limit lower=0.0 upper=0.9879 effort=1000.0 velocity=1
- added joint left_hand_f4: type fixed, parent left_hand_base_link, child left_hand_e1, origin xyz=0 -0.01313 0 rpy=0 0 0
- added joint left_hand_index_spread: type revolute, parent left_hand_e1, child left_hand_virtual_l, origin xyz=0.025 0 0.110 rpy=0 -1.5707 1.5707, axis 0 0 1, limit lower=-0.28833 upper=0.0 effort=1000.0 velocity=1, mimic joint=left_hand_Finger_Spread multiplier=0.5 offset=0
- added joint left_hand_j12: type revolute, parent left_hand_j, child left_hand_n, origin xyz=0.05004 0 0 rpy=0 0 0, axis 0 0 1, limit lower=0 upper=1.334 effort=1000.0 velocity=1, mimic joint=left_hand_Ring_Finger multiplier=1.3588 offset=0
- added joint left_hand_j13: type revolute, parent left_hand_i, child left_hand_m, origin xyz=0.04454 0 0 rpy=0 0 0, axis 0 0 1, limit lower=0 upper=1.334 effort=1000.0 velocity=1, mimic joint=left_hand_Pinky multiplier=1.35880 offset=0
- added joint left_hand_j14: type revolute, parent left_hand_p, child left_hand_t, origin xyz=0.026 0 0 rpy=0 0 0, axis 0 0 1, limit lower=0 upper=1.394 effort=1000.0 velocity=1, mimic joint=left_hand_Index_Finger_Distal multiplier=1.0450 offset=0
- added joint left_hand_j15: type revolute, parent left_hand_o, child left_hand_s, origin xyz=0.032 0 0 rpy=0 0 0, axis 0 0 1, limit lower=0 upper=1.334 effort=1000.0 velocity=1, mimic joint=left_hand_Middle_Finger_Distal multiplier=1.0454 offset=0
- added joint left_hand_j16: type revolute, parent left_hand_n, child left_hand_r, origin xyz=0.032 0 0 rpy=0 0 0, axis 0 0 1, limit lower=0 upper=1.395 effort=1000.0 velocity=1, mimic joint=left_hand_Ring_Finger multiplier=1.42093 offset=0
- added joint left_hand_j17: type revolute, parent left_hand_m, child left_hand_q, origin xyz=0.022 0 0 rpy=0 0 0, axis 0 0 1, limit lower=0 upper=1.3971 effort=1000.0 velocity=1, mimic joint=left_hand_Pinky multiplier=1.42307 offset=0
- added joint left_hand_j3: type revolute, parent left_hand_a, child left_hand_b, origin xyz=0.0485 0 0 rpy=0 0 0, axis 0 0 1, limit lower=-0.98506 upper=0.0 effort=1000.0 velocity=1, mimic joint=left_hand_Thumb_Flexion multiplier=1.01511 offset=0
- added joint left_hand_j4: type revolute, parent left_hand_b, child left_hand_c, origin xyz=0.030 0 0 rpy=0 0 0, axis 0 0 1, limit lower=-1.406 upper=0 effort=1000.0 velocity=1, mimic joint=left_hand_Thumb_Flexion multiplier=1.44889 offset=0
- added joint left_hand_j5: type revolute, parent left_hand_e1, child left_hand_e2, origin xyz=-0.0184 0.006 0.0375 rpy=0 0 0, axis 0 0 1, limit lower=-0.98786 upper=0.0 effort=1000.0 velocity=1, mimic joint=left_hand_Thumb_Opposition multiplier=1 offset=0
- added joint left_hand_middle_spread_dummy: type fixed, parent left_hand_e1, child left_hand_virtual_k, origin xyz=0 0 0.110 rpy=0 -1.5707 1.5707
- added joint left_hand_ring_spread: type revolute, parent left_hand_e2, child left_hand_virtual_j, origin xyz=-0.003855 -0.006 0.0655 rpy=-1.5707 -1.5707 0, axis 0 0 1, limit lower=-0.28833 upper=0.0 effort=1000.0 velocity=1, mimic joint=left_hand_Finger_Spread multiplier=0.5 offset=0
- joint fftip_joint: parent right_hand_t -> left_hand_t
- joint lftip_joint: parent right_hand_q -> left_hand_q
- joint mftip_joint: parent right_hand_s -> left_hand_s
- joint rftip_joint: parent right_hand_r -> left_hand_r
- joint root_joint: child right_hand_base_link -> left_hand_base_link
- joint thtip_joint: parent right_hand_c -> left_hand_c
