Commit message: [fix] fix simple allegro tactile model

File: robots/hands/allegro_hand/variation/allegro_hand_right_fsr_simple.urdf (robot description, URDF)
Before this commit: robot allegro_right, 39 links, 38 joints
Links:
- link link_15.0_tip_fsr: geometry collision box size=0.003 0.0228 0.0168; visual box size=0.003 0.0228 0.0168
