Commit message: [add] add aux finger tip frame for dclaw

File: robots/hands/dclaw_gripper/dclaw_gripper.urdf (robot description, URDF)
Before this commit: robot dclaw_gripper, 11 links, 10 joints
Links:
- added link link_f1_head
- added link link_f2_head
- added link link_f3_head
Joints:
- added joint joint_f1_head: type fixed, parent link_f1_3, child link_f1_head, origin xyz=0.084 0 0 rpy=0 0 0
- added joint joint_f2_head: type fixed, parent link_f2_3, child link_f2_head, origin xyz=0.084 0 0 rpy=0 0 0
- added joint joint_f3_head: type fixed, parent link_f3_3, child link_f3_head, origin xyz=0.084 0 0 rpy=0 0 0

File: robots/hands/dclaw_gripper/dclaw_gripper_glb.urdf (robot description, URDF)
Before this commit: robot dclaw_gripper, 11 links, 10 joints
Links:
- added link link_f1_head
- added link link_f2_head
- added link link_f3_head
Joints:
- added joint joint_f1_head: type fixed, parent link_f1_3, child link_f1_head, origin xyz=0.084 0 0 rpy=0 0 0
- added joint joint_f2_head: type fixed, parent link_f2_3, child link_f2_head, origin xyz=0.084 0 0 rpy=0 0 0
- added joint joint_f3_head: type fixed, parent link_f3_3, child link_f3_head, origin xyz=0.084 0 0 rpy=0 0 0
