Commit message: [fix] fix ability hand model

File: robots/hands/ability_hand/ability_hand_left.urdf (robot description, URDF)
Before this commit: robot ability_hand, 18 links, 17 joints
Links:
- link index_L1: geometry collision box size=0.012 0.012 0.002; collision box size=0.012 0.012 0.002

File: robots/hands/ability_hand/ability_hand_left_glb.urdf (robot description, URDF)
Before this commit: robot ability_hand, 18 links, 17 joints
Links:
- link index_L1: geometry collision box size=0.012 0.012 0.002; collision box size=0.012 0.012 0.002

File: robots/hands/ability_hand/ability_hand_right.urdf (robot description, URDF)
Before this commit: robot ability_hand, 18 links, 17 joints
Links:
- link index_L1: geometry collision box size=0.012 0.012 0.002; collision box size=0.012 0.012 0.002

File: robots/hands/ability_hand/ability_hand_right_glb.urdf (robot description, URDF)
Before this commit: robot ability_hand, 18 links, 17 joints
Links:
- link index_L1: geometry collision box size=0.012 0.012 0.002; collision box size=0.012 0.012 0.002

Commit message: [update] update ability finger tip

File: robots/hands/ability_hand/ability_hand_left.urdf (robot description, URDF)
Before this commit: robot ability_hand, 18 links, 17 joints
Links:
- removed link index_anchor
- removed link middle_anchor
- removed link pinky_anchor
- removed link ring_anchor
- removed link thumb_anchor
- added link index_tip
- added link middle_tip
- added link pinky_tip
- added link ring_tip
- added link thumb_tip
Joints:
- removed joint idx_anchor
- removed joint mid_anchor
- removed joint pnky_anchor
- removed joint rng_anchor
- removed joint thmb_anchor
- added joint index_tip_joint: type fixed, parent index_L2, child index_tip, origin xyz=0.035  -0.018 0 rpy=0 0 0
- added joint middle_tip_joint: type fixed, parent middle_L2, child middle_tip, origin xyz=0.035  -0.018 0 rpy=0 0 0
- added joint pinky_tip_joint: type fixed, parent pinky_L2, child pinky_tip, origin xyz=0.035  -0.018 0 rpy=0 0 0
- added joint ring_tip_joint: type fixed, parent ring_L2, child ring_tip, origin xyz=0.035  -0.018 0 rpy=0 0 0
- added joint thumb_tip_joint: type fixed, parent thumb_L2, child thumb_tip, origin xyz=0.065 0.016 0 rpy=0 0 0

File: robots/hands/ability_hand/ability_hand_left_glb.urdf (robot description, URDF)
Before this commit: robot ability_hand, 18 links, 17 joints
Links:
- removed link index_anchor
- removed link middle_anchor
- removed link pinky_anchor
- removed link ring_anchor
- removed link thumb_anchor
- added link index_tip
- added link middle_tip
- added link pinky_tip
- added link ring_tip
- added link thumb_tip
Joints:
- removed joint idx_anchor
- removed joint mid_anchor
- removed joint pnky_anchor
- removed joint rng_anchor
- removed joint thmb_anchor
- added joint index_tip_joint: type fixed, parent index_L2, child index_tip, origin xyz=0.035  -0.018 0 rpy=0 0 0
- added joint middle_tip_joint: type fixed, parent middle_L2, child middle_tip, origin xyz=0.035  -0.018 0 rpy=0 0 0
- added joint pinky_tip_joint: type fixed, parent pinky_L2, child pinky_tip, origin xyz=0.035  -0.018 0 rpy=0 0 0
- added joint ring_tip_joint: type fixed, parent ring_L2, child ring_tip, origin xyz=0.035  -0.018 0 rpy=0 0 0
- added joint thumb_tip_joint: type fixed, parent thumb_L2, child thumb_tip, origin xyz=0.065 0.016 0 rpy=0 0 0

File: robots/hands/ability_hand/ability_hand_right.urdf (robot description, URDF)
Before this commit: robot ability_hand, 18 links, 17 joints
Links:
- removed link index_anchor
- removed link middle_anchor
- removed link pinky_anchor
- removed link ring_anchor
- removed link thumb_anchor
- added link index_tip
- added link middle_tip
- added link pinky_tip
- added link ring_tip
- added link thumb_tip
Joints:
- removed joint idx_anchor
- removed joint mid_anchor
- removed joint pnky_anchor
- removed joint rng_anchor
- removed joint thmb_anchor
- added joint index_tip_joint: type fixed, parent index_L2, child index_tip, origin xyz=0.035  -0.018 0 rpy=0 0 0
- added joint middle_tip_joint: type fixed, parent middle_L2, child middle_tip, origin xyz=0.035  -0.018 0 rpy=0 0 0
- added joint pinky_tip_joint: type fixed, parent pinky_L2, child pinky_tip, origin xyz=0.035  -0.018 0 rpy=0 0 0
- added joint ring_tip_joint: type fixed, parent ring_L2, child ring_tip, origin xyz=0.035  -0.018 0 rpy=0 0 0
- added joint thumb_tip_joint: type fixed, parent thumb_L2, child thumb_tip, origin xyz=0.065 0.016 0 rpy=0 0 0

File: robots/hands/ability_hand/ability_hand_right_glb.urdf (robot description, URDF)
Before this commit: robot ability_hand, 18 links, 17 joints
Links:
- removed link index_anchor
- removed link middle_anchor
- removed link pinky_anchor
- removed link ring_anchor
- removed link thumb_anchor
- added link index_tip
- added link middle_tip
- added link pinky_tip
- added link ring_tip
- added link thumb_tip
Joints:
- removed joint idx_anchor
- removed joint mid_anchor
- removed joint pnky_anchor
- removed joint rng_anchor
- removed joint thmb_anchor
- added joint index_tip_joint: type fixed, parent index_L2, child index_tip, origin xyz=0.035  -0.018 0 rpy=0 0 0
- added joint middle_tip_joint: type fixed, parent middle_L2, child middle_tip, origin xyz=0.035  -0.018 0 rpy=0 0 0
- added joint pinky_tip_joint: type fixed, parent pinky_L2, child pinky_tip, origin xyz=0.035  -0.018 0 rpy=0 0 0
- added joint ring_tip_joint: type fixed, parent ring_L2, child ring_tip, origin xyz=0.035  -0.018 0 rpy=0 0 0
- added joint thumb_tip_joint: type fixed, parent thumb_L2, child thumb_tip, origin xyz=0.065 0.016 0 rpy=0 0 0
