Commit message: [update] update xarm7 ability finger tip

File: robots/assembly/xarm7_ability/xarm7_ability_right_hand.urdf (robot description, URDF)
Before this commit: robot xarm7, 25 links, 24 joints
Links:
- removed link index_anchor
- removed link middle_anchor
- removed link pinky_anchor
- removed link ring_anchor
- removed link thumb_anchor
- added link index_tip
- added link middle_tip
- added link pinky_tip
- added link ring_tip
- added link thumb_tip
- link index_L1: geometry collision box size=0.012 0.012 0.002; collision box size=0.012 0.012 0.002
Joints:
- removed joint idx_anchor
- removed joint mid_anchor
- removed joint pnky_anchor
- removed joint rng_anchor
- removed joint thmb_anchor
- added joint index_tip_joint: type fixed, parent index_L2, child index_tip, origin xyz=0.035  -0.018 0 rpy=0 0 0
- added joint middle_tip_joint: type fixed, parent middle_L2, child middle_tip, origin xyz=0.035  -0.018 0 rpy=0 0 0
- added joint pinky_tip_joint: type fixed, parent pinky_L2, child pinky_tip, origin xyz=0.035  -0.018 0 rpy=0 0 0
- added joint ring_tip_joint: type fixed, parent ring_L2, child ring_tip, origin xyz=0.035  -0.018 0 rpy=0 0 0
- added joint thumb_tip_joint: type fixed, parent thumb_L2, child thumb_tip, origin xyz=0.065 0.016 0 rpy=0 0 0

Commit message: [add] add ability mount

File: robots/assembly/xarm7_ability/xarm7_ability_right_hand.urdf (robot description, URDF)
Before this commit: robot xarm7, 25 links, 24 joints
Links:
- link link7: geometry collision cylinder length=0.018 radius=0.0365; collision mesh filename=../../arms/xarm7/meshes/collision/link7.obj
Joints:
- joint joint_eef: origin xyz=0 0 0 rpy=0 0 -1.57079 -> xyz=0 0 0.018 rpy=0 0 -1.57079
