Commit message: [update] update xarm7 ability assembly

File: robots/assembly/xarm7_ability/xarm7_ability_left_hand_glb.urdf (robot description, URDF)
Before this commit: robot xarm7, 26 links, 25 joints
Links:
- link base: geometry collision mesh filename=../../hands/ability_hand/meshes/collision/wristmesh_C.obj; visual mesh filename=../../hands/ability_hand/meshes/visual/wristmesh.glb
- link index_L1: geometry collision box size=0.012 0.012 0.002; collision box size=0.012 0.012 0.002
- link index_L2: geometry collision mesh filename=../../hands/ability_hand/meshes/collision/idx-F2_C.obj; collision sphere radius=0.007
- link link1: geometry collision mesh filename=../../arms/xarm7/meshes/collision/link1.obj; visual mesh filename=../../arms/xarm7/meshes/visual/link1.glb
- link link2: geometry collision mesh filename=../../arms/xarm7/meshes/collision/link2.obj; visual mesh filename=../../arms/xarm7/meshes/visual/link2.glb
- link link3: geometry collision mesh filename=../../arms/xarm7/meshes/collision/link3.obj; visual mesh filename=../../arms/xarm7/meshes/visual/link3.glb
- link link4: geometry collision mesh filename=../../arms/xarm7/meshes/collision/link4.obj; visual mesh filename=../../arms/xarm7/meshes/visual/link4.glb
- link link5: geometry collision mesh filename=../../arms/xarm7/meshes/collision/link5.obj; visual mesh filename=../../arms/xarm7/meshes/visual/link5.glb
- link link6: geometry collision mesh filename=../../arms/xarm7/meshes/collision/link6.obj; visual mesh filename=../../arms/xarm7/meshes/visual/link6.glb
- link link7: geometry collision cylinder length=0.018 radius=0.0365; collision mesh filename=../../arms/xarm7/meshes/collision/link7.obj
- link link_base: geometry collision mesh filename=../../arms/xarm7/meshes/collision/link_base.obj; visual mesh filename=../../arms/xarm7/meshes/visual/link_base.glb
- link middle_L1: geometry collision box size=0.012 0.012 0.002; collision box size=0.012 0.012 0.002
- link middle_L2: geometry collision mesh filename=../../hands/ability_hand/meshes/collision/idx-F2_C.obj; collision sphere radius=0.007
- link pinky_L1: geometry collision box size=0.012 0.012 0.002; collision box size=0.012 0.012 0.002
- link pinky_L2: geometry collision mesh filename=../../hands/ability_hand/meshes/collision/idx-F2_C.obj; collision sphere radius=0.007
- link ring_L1: geometry collision box size=0.012 0.012 0.002; collision box size=0.012 0.012 0.002
- link ring_L2: geometry collision mesh filename=../../hands/ability_hand/meshes/collision/idx-F2_C.obj; collision sphere radius=0.007
- link thumb_L1: geometry collision mesh filename=../../hands/ability_hand/meshes/collision/thumb-F1_C.obj; visual mesh filename=../../hands/ability_hand/meshes/visual/thumb-F1.glb
- link thumb_L2: geometry collision mesh filename=../../hands/ability_hand/meshes/collision/thumb-F2_C.obj; visual mesh filename=../../hands/ability_hand/meshes/visual/thumb-F2.glb
- link thumb_base: geometry collision mesh filename=../../hands/ability_hand/meshes/collision/FB_palm_ref.obj; visual mesh filename=../../hands/ability_hand/meshes/visual/FB_palm_ref.glb

File: robots/assembly/xarm7_ability/xarm7_ability_right_hand.urdf (robot description, URDF)
Before this commit: robot xarm7, 26 links, 25 joints
Links:
- link base: geometry collision mesh filename=../../hands/ability_hand/meshes/collision/wristmesh_C.obj; visual mesh filename=../../hands/ability_hand/meshes/visual/wristmesh.obj
- link index_L1: geometry collision box size=0.012 0.012 0.002; collision box size=0.012 0.012 0.002
- link index_L2: geometry collision mesh filename=../../hands/ability_hand/meshes/collision/idx-F2_C.obj; collision sphere radius=0.007
- link link1: geometry collision mesh filename=../../arms/xarm7/meshes/collision/link1.obj; visual mesh filename=../../arms/xarm7/meshes/visual/link1.obj
- link link2: geometry collision mesh filename=../../arms/xarm7/meshes/collision/link2.obj; visual mesh filename=../../arms/xarm7/meshes/visual/link2.obj
- link link3: geometry collision mesh filename=../../arms/xarm7/meshes/collision/link3.obj; visual mesh filename=../../arms/xarm7/meshes/visual/link3.obj
- link link4: geometry collision mesh filename=../../arms/xarm7/meshes/collision/link4.obj; visual mesh filename=../../arms/xarm7/meshes/visual/link4.obj
- link link5: geometry collision mesh filename=../../arms/xarm7/meshes/collision/link5.obj; visual mesh filename=../../arms/xarm7/meshes/visual/link5.obj
- link link6: geometry collision mesh filename=../../arms/xarm7/meshes/collision/link6.obj; visual mesh filename=../../arms/xarm7/meshes/visual/link6.obj
- link link7: geometry collision cylinder length=0.018 radius=0.0365; collision mesh filename=../../arms/xarm7/meshes/collision/link7.obj
- link link_base: geometry collision mesh filename=../../arms/xarm7/meshes/collision/link_base.obj; visual mesh filename=../../arms/xarm7/meshes/visual/link_base.obj
- link middle_L1: geometry collision box size=0.012 0.012 0.002; collision box size=0.012 0.012 0.002
- link middle_L2: geometry collision mesh filename=../../hands/ability_hand/meshes/collision/idx-F2_C.obj; collision sphere radius=0.007
- link pinky_L1: geometry collision box size=0.012 0.012 0.002; collision box size=0.012 0.012 0.002
- link pinky_L2: geometry collision mesh filename=../../hands/ability_hand/meshes/collision/idx-F2_C.obj; collision sphere radius=0.007
- link ring_L1: geometry collision box size=0.012 0.012 0.002; collision box size=0.012 0.012 0.002
- link ring_L2: geometry collision mesh filename=../../hands/ability_hand/meshes/collision/idx-F2_C.obj; collision sphere radius=0.007
- link thumb_L1: geometry collision mesh filename=../../hands/ability_hand/meshes/collision/thumb-F1-MIR_C.obj; visual mesh filename=../../hands/ability_hand/meshes/visual/thumb-F1-MIR.obj
- link thumb_L2: geometry collision mesh filename=../../hands/ability_hand/meshes/collision/thumb-F2_C.obj; visual mesh filename=../../hands/ability_hand/meshes/visual/thumb-F2.obj
- link thumb_base: geometry collision mesh filename=../../hands/ability_hand/meshes/collision/FB_palm_ref_MIR.o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; visual mesh filename=../../hands/ability_hand/meshes/visual/FB_palm_ref_MIR.obj

File: robots/assembly/xarm7_ability/xarm7_ability_right_hand_glb.urdf (robot description, URDF)
Before this commit: robot xarm7, 26 links, 25 joints
Links:
- link base: geometry collision mesh filename=../../hands/ability_hand/meshes/collision/wristmesh_C.obj; visual mesh filename=../../hands/ability_hand/meshes/visual/wristmesh.glb
- link index_L1: geometry collision box size=0.012 0.012 0.002; collision box size=0.012 0.012 0.002
- link index_L2: geometry collision mesh filename=../../hands/ability_hand/meshes/collision/idx-F2_C.obj; collision sphere radius=0.007
- link link1: geometry collision mesh filename=../../arms/xarm7/meshes/collision/link1.obj; visual mesh filename=../../arms/xarm7/meshes/visual/link1.glb
- link link2: geometry collision mesh filename=../../arms/xarm7/meshes/collision/link2.obj; visual mesh filename=../../arms/xarm7/meshes/visual/link2.glb
- link link3: geometry collision mesh filename=../../arms/xarm7/meshes/collision/link3.obj; visual mesh filename=../../arms/xarm7/meshes/visual/link3.glb
- link link4: geometry collision mesh filename=../../arms/xarm7/meshes/collision/link4.obj; visual mesh filename=../../arms/xarm7/meshes/visual/link4.glb
- link link5: geometry collision mesh filename=../../arms/xarm7/meshes/collision/link5.obj; visual mesh filename=../../arms/xarm7/meshes/visual/link5.glb
- link link6: geometry collision mesh filename=../../arms/xarm7/meshes/collision/link6.obj; visual mesh filename=../../arms/xarm7/meshes/visual/link6.glb
- link link7: geometry collision cylinder length=0.018 radius=0.0365; collision mesh filename=../../arms/xarm7/meshes/collision/link7.obj
- link link_base: geometry collision mesh filename=../../arms/xarm7/meshes/collision/link_base.obj; visual mesh filename=../../arms/xarm7/meshes/visual/link_base.glb
- link middle_L1: geometry collision box size=0.012 0.012 0.002; collision box size=0.012 0.012 0.002
- link middle_L2: geometry collision mesh filename=../../hands/ability_hand/meshes/collision/idx-F2_C.obj; collision sphere radius=0.007
- link pinky_L1: geometry collision box size=0.012 0.012 0.002; collision box size=0.012 0.012 0.002
- link pinky_L2: geometry collision mesh filename=../../hands/ability_hand/meshes/collision/idx-F2_C.obj; collision sphere radius=0.007
- link ring_L1: geometry collision box size=0.012 0.012 0.002; collision box size=0.012 0.012 0.002
- link ring_L2: geometry collision mesh filename=../../hands/ability_hand/meshes/collision/idx-F2_C.obj; collision sphere radius=0.007
- link thumb_L1: geometry collision mesh filename=../../hands/ability_hand/meshes/collision/thumb-F1-MIR_C.obj; visual mesh filename=../../hands/ability_hand/meshes/visual/thumb-F1-MIR.glb
- link thumb_L2: geometry collision mesh filename=../../hands/ability_hand/meshes/collision/thumb-F2_C.obj; visual mesh filename=../../hands/ability_hand/meshes/visual/thumb-F2.glb
- link thumb_base: geometry collision mesh filename=../../hands/ability_hand/meshes/collision/FB_palm_ref_MIR.o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; visual mesh filename=../../hands/ability_hand/meshes/visual/FB_palm_ref_MIR.glb
Joints:
- joint index_q1: origin xyz=-9.49e-3 -13.04e-3 -62.95e-3 rpy=-1.982050 1.284473 -2.090591 -> xyz=9.49e-3 -13.04e-3 -62.95e-3  rpy= -1.1595426535897932 1.284473 -1.0510016535897932 
- joint middle_q1: origin xyz=9.653191e-3 -15.310271e-3 -67.853949e-3 rpy=-1.860531 1.308458 -1.896217 -> xyz=-9.653191e-3 -15.310271e-3 -67.853949e-3  rpy= -1.2810616535897934 1.308458 -1.2453756535897933 
- joint pinky_q1: origin xyz=49.521293e-3 -11.004583e-3 -63.029065e-3 rpy=-1.765110 1.322220 -1.658383 -> xyz=-49.521293e-3 -11.004583e-3 -63.029065e-3  rpy= -1.3764826535897934 1.32222 -1.4832096535897932 
- joint ring_q1: origin xyz=29.954260e-3 -14.212492e-3 -67.286105e-3 rpy=-1.716598 1.321452 -1.675862 -> xyz=-29.95426e-3 -14.212492e-3 -67.286105e-3  rpy= -1.424994653589793 1.321452 -1.4657306535897934 
- joint thumb_q1: origin xyz=0 0 0 rpy=0 0 3.330437 -> xyz= 0.0 0.0 0.0  rpy= 3.141592653589793 -0.0 -0.18884434641020664 
- joint thumb_q2: origin xyz=27.8283501e-3 0 -14.7507000e-3 rpy=4.450589592585541 0 0 -> xyz=27.8283501e-3 0 14.7507e-3  rpy=1.832595714594045 -0.0 5.366520605522463e-18 
- joint wrist2thumb: origin xyz=24.0476665e-3 3.78124745e-3 32.32964923e-3 rpy=3.14148426 0.08848813 3.14036612 -> xyz=-24.0476665e-3 3.78124745e-3 32.32964923e-3 rpy=3.14148426 -0.08848813 -3.14036612
