Commit message: [update] update ability hand and assembly

File: robots/assembly/xarm7_ability/xarm7_ability_left_hand.urdf (robot description, URDF)
Before this commit: robot ability_hand, 18 links, 17 joints
Links:
- removed link base_link
- removed link index_tip
- removed link middle_tip
- removed link pinky_tip
- removed link ring_tip
- removed link thumb_tip
- added link ee_link
- added link index_anchor
- added link link1, mass 2.382; collision mesh filename=../../arms/xarm7/meshes/collision/link1.obj; visual mesh filename=../../arms/xarm7/meshes/visual/link1.glb
- added link link2, mass 1.869; collision mesh filename=../../arms/xarm7/meshes/collision/link2.obj; visual mesh filename=../../arms/xarm7/meshes/visual/link2.glb
- added link link3, mass 1.6383; collision mesh filename=../../arms/xarm7/meshes/collision/link3.obj; visual mesh filename=../../arms/xarm7/meshes/visual/link3.glb
- added link link4, mass 1.7269; collision mesh filename=../../arms/xarm7/meshes/collision/link4.obj; visual mesh filename=../../arms/xarm7/meshes/visual/link4.glb
- added link link5, mass 1.3203; collision mesh filename=../../arms/xarm7/meshes/collision/link5.obj; visual mesh filename=../../arms/xarm7/meshes/visual/link5.glb
- added link link6, mass 1.325; collision mesh filename=../../arms/xarm7/meshes/collision/link6.obj; visual mesh filename=../../arms/xarm7/meshes/visual/link6.glb
- added link link7, mass 0.17; collision cylinder length=0.018 radius=0.0365; collision mesh filename=../../arms/xarm7/meshes/collision/link7.obj
- added link link_base, mass 0.88556; collision mesh filename=../../arms/xarm7/meshes/collision/link_base.obj; visual mesh filename=../../arms/xarm7/meshes/visual/link_base.glb
- added link middle_anchor
- added link pinky_anchor
- added link ring_anchor
- added link thumb_anchor
- link base: geometry collision mesh filename=../../hands/ability_hand/meshes/collision/wristmesh_C.obj; visual mesh filename=../../hands/ability_hand/meshes/visual/wristmesh.glb
- link index_L1: geometry collision box size=0.012 0.012 0.002; collision box size=0.012 0.012 0.002
- link index_L2: geometry collision mesh filename=../../hands/ability_hand/meshes/collision/idx-F2_C.obj; collision sphere radius=0.007
- link middle_L1: geometry collision box size=0.012 0.012 0.002; collision box size=0.012 0.012 0.002
- link middle_L2: geometry collision mesh filename=../../hands/ability_hand/meshes/collision/idx-F2_C.obj; collision sphere radius=0.007
- link pinky_L1: geometry collision box size=0.012 0.012 0.002; collision box size=0.012 0.012 0.002
- link pinky_L2: geometry collision mesh filename=../../hands/ability_hand/meshes/collision/idx-F2_C.obj; collision sphere radius=0.007
- link ring_L1: geometry collision box size=0.012 0.012 0.002; collision box size=0.012 0.012 0.002
- link ring_L2: geometry collision mesh filename=../../hands/ability_hand/meshes/collision/idx-F2_C.obj; collision sphere radius=0.007
- link thumb_L1: geometry collision mesh filename=../../hands/ability_hand/meshes/collision/thumb-F1_C.obj; visual mesh filename=../../hands/ability_hand/meshes/visual/thumb-F1.glb
- link thumb_L2: geometry collision mesh filename=../../hands/ability_hand/meshes/collision/thumb-F2_C.obj; visual mesh filename=../../hands/ability_hand/meshes/visual/thumb-F2.glb
- link thumb_base: geometry collision mesh filename=../../hands/ability_hand/meshes/collision/FB_palm_ref.obj; visual mesh filename=../../hands/ability_hand/meshes/visual/FB_palm_ref.glb
Joints:
- removed joint base_joint
- removed joint index_tip_joint
- removed joint middle_tip_joint
- removed joint pinky_tip_joint
- removed joint ring_tip_joint
- removed joint thumb_tip_joint
- added joint ee_joint: type fixed, parent base, child ee_link, origin xyz=0 0 0 rpy=0 0 1.57079
- added joint idx_anchor: type fixed, parent index_L2, child index_anchor, origin xyz=31.5541e-3  -10.44e-3 0.14e-3 rpy=0 0 0
- added joint joint1: type revolute, parent link_base, child link1, origin xyz=0 0 0.267 rpy=0 0 0, axis 0 0 1, limit lower=-6.28318530718 upper=6.28318530718 effort=50 velocity=3.14
- added joint joint2: type revolute, parent link1, child link2, origin xyz=0 0 0 rpy=-1.5708 0 0, axis 0 0 1, limit lower=-2.059 upper=2.0944 effort=50 velocity=3.14
- added joint joint3: type revolute, parent link2, child link3, origin xyz=0 -0.293 0 rpy=1.5708 0 0, axis 0 0 1, limit lower=-6.28318530718 upper=6.28318530718 effort=30 velocity=3.14
- added joint joint4: type revolute, parent link3, child link4, origin xyz=0.0525 0 0 rpy=1.5708 0 0, axis 0 0 1, limit lower=-0.19198 upper=3.927 effort=30 velocity=3.14
- added joint joint5: type revolute, parent link4, child link5, origin xyz=0.0775 -0.3425 0 rpy=1.5708 0 0, axis 0 0 1, limit lower=-6.28318530718 upper=6.28318530718 effort=30 velocity=3.14
- added joint joint6: type revolute, parent link5, child link6, origin xyz=0 0 0 rpy=1.5708 0 0, axis 0 0 1, limit lower=-1.69297 upper=3.14159265359 effort=20 velocity=3.14
- added joint joint7: type revolute, parent link6, child link7, origin xyz=0.076 0.097 0 rpy=-1.5708 0 0, axis 0 0 1, limit lower=-6.28318530718 upper=6.28318530718 effort=20 velocity=3.14
- added joint joint_eef: type fixed, parent link7, child base, origin xyz=0 0 0.018 rpy=0 0 -1.57079
- added joint mid_anchor: type fixed, parent middle_L2, child middle_anchor, origin xyz=31.5541e-3  -10.44e-3 0.14e-3 rpy=0 0 0
- added joint pnky_anchor: type fixed, parent pinky_L2, child pinky_anchor, origin xyz=31.5541e-3  -10.44e-3 0.14e-3 rpy=0 0 0
- added joint rng_anchor: type fixed, parent ring_L2, child ring_anchor, origin xyz=31.5541e-3  -10.44e-3 0.14e-3 rpy=0 0 0
- added joint thmb_anchor: type fixed, parent thumb_L2, child thumb_anchor, origin xyz=52.0012259e-3  28.0086971e-3 -.884835778e-3 rpy=0 0 0

File: robots/assembly/xarm7_ability/xarm7_ability_right_hand.urdf (robot description, URDF)
Before this commit: robot xarm7, 25 links, 24 joints
Links:
- added link ee_link
Joints:
- added joint ee_joint: type fixed, parent base, child ee_link, origin xyz=0 0 0 rpy=0 0 1.57079
- joint index_q2: mimic joint=index_q1 multiplier=1.05851325 offset=0.72349796 -> (none)
- joint middle_q2: mimic joint=middle_q1 multiplier=1.05851325 offset=0.72349796 -> (none)
- joint pinky_q2: mimic joint=pinky_q1 multiplier=1.05851325 offset=0.72349796 -> (none)
- joint ring_q2: mimic joint=ring_q1 multiplier=1.05851325 offset=0.72349796 -> (none)

File: robots/hands/ability_hand/ability_hand_left.urdf (robot description, URDF)
Before this commit: robot ability_hand, 18 links, 17 joints
Joints:
- joint index_q2: mimic joint=index_q1 multiplier=1.05851325 offset=0.72349796 -> (none)
- joint middle_q2: mimic joint=middle_q1 multiplier=1.05851325 offset=0.72349796 -> (none)
- joint pinky_q2: mimic joint=pinky_q1 multiplier=1.05851325 offset=0.72349796 -> (none)
- joint ring_q2: mimic joint=ring_q1 multiplier=1.05851325 offset=0.72349796 -> (none)

File: robots/hands/ability_hand/ability_hand_right.urdf (robot description, URDF)
Before this commit: robot ability_hand, 18 links, 17 joints
Joints:
- joint index_q2: mimic joint=index_q1 multiplier=1.05851325 offset=0.72349796 -> (none)
- joint middle_q2: mimic joint=middle_q1 multiplier=1.05851325 offset=0.72349796 -> (none)
- joint pinky_q2: mimic joint=pinky_q1 multiplier=1.05851325 offset=0.72349796 -> (none)
- joint ring_q2: mimic joint=ring_q1 multiplier=1.05851325 offset=0.72349796 -> (none)

File: robots/hands/ability_hand/ability_hand_right_glb.urdf (robot description, URDF)
Before this commit: robot ability_hand, 18 links, 17 joints
Joints:
- joint index_q2: mimic joint=index_q1 multiplier=1.05851325 offset=0.72349796 -> (none)
- joint middle_q2: mimic joint=middle_q1 multiplier=1.05851325 offset=0.72349796 -> (none)
- joint pinky_q2: mimic joint=pinky_q1 multiplier=1.05851325 offset=0.72349796 -> (none)
- joint ring_q2: mimic joint=ring_q1 multiplier=1.05851325 offset=0.72349796 -> (none)

Commit message: [update] improve ability hand consistency

File: robots/assembly/xarm7_ability/xarm7_ability_left_hand.urdf (robot description, URDF)
Before this commit: robot xarm7, 26 links, 25 joints
Links:
- removed link index_anchor
- removed link middle_anchor
- removed link pinky_anchor
- removed link ring_anchor
- removed link thumb_anchor
- added link index_tip
- added link middle_tip
- added link pinky_tip
- added link ring_tip
- added link thumb_tip
- link index_L1: geometry collision box size=0.012 0.012 0.002; collision box size=0.012 0.012 0.002
Joints:
- removed joint idx_anchor
- removed joint mid_anchor
- removed joint pnky_anchor
- removed joint rng_anchor
- removed joint thmb_anchor
- added joint index_tip_joint: type fixed, parent index_L2, child index_tip, origin xyz=0.035  -0.018 0 rpy=0 0 0
- added joint middle_tip_joint: type fixed, parent middle_L2, child middle_tip, origin xyz=0.035  -0.018 0 rpy=0 0 0
- added joint pinky_tip_joint: type fixed, parent pinky_L2, child pinky_tip, origin xyz=0.035  -0.018 0 rpy=0 0 0
- added joint ring_tip_joint: type fixed, parent ring_L2, child ring_tip, origin xyz=0.035  -0.018 0 rpy=0 0 0
- added joint thumb_tip_joint: type fixed, parent thumb_L2, child thumb_tip, origin xyz=0.065 0.016 0 rpy=0 0 0

File: robots/assembly/xarm7_ability/xarm7_ability_right_hand.urdf (robot description, URDF)
Before this commit: robot xarm7, 26 links, 25 joints
Links:
- link thumb_base: mass 0.200 -> 0.400
Joints:
- joint index_q1: origin xyz= 9.49e-3 -13.04e-3 -62.95e-3  rpy= -1.1595426535897932 1.284473 -1.0510016535897932  -> xyz=9.49e-3 -13.04e-3 -62.95e-3  rpy= -1.1595426535897932 1.284473 -1.0510016535897932 
- joint middle_q1: origin xyz= -9.653191e-3 -15.310271e-3 -67.853949e-3  rpy= -1.2810616535897934 1.308458 -1.2453756535897933  -> xyz=-9.653191e-3 -15.310271e-3 -67.853949e-3  rpy= -1.2810616535897934 1.308458 -1.2453756535897933 
- joint pinky_q1: origin xyz= -49.521293e-3 -11.004583e-3 -63.029065e-3  rpy= -1.3764826535897934 1.32222 -1.4832096535897932  -> xyz=-49.521293e-3 -11.004583e-3 -63.029065e-3  rpy= -1.3764826535897934 1.32222 -1.4832096535897932 
- joint ring_q1: origin xyz= -29.95426e-3 -14.212492e-3 -67.286105e-3  rpy= -1.424994653589793 1.321452 -1.4657306535897934  -> xyz=-29.95426e-3 -14.212492e-3 -67.286105e-3  rpy= -1.424994653589793 1.321452 -1.4657306535897934 
- joint thumb_q2: origin xyz= 27.8283501e-3 1.7436510745838653e-19 14.7507e-3  rpy= 1.832595714594045 -0.0 5.366520605522463e-18  -> xyz=27.8283501e-3 0 14.7507e-3  rpy=1.832595714594045 -0.0 5.366520605522463e-18 

Commit message: [update] update ability hand to include mimic joint definition

File: robots/assembly/xarm7_ability/xarm7_ability_left_hand.urdf (robot description, URDF)
Before this commit: robot xarm7, 26 links, 25 joints
Joints:
- joint index_q2: mimic (none) -> joint=index_q1 multiplier=1.05851325 offset=0.72349796
- joint middle_q2: mimic (none) -> joint=middle_q1 multiplier=1.05851325 offset=0.72349796
- joint pinky_q2: mimic (none) -> joint=pinky_q1 multiplier=1.05851325 offset=0.72349796
- joint ring_q2: mimic (none) -> joint=ring_q1 multiplier=1.05851325 offset=0.72349796

File: robots/assembly/xarm7_ability/xarm7_ability_left_hand_glb.urdf (robot description, URDF)
Before this commit: robot xarm7, 26 links, 25 joints
Joints:
- joint index_q2: mimic (none) -> joint=index_q1 multiplier=1.05851325 offset=0.72349796
- joint middle_q2: mimic (none) -> joint=middle_q1 multiplier=1.05851325 offset=0.72349796
- joint pinky_q2: mimic (none) -> joint=pinky_q1 multiplier=1.05851325 offset=0.72349796
- joint ring_q2: mimic (none) -> joint=ring_q1 multiplier=1.05851325 offset=0.72349796

File: robots/assembly/xarm7_ability/xarm7_ability_right_hand.urdf (robot description, URDF)
Before this commit: robot xarm7, 26 links, 25 joints
Joints:
- joint index_q2: mimic (none) -> joint=index_q1 multiplier=1.05851325 offset=0.72349796
- joint middle_q2: mimic (none) -> joint=middle_q1 multiplier=1.05851325 offset=0.72349796
- joint pinky_q2: mimic (none) -> joint=pinky_q1 multiplier=1.05851325 offset=0.72349796
- joint ring_q2: mimic (none) -> joint=ring_q1 multiplier=1.05851325 offset=0.72349796

File: robots/assembly/xarm7_ability/xarm7_ability_right_hand_glb.urdf (robot description, URDF)
Before this commit: robot xarm7, 26 links, 25 joints
Joints:
- joint index_q2: mimic (none) -> joint=index_q1 multiplier=1.05851325 offset=0.72349796
- joint middle_q2: mimic (none) -> joint=middle_q1 multiplier=1.05851325 offset=0.72349796
- joint pinky_q2: mimic (none) -> joint=pinky_q1 multiplier=1.05851325 offset=0.72349796
- joint ring_q2: mimic (none) -> joint=ring_q1 multiplier=1.05851325 offset=0.72349796

File: robots/hands/ability_hand/ability_hand_left.urdf (robot description, URDF)
Before this commit: robot ability_hand, 18 links, 17 joints
Joints:
- joint index_q2: mimic (none) -> joint=index_q1 multiplier=1.05851325 offset=0.72349796
- joint middle_q2: mimic (none) -> joint=middle_q1 multiplier=1.05851325 offset=0.72349796
- joint pinky_q2: mimic (none) -> joint=pinky_q1 multiplier=1.05851325 offset=0.72349796
- joint ring_q2: mimic (none) -> joint=ring_q1 multiplier=1.05851325 offset=0.72349796

File: robots/hands/ability_hand/ability_hand_left_glb.urdf (robot description, URDF)
Before this commit: robot ability_hand, 18 links, 17 joints
Joints:
- joint index_q2: mimic (none) -> joint=index_q1 multiplier=1.05851325 offset=0.72349796
- joint middle_q2: mimic (none) -> joint=middle_q1 multiplier=1.05851325 offset=0.72349796
- joint pinky_q2: mimic (none) -> joint=pinky_q1 multiplier=1.05851325 offset=0.72349796
- joint ring_q2: mimic (none) -> joint=ring_q1 multiplier=1.05851325 offset=0.72349796

File: robots/hands/ability_hand/ability_hand_right.urdf (robot description, URDF)
Before this commit: robot ability_hand, 18 links, 17 joints
Joints:
- joint index_q2: mimic (none) -> joint=index_q1 multiplier=1.05851325 offset=0.72349796
- joint middle_q2: mimic (none) -> joint=middle_q1 multiplier=1.05851325 offset=0.72349796
- joint pinky_q2: mimic (none) -> joint=pinky_q1 multiplier=1.05851325 offset=0.72349796
- joint ring_q2: mimic (none) -> joint=ring_q1 multiplier=1.05851325 offset=0.72349796

File: robots/hands/ability_hand/ability_hand_right_glb.urdf (robot description, URDF)
Before this commit: robot ability_hand, 18 links, 17 joints
Joints:
- joint index_q2: mimic (none) -> joint=index_q1 multiplier=1.05851325 offset=0.72349796
- joint middle_q2: mimic (none) -> joint=middle_q1 multiplier=1.05851325 offset=0.72349796
- joint pinky_q2: mimic (none) -> joint=pinky_q1 multiplier=1.05851325 offset=0.72349796
- joint ring_q2: mimic (none) -> joint=ring_q1 multiplier=1.05851325 offset=0.72349796
