Commit message: [update] add xarm7 none glb version

File: robots/arms/xarm7/xarm7_glb.urdf (robot description, URDF)
Before this commit: robot xarm7, 9 links, 8 joints
Links:
- link link1: geometry collision mesh filename=meshes/collision/link1.obj; visual mesh filename=meshes/visual/link1.glb
- link link2: geometry collision mesh filename=meshes/collision/link2.obj; visual mesh filename=meshes/visual/link2.glb
- link link3: geometry collision mesh filename=meshes/collision/link3.obj; visual mesh filename=meshes/visual/link3.glb
- link link4: geometry collision mesh filename=meshes/collision/link4.obj; visual mesh filename=meshes/visual/link4.glb
- link link5: geometry collision mesh filename=meshes/collision/link5.obj; visual mesh filename=meshes/visual/link5.glb
- link link6: geometry collision mesh filename=meshes/collision/link6.obj; visual mesh filename=meshes/visual/link6.glb
- link link7: geometry collision mesh filename=meshes/collision/link7.obj; visual mesh filename=meshes/visual/link7.glb
- link link_base: geometry collision mesh filename=meshes/collision/link_base.obj; visual mesh filename=meshes/visual/link_base.glb
