Commit message: [fix] fix shadow hand joint and link share the same name

File: robots/hands/shadow_hand/shadow_hand_left.urdf (robot description, URDF)
Before this commit: robot shadow_left, 33 links, 32 joints
Joints:
- removed joint thtip
- added joint THtip: type fixed, parent thdistal, child thtip, origin xyz=0 0 0.0275 rpy=0 0 0

File: robots/hands/shadow_hand/shadow_hand_left_glb.urdf (robot description, URDF)
Before this commit: robot shadow_left, 33 links, 32 joints
Joints:
- removed joint thtip
- added joint THtip: type fixed, parent thdistal, child thtip, origin xyz=0 0 0.0275 rpy=0 0 0

File: robots/hands/shadow_hand/shadow_hand_right.urdf (robot description, URDF)
Before this commit: robot shadow_right, 33 links, 32 joints
Joints:
- removed joint thtip
- added joint THtip: type fixed, parent thdistal, child thtip, origin xyz=0 0 0.0275 rpy=0 0 0

File: robots/hands/shadow_hand/shadow_hand_right_glb.urdf (robot description, URDF)
Before this commit: robot shadow_right, 33 links, 32 joints
Joints:
- removed joint thtip
- added joint THtip: type fixed, parent thdistal, child thtip, origin xyz=0 0 0.0275 rpy=0 0 0
