Commit message: [update] update ur5 ee definition

File: robots/arms/ur5e/ur5e.urdf (robot description, URDF)
Before this commit: robot ur5e_robot, 11 links, 10 joints
Links:
- removed link flange
- removed link tool0
- added link ee_link
Joints:
- removed joint flange-tool0
- joint wrist_3-flange: child flange -> ee_link

File: robots/arms/ur5e/ur5e_glb.urdf (robot description, URDF)
Before this commit: robot ur5e_robot, 11 links, 10 joints
Links:
- removed link flange
- removed link tool0
- added link ee_link
Joints:
- removed joint flange-tool0
- joint wrist_3-flange: child flange -> ee_link
