Commit message: [update] clean up leap hand values

File: robots/hands/leap_hand/leap_hand_right.urdf (robot description, URDF)
Before this commit: robot onshape, 18 links, 17 joints
Joints:
- joint 0: origin xyz=-0.012200000000000007713 0.038099999999999994982 0.014500000000000000736 rpy=-1.570796326794896558 -1.0065212660796336576e-15 1.5707963267948943376 -> xyz=-0.0122 0.03810 0.01450 rpy=-1.57079 0 1.57079
- joint 1: origin xyz=-0.0070952496528625457958 0.023057756134899472233 -0.01872240357846021927 rpy=1.5707963267948950037 1.5707963267948945596 0 -> xyz=-0.0070 0.0230 -0.0187 rpy=1.57079 1.57079 0
- joint 10: origin xyz=0.014999999999999971689 0.014299999999999951639 -0.012999999999999959505 rpy=1.5707963267948958919 -1.570796326794896336 0 -> xyz=0.015 0.0143 -0.013 rpy=1.57079 -1.57079 0
- joint 11: origin xyz=9.7144514654701197287e-17 -0.036099999999999868305 0.00020000000000007511769 rpy=4.5935029425113685044e-17 -2.8730071914463799514e-16 1.5565411607615035382e-32 -> xyz=0 -0.03609 0.0002 rpy=0 0 0
- joint 12: origin xyz=-0.069395249652862533996 -0.0012422438651005258004 -0.021622403578460215601 rpy=-8.2381766464939424156e-17 1.5707963267948956698 0 -> xyz=-0.0693 -0.0012 -0.0216 rpy=0 1.57079 0
- joint 13: origin xyz=-2.7755575615628913511e-17 0.014300000000000005415 -0.013000000000000011546 rpy=1.5707963267948958919 -1.570796326794896336 0 -> xyz=0 0.0143 -0.013 rpy=1.57079 -1.57079 0
- joint 14: origin xyz=0 0.014499999999999966041 -0.017000000000000053263 rpy=-1.570796326794896558 1.6050198443300131245e-46 -1.9721522630516624601e-31 -> xyz=0 0.0145 -0.017 rpy=-1.57079 0 0
- joint 15: origin xyz=-1.249000902703301108e-16 0.046599999999999863753 0.00019999999999997710581 rpy=1.5063958491491781023e-44 5.4234187233935260503e-31 3.141592653589793116 -> xyz=0 0.0466 0.0002 rpy=0 0 3.14159
- joint 2: origin xyz=0.01499999999999996822 0.014299999999999904801 -0.012999999999999824196 rpy=1.5707963267948958919 -1.570796326794896336 0 -> xyz=0.015 0.0143 -0.013 rpy=1.57079 -1.57079 0
- joint 3: origin xyz=-4.0880582495572692636e-09 -0.036100004210367367397 0.00020000000000007858714 rpy=0 0 0 -> xyz=0 -0.0361 0.0002 rpy=0 0 0
- joint 4: origin xyz=-0.012200000000000019856 0.038099999999999981104 0.01450000000000000594 rpy=-1.570796326794896558 -1.0065212760057939085e-15 1.5707963267948943376 -> xyz=-0.0122 0.0381 0.0145 rpy=-1.57079 0 1.57079
- joint 5: origin xyz=-0.0070952496528625388569 -0.022392243865100525113 -0.018722403578460229678 rpy=1.570796326794896558 1.570796326794896558 0 -> xyz=-0.0071 -0.0224 -0.0187 rpy=1.57079 1.57079 0
- joint 6: origin xyz=0.014999999999999975159 0.014300000000000000211 -0.013000000000000018485 rpy=1.5707963267948958919 -1.570796326794896336 0 -> xyz=0.015 0.0143 -0.013 rpy=1.57079 -1.57079 0
- joint 7: origin xyz=1.0061396160665481148e-16 -0.036099999999999854428 0.00020000000000007858714 rpy=4.5935029425113654229e-17 -2.8730071914463794583e-16 1.4408183216511868558e-31 -> xyz=0 -0.0361 0.0002 rpy=0 0 0
- joint 8: origin xyz=-0.012200000000000004244 0.038100000000000001921 0.014499999999999999001 rpy=-1.570796326794896558 -1.0065212660796360242e-15 1.5707963267948943376 -> xyz=-0.0122 0.0381 0.0145 rpy=-1.57079 0 1.57079
- joint 9: origin xyz=-0.0070952454426398371343 -0.067842243865100515521 -0.018722407666402932774 rpy=1.5707963267948950037 1.5707963267948945596 0 -> xyz=-0.00709 -0.0678 -0.0187 rpy=1.57079 1.57079 0

File: robots/hands/leap_hand/leap_hand_right_glb.urdf (robot description, URDF)
Before this commit: robot onshape, 18 links, 17 joints
Joints:
- joint 0: origin xyz=-0.012200000000000007713 0.038099999999999994982 0.014500000000000000736 rpy=-1.570796326794896558 -1.0065212660796336576e-15 1.5707963267948943376 -> xyz=-0.0122 0.03810 0.01450 rpy=-1.57079 0 1.57079
- joint 1: origin xyz=-0.0070952496528625457958 0.023057756134899472233 -0.01872240357846021927 rpy=1.5707963267948950037 1.5707963267948945596 0 -> xyz=-0.0070 0.0230 -0.0187 rpy=1.57079 1.57079 0
- joint 10: origin xyz=0.014999999999999971689 0.014299999999999951639 -0.012999999999999959505 rpy=1.5707963267948958919 -1.570796326794896336 0 -> xyz=0.015 0.0143 -0.013 rpy=1.57079 -1.57079 0
- joint 11: origin xyz=9.7144514654701197287e-17 -0.036099999999999868305 0.00020000000000007511769 rpy=4.5935029425113685044e-17 -2.8730071914463799514e-16 1.5565411607615035382e-32 -> xyz=0 -0.03609 0.0002 rpy=0 0 0
- joint 12: origin xyz=-0.069395249652862533996 -0.0012422438651005258004 -0.021622403578460215601 rpy=-8.2381766464939424156e-17 1.5707963267948956698 0 -> xyz=-0.0693 -0.0012 -0.0216 rpy=0 1.57079 0
- joint 13: origin xyz=-2.7755575615628913511e-17 0.014300000000000005415 -0.013000000000000011546 rpy=1.5707963267948958919 -1.570796326794896336 0 -> xyz=0 0.0143 -0.013 rpy=1.57079 -1.57079 0
- joint 14: origin xyz=0 0.014499999999999966041 -0.017000000000000053263 rpy=-1.570796326794896558 1.6050198443300131245e-46 -1.9721522630516624601e-31 -> xyz=0 0.0145 -0.017 rpy=-1.57079 0 0
- joint 15: origin xyz=-1.249000902703301108e-16 0.046599999999999863753 0.00019999999999997710581 rpy=1.5063958491491781023e-44 5.4234187233935260503e-31 3.141592653589793116 -> xyz=0 0.0466 0.0002 rpy=0 0 3.14159
- joint 2: origin xyz=0.01499999999999996822 0.014299999999999904801 -0.012999999999999824196 rpy=1.5707963267948958919 -1.570796326794896336 0 -> xyz=0.015 0.0143 -0.013 rpy=1.57079 -1.57079 0
- joint 3: origin xyz=-4.0880582495572692636e-09 -0.036100004210367367397 0.00020000000000007858714 rpy=0 0 0 -> xyz=0 -0.0361 0.0002 rpy=0 0 0
- joint 4: origin xyz=-0.012200000000000019856 0.038099999999999981104 0.01450000000000000594 rpy=-1.570796326794896558 -1.0065212760057939085e-15 1.5707963267948943376 -> xyz=-0.0122 0.0381 0.0145 rpy=-1.57079 0 1.57079
- joint 5: origin xyz=-0.0070952496528625388569 -0.022392243865100525113 -0.018722403578460229678 rpy=1.570796326794896558 1.570796326794896558 0 -> xyz=-0.0071 -0.0224 -0.0187 rpy=1.57079 1.57079 0
- joint 6: origin xyz=0.014999999999999975159 0.014300000000000000211 -0.013000000000000018485 rpy=1.5707963267948958919 -1.570796326794896336 0 -> xyz=0.015 0.0143 -0.013 rpy=1.57079 -1.57079 0
- joint 7: origin xyz=1.0061396160665481148e-16 -0.036099999999999854428 0.00020000000000007858714 rpy=4.5935029425113654229e-17 -2.8730071914463794583e-16 1.4408183216511868558e-31 -> xyz=0 -0.0361 0.0002 rpy=0 0 0
- joint 8: origin xyz=-0.012200000000000004244 0.038100000000000001921 0.014499999999999999001 rpy=-1.570796326794896558 -1.0065212660796360242e-15 1.5707963267948943376 -> xyz=-0.0122 0.0381 0.0145 rpy=-1.57079 0 1.57079
- joint 9: origin xyz=-0.0070952454426398371343 -0.067842243865100515521 -0.018722407666402932774 rpy=1.5707963267948950037 1.5707963267948945596 0 -> xyz=-0.00709 -0.0678 -0.0187 rpy=1.57079 1.57079 0

Commit message: [update] leap hand add virtual finger tip frame

File: robots/hands/leap_hand/leap_hand_right.urdf (robot description, URDF)
Before this commit: robot onshape, 18 links, 17 joints
Links:
- added link index_tip_head
- added link middle_tip_head
- added link ring_tip_head
- added link thumb_tip_head
Joints:
- added joint index_tip: type fixed, parent fingertip, child index_tip_head, origin xyz=0 -0.048 0.015 rpy=0 0 0
- added joint middle_tip: type fixed, parent fingertip_2, child middle_tip_head, origin xyz=0 -0.048 0.015 rpy=0 0 0
- added joint ring_tip: type fixed, parent fingertip_3, child ring_tip_head, origin xyz=0 -0.048 0.015 rpy=0 0 0
- added joint thumb_tip: type fixed, parent thumb_fingertip, child thumb_tip_head, origin xyz=0 -0.06 -0.015 rpy=0 0 0

Commit message: [add] add leap hand left and make left and right more consistent

File: robots/hands/leap_hand/leap_hand_right.urdf (robot description, URDF)
Before this commit: robot leap_right, 22 links, 21 joints
Links:
- removed link pip_4
- added link thumb_temp_base, mass 0.032; collision box size=0.034 0.026 0.022; visual mesh filename=meshes/visual/pip.obj
Joints:
- joint 12: child pip_4 -> thumb_temp_base
- joint 13: parent pip_4 -> thumb_temp_base

File: robots/hands/leap_hand/leap_hand_right_glb.urdf (robot description, URDF)
Before this commit: robot leap_right, 22 links, 21 joints
Links:
- removed link pip_4
- added link thumb_temp_base, mass 0.032; collision box size=0.034 0.026 0.022; visual mesh filename=meshes/visual/pip.glb
Joints:
- joint 12: child pip_4 -> thumb_temp_base
- joint 13: parent pip_4 -> thumb_temp_base
