Commit message: [add] add inspire hand fingertip

File: robots/hands/inspire_hand/inspire_hand_left.urdf (robot description, URDF)
Before this commit: robot inspire_hand_left, 14 links, 13 joints
Links:
- added link index_tip
- added link middle_tip
- added link pinky_tip
- added link ring_tip
- added link thumb_tip
Joints:
- added joint index_tip_joint: type fixed, parent index_intermediate, child index_tip, origin xyz=-0.0008 -0.045 -0.005 rpy=0 0 0
- added joint middle_tip_joint: type fixed, parent middle_intermediate, child middle_tip, origin xyz=-0.001 -0.048 -0.005 rpy=0 0 0
- added joint pinky_tip_joint: type fixed, parent pinky_intermediate, child pinky_tip, origin xyz=-0.0008 -0.037 -0.005 rpy=0 0 0
- added joint ring_tip_joint: type fixed, parent ring_intermediate, child ring_tip, origin xyz=-0.0008 -0.045 -0.005 rpy=0 0 0
- added joint thumb_tip_joint: type fixed, parent thumb_distal, child thumb_tip, origin xyz=0.0202 -0.0140 -0.006 rpy=0 0 0

File: robots/hands/inspire_hand/inspire_hand_right.urdf (robot description, URDF)
Before this commit: robot inspire_hand_right, 14 links, 13 joints
Links:
- added link index_tip
- added link middle_tip
- added link pinky_tip
- added link ring_tip
- added link thumb_tip
Joints:
- added joint index_tip_joint: type fixed, parent index_intermediate, child index_tip, origin xyz=-0.0008 0.045 -0.005 rpy=0 0 0
- added joint middle_tip_joint: type fixed, parent middle_intermediate, child middle_tip, origin xyz=-0.001 0.048 -0.005 rpy=0 0 0
- added joint pinky_tip_joint: type fixed, parent pinky_intermediate, child pinky_tip, origin xyz=-0.0008 0.037 -0.005 rpy=0 0 0
- added joint ring_tip_joint: type fixed, parent ring_intermediate, child ring_tip, origin xyz=-0.0008 0.045 -0.005 rpy=0 0 0
- added joint thumb_tip_joint: type fixed, parent thumb_distal, child thumb_tip, origin xyz=0.0202 0.0140 -0.006 rpy=0 0 0

Commit message: [update] update inspire hand joint limit and mimic property

File: robots/hands/inspire_hand/inspire_hand_left.urdf (robot description, URDF)
Before this commit: robot inspire_hand_left, 19 links, 18 joints
Joints:
- joint index_intermediate_joint: limit lower=0 upper=1.7 effort=1 velocity=0.5 -> lower=0 upper=1.6 effort=1 velocity=0.5
- joint index_proximal_joint: limit lower=0 upper=1.7 effort=1 velocity=0.5 -> lower=0 upper=1.45 effort=1 velocity=0.5
- joint middle_intermediate_joint: limit lower=0 upper=1.7 effort=1 velocity=0.5 -> lower=0 upper=1.6 effort=1 velocity=0.5
- joint middle_proximal_joint: limit lower=0 upper=1.7 effort=1 velocity=0.5 -> lower=0 upper=1.45 effort=1 velocity=0.5
- joint pinky_intermediate_joint: limit lower=0 upper=1.7 effort=1 velocity=0.5 -> lower=0 upper=1.6 effort=1 velocity=0.5
- joint pinky_proximal_joint: limit lower=0 upper=1.7 effort=1 velocity=0.5 -> lower=0 upper=1.45 effort=1 velocity=0.5
- joint ring_intermediate_joint: limit lower=0 upper=1.7 effort=1 velocity=0.5 -> lower=0 upper=1.6 effort=1 velocity=0.5
- joint ring_proximal_joint: limit lower=0 upper=1.7 effort=1 velocity=0.5 -> lower=0 upper=1.45 effort=1 velocity=0.5
- joint thumb_distal_joint: limit lower=0 upper=1.2 effort=1 velocity=0.5 -> lower=0 upper=0.4 effort=1 velocity=0.5; mimic joint=thumb_proximal_pitch_joint multiplier=2.4 offset=0 -> joint=thumb_proximal_pitch_joint multiplier=0.667 offset=0
- joint thumb_intermediate_joint: mimic joint=thumb_proximal_pitch_joint multiplier=1.6 offset=0 -> joint=thumb_proximal_pitch_joint multiplier=1.334 offset=0
- joint thumb_proximal_pitch_joint: limit lower=-0.1 upper=0.6 effort=1 velocity=0.5 -> lower=0 upper=0.6 effort=1 velocity=0.5
- joint thumb_proximal_yaw_joint: limit lower=-0.1 upper=1.30 effort=1 velocity=0.5 -> lower=0 upper=1.30 effort=1 velocity=0.5

File: robots/hands/inspire_hand/inspire_hand_right.urdf (robot description, URDF)
Before this commit: robot inspire_hand_right, 19 links, 18 joints
Joints:
- joint index_intermediate_joint: limit lower=0 upper=1.7 effort=1 velocity=0.5 -> lower=0 upper=1.6 effort=1 velocity=0.5
- joint index_proximal_joint: limit lower=0 upper=1.7 effort=1 velocity=0.5 -> lower=0 upper=1.45 effort=1 velocity=0.5
- joint middle_intermediate_joint: limit lower=0 upper=1.7 effort=1 velocity=0.5 -> lower=0 upper=1.6 effort=1 velocity=0.5
- joint middle_proximal_joint: limit lower=0 upper=1.7 effort=1 velocity=0.5 -> lower=0 upper=1.45 effort=1 velocity=0.5
- joint pinky_intermediate_joint: limit lower=0 upper=1.7 effort=1 velocity=0.5 -> lower=0 upper=1.6 effort=1 velocity=0.5
- joint pinky_proximal_joint: limit lower=0 upper=1.7 effort=1 velocity=0.5 -> lower=0 upper=1.45 effort=1 velocity=0.5
- joint ring_intermediate_joint: limit lower=0 upper=1.7 effort=1 velocity=0.5 -> lower=0 upper=1.6 effort=1 velocity=0.5
- joint ring_proximal_joint: limit lower=0 upper=1.7 effort=1 velocity=0.5 -> lower=0 upper=1.45 effort=1 velocity=0.5
- joint thumb_distal_joint: limit lower=0 upper=1.2 effort=1 velocity=0.5 -> lower=0 upper=0.4 effort=1 velocity=0.5; mimic joint=thumb_proximal_pitch_joint multiplier=2.4 offset=0 -> joint=thumb_proximal_pitch_joint multiplier=0.667 offset=0
- joint thumb_intermediate_joint: mimic joint=thumb_proximal_pitch_joint multiplier=1.6 offset=0 -> joint=thumb_proximal_pitch_joint multiplier=1.334 offset=0
- joint thumb_proximal_pitch_joint: limit lower=-0.1 upper=0.6 effort=1 velocity=0.5 -> lower=0 upper=0.6 effort=1 velocity=0.5
- joint thumb_proximal_yaw_joint: limit lower=-0.1 upper=1.3 effort=1 velocity=0.5 -> lower=0.0 upper=1.3 effort=1 velocity=0.5

Commit message: [update] update inspire hand mimic property based on test data linfit

File: robots/hands/inspire_hand/inspire_hand_left.urdf (robot description, URDF)
Before this commit: robot inspire_hand_left, 19 links, 18 joints
Joints:
- joint index_intermediate_joint: limit lower=0 upper=1.6 effort=1 velocity=0.5 -> lower=-0.04545 upper=1.56 effort=1 velocity=0.5; mimic joint=index_proximal_joint multiplier=1 offset=0 -> joint=index_proximal_joint multiplier=1.06399 offset=-0.04545
- joint index_proximal_joint: limit lower=0 upper=1.45 effort=1 velocity=0.5 -> lower=0 upper=1.47 effort=1 velocity=0.5
- joint middle_intermediate_joint: limit lower=0 upper=1.6 effort=1 velocity=0.5 -> lower=-0.04545 upper=1.56 effort=1 velocity=0.5; mimic joint=middle_proximal_joint multiplier=1 offset=0 -> joint=middle_proximal_joint multiplier=1.06399 offset=-0.04545
- joint middle_proximal_joint: limit lower=0 upper=1.45 effort=1 velocity=0.5 -> lower=0 upper=1.47 effort=1 velocity=0.5
- joint pinky_intermediate_joint: limit lower=0 upper=1.6 effort=1 velocity=0.5 -> lower=-0.04545 upper=1.56 effort=1 velocity=0.5; mimic joint=pinky_proximal_joint multiplier=1 offset=0 -> joint=pinky_proximal_joint multiplier=1.06399 offset=-0.04545
- joint pinky_proximal_joint: limit lower=0 upper=1.45 effort=1 velocity=0.5 -> lower=0 upper=1.47 effort=1 velocity=0.5
- joint ring_intermediate_joint: limit lower=0 upper=1.6 effort=1 velocity=0.5 -> lower=-0.04545 upper=1.56 effort=1 velocity=0.5; mimic joint=ring_proximal_joint multiplier=1 offset=0 -> joint=ring_proximal_joint multiplier=1.06399 offset=-0.04545
- joint ring_proximal_joint: limit lower=0 upper=1.45 effort=1 velocity=0.5 -> lower=0 upper=1.47 effort=1 velocity=0.5
- joint thumb_proximal_yaw_joint: limit lower=0 upper=1.30 effort=1 velocity=0.5 -> lower=0 upper=1.308 effort=1 velocity=0.5

File: robots/hands/inspire_hand/inspire_hand_right.urdf (robot description, URDF)
Before this commit: robot inspire_hand_right, 19 links, 18 joints
Joints:
- joint index_intermediate_joint: limit lower=0 upper=1.6 effort=1 velocity=0.5 -> lower=-0.04545 upper=1.56 effort=1 velocity=0.5; mimic joint=index_proximal_joint multiplier=1 offset=0 -> joint=index_proximal_joint multiplier=1.06399 offset=-0.04545
- joint index_proximal_joint: limit lower=0 upper=1.45 effort=1 velocity=0.5 -> lower=0 upper=1.47 effort=1 velocity=0.5
- joint middle_intermediate_joint: limit lower=0 upper=1.6 effort=1 velocity=0.5 -> lower=-0.04545 upper=1.56 effort=1 velocity=0.5; mimic joint=middle_proximal_joint multiplier=1 offset=0 -> joint=middle_proximal_joint multiplier=1.06399 offset=-0.04545
- joint middle_proximal_joint: limit lower=0 upper=1.45 effort=1 velocity=0.5 -> lower=0 upper=1.47 effort=1 velocity=0.5
- joint pinky_intermediate_joint: limit lower=0 upper=1.6 effort=1 velocity=0.5 -> lower=-0.04545 upper=1.56 effort=1 velocity=0.5; mimic joint=pinky_proximal_joint multiplier=1 offset=0 -> joint=pinky_proximal_joint multiplier=1.06399 offset=-0.04545
- joint pinky_proximal_joint: limit lower=0 upper=1.45 effort=1 velocity=0.5 -> lower=0 upper=1.47 effort=1 velocity=0.5
- joint ring_intermediate_joint: limit lower=0 upper=1.6 effort=1 velocity=0.5 -> lower=-0.04545 upper=1.56 effort=1 velocity=0.5; mimic joint=ring_proximal_joint multiplier=1 offset=0 -> joint=ring_proximal_joint multiplier=1.06399 offset=-0.04545
- joint ring_proximal_joint: limit lower=0 upper=1.45 effort=1 velocity=0.5 -> lower=0 upper=1.47 effort=1 velocity=0.5
- joint thumb_proximal_yaw_joint: limit lower=0.0 upper=1.3 effort=1 velocity=0.5 -> lower=0.0 upper=1.308 effort=1 velocity=0.5

Commit message: [update] update inspire hand visual model

File: robots/hands/inspire_hand/inspire_hand_left.urdf (robot description, URDF)
Before this commit: robot inspire_hand_left, 19 links, 18 joints
Links:
- link hand_base_link: geometry collision box size=0.0125 0.0111 0.0089; collision box size=0.0125 0.0111 0.0089
- link index_intermediate: geometry collision mesh filename=meshes/collision/left_index_intermediate.obj; visual mesh filename=meshes/visual/left_index_intermediate.glb
- link index_proximal: geometry collision mesh filename=meshes/collision/left_index_proximal.obj; visual mesh filename=meshes/visual/left_index_proximal.glb
- link middle_intermediate: geometry collision mesh filename=meshes/collision/left_middle_intermediate.obj; visual mesh filename=meshes/visual/left_middle_intermediate.glb
- link middle_proximal: geometry collision mesh filename=meshes/collision/left_index_proximal.obj; visual mesh filename=meshes/visual/left_index_proximal.glb
- link pinky_intermediate: geometry collision mesh filename=meshes/collision/left_pinky_intermediate.obj; visual mesh filename=meshes/visual/left_pinky_intermediate.glb
- link pinky_proximal: geometry collision mesh filename=meshes/collision/left_index_proximal.obj; visual mesh filename=meshes/visual/left_index_proximal.glb
- link ring_intermediate: geometry collision mesh filename=meshes/collision/left_index_intermediate.obj; visual mesh filename=meshes/visual/left_index_intermediate.glb
- link ring_proximal: geometry collision mesh filename=meshes/collision/left_index_proximal.obj; visual mesh filename=meshes/visual/left_index_proximal.glb
- link thumb_distal: geometry collision mesh filename=meshes/collision/left_thumb_distal.obj scale=1 1 1; visual mesh filename=meshes/visual/left_thumb_distal.glb
- link thumb_intermediate: geometry collision mesh filename=meshes/collision/left_thumb_intermediate.obj; visual mesh filename=meshes/visual/left_thumb_intermediate.glb
- link thumb_proximal: geometry collision mesh filename=meshes/collision/left_thumb_proximal.obj; visual mesh filename=meshes/visual/left_thumb_proximal.glb
- link thumb_proximal_base: geometry collision mesh filename=meshes/collision/left_thumb_proximal_base.obj; visual mesh filename=meshes/visual/left_thumb_proximal_base.glb
