Commit message: [update] update inspire hand left and right visual

File: robots/hands/inspire_hand/inspire_hand_right.urdf (robot description, URDF)
Before this commit: robot inspire_hand_right, 19 links, 18 joints
Links:
- link hand_base_link: geometry collision box size=0.0125 0.0111 0.0089; collision box size=0.0125 0.0111 0.0089
- link index_intermediate: geometry collision mesh filename=meshes/collision/right_index_intermediate.obj; visual mesh filename=meshes/visual/right_index_intermediate.glb
- link index_proximal: geometry collision mesh filename=meshes/collision/right_index_proximal.obj; visual mesh filename=meshes/visual/right_index_proximal.glb
- link middle_intermediate: geometry collision mesh filename=meshes/collision/right_middle_intermediate.obj; visual mesh filename=meshes/visual/right_middle_intermediate.glb
- link middle_proximal: geometry collision mesh filename=meshes/collision/right_index_proximal.obj; visual mesh filename=meshes/visual/right_index_proximal.glb
- link pinky_intermediate: geometry collision mesh filename=meshes/collision/right_pinky_intermediate.obj; visual mesh filename=meshes/visual/right_pinky_intermediate.glb
- link pinky_proximal: geometry collision mesh filename=meshes/collision/right_index_proximal.obj; visual mesh filename=meshes/visual/right_index_proximal.glb
- link ring_intermediate: geometry collision mesh filename=meshes/collision/right_index_intermediate.obj; visual mesh filename=meshes/visual/right_index_intermediate.glb
- link ring_proximal: geometry collision mesh filename=meshes/collision/right_index_proximal.obj; visual mesh filename=meshes/visual/right_index_proximal.glb
- link thumb_distal: geometry collision mesh filename=meshes/collision/right_thumb_distal.obj; visual mesh filename=meshes/visual/right_thumb_distal.glb
- link thumb_intermediate: geometry collision mesh filename=meshes/collision/right_thumb_intermediate.obj; visual mesh filename=meshes/visual/right_thumb_intermediate.glb
- link thumb_proximal: geometry collision mesh filename=meshes/collision/right_thumb_proximal.obj; visual mesh filename=meshes/visual/right_thumb_proximal.glb
- link thumb_proximal_base: geometry collision mesh filename=meshes/collision/right_thumb_proximal_base.obj; visual mesh filename=meshes/visual/right_thumb_proximal_base.glb
