Commit message: [update] update rm75 assembly for better consistency with the real one

File: robots/arms/rm75/rm75.urdf (robot description, URDF)
Before this commit: robot rm75, 10 links, 9 joints
Joints:
- joint joint_2: axis -1 0 0 -> 1 0 0
- joint joint_4: axis -1 0 0 -> 1 0 0
- joint joint_6: axis -1 0 0 -> 1 0 0
- joint world_joint: origin xyz=0 0 0 rpy=-1.57079 0 0 -> xyz=0.138497 0 0 rpy=-1.57079 1.57079 0

File: robots/arms/rm75/rm75_glb.urdf (robot description, URDF)
Before this commit: robot rm75, 10 links, 9 joints
Joints:
- joint joint_2: axis -1 0 0 -> 1 0 0
- joint joint_4: axis -1 0 0 -> 1 0 0
- joint joint_6: axis -1 0 0 -> 1 0 0
- joint world_joint: origin xyz=0 0 0 rpy=-1.57079 0 0 -> xyz=0.138497 0 0 rpy=-1.57079 1.57079 0
