Commit message: [update] update panda gripper visual & collision mesh

File: robots/hands/panda_gripper/panda_gripper_glb.urdf (robot description, URDF)
Before this commit: robot panda, 4 links, 3 joints
Links:
- link panda_hand: geometry collision box size=0.036 0.08 0.2; collision cylinder length=0.0077 radius=0.03

Commit message: [fix] fix convention consistency for the panda gripper

File: robots/hands/panda_gripper/panda_gripper_glb.urdf (robot description, URDF)
Before this commit: robot panda, 4 links, 3 joints
Links:
- link panda_hand: geometry collision box size=0.036 0.08 0.2; collision cylinder length=0.0077 radius=0.03
- link panda_leftfinger: geometry collision box size=17.5e-3 15.2e-3 18.5e-3; collision box size=17.5e-3 7e-3 23.5e-3
- link panda_rightfinger: geometry collision box size=17.5e-3 15.2e-3 18.5e-3; collision box size=17.5e-3 7e-3 23.5e-3

Commit message: [fix] small fix for panda gripper

File: robots/hands/panda_gripper/panda_gripper_glb.urdf (robot description, URDF)
Before this commit: robot panda_gripper, 4 links, 3 joints
Joints:
- joint panda_finger_joint2: mimic joint=panda_finger_joint1 -> joint=panda_finger_joint1 multiplier=1 offset=0
