Commit message: [fix] fix shadow hand mesh reference

File: robots/assembly/ur5e_shadow/ur5e_shadow_right_hand_glb.urdf (robot description, URDF)
Before this commit: robot ur5e_shadow, 41 links, 40 joints
Links:
- link ffdistal: geometry collision mesh filename=../../hands/shadow_hand/meshes/collision/f_distal_pst.obj scale=0.001 0.001 0.001; visual mesh filename=../../hands/shadow_hand/meshes/visual/f_distal_pst.glb scale=0.001 0.001 0.001
- link thdistal: geometry collision mesh filename=../../hands/shadow_hand/meshes/collision/th_distal_pst.obj scale=0.001 0.001 0.001; visual mesh filename=../../hands/shadow_hand/meshes/visual/th_distal_pst.glb scale=0.001 0.001 0.001
Joints:
- joint mount_joint: origin xyz=-0.01 0.0 0.00 rpy=1.57079 0 1.57079 -> xyz=0.0 -0.01 0.0 rpy=-1.5707926 0 0
- joint wrist_3-flange: origin xyz=0 0 0 rpy=0 -1.57079632679 -1.57079632679 -> xyz=0 0 0 rpy=1.5707926 0 0

File: robots/hands/shadow_hand/shadow_hand_left_glb.urdf (robot description, URDF)
Before this commit: robot shadow_left, 33 links, 32 joints
Links:
- link ffmiddle: geometry collision cylinder length=0.025 radius=0.007; collision sphere radius=0.007
- link lfdistal: geometry collision mesh filename=meshes/collision/f_distal_pst.obj scale=0.001 0.001 0.001; visual mesh filename=meshes/visual/f_distal_pst.glb scale=0.001 0.001 0.001

File: robots/hands/shadow_hand/shadow_hand_right_glb.urdf (robot description, URDF)
Before this commit: robot shadow_right, 33 links, 32 joints
Links:
- link ffdistal: geometry collision mesh filename=meshes/collision/f_distal_pst.obj scale=0.001 0.001 0.001; visual mesh filename=meshes/visual/f_distal_pst.glb scale=0.001 0.001 0.001

Commit message: [fix] fix ur5e + shadow ee_link orientation

File: robots/assembly/ur5e_shadow/ur5e_shadow_right_hand_glb.urdf (robot description, URDF)
Before this commit: robot ur5e_shadow_right, 41 links, 40 joints
Joints:
- joint wrist_3-flange: origin xyz=0 0 0 rpy=0 0 1.5707926 -> xyz=0 0 0 rpy=0 0 -1.5707926
