Commit message: [fix] fix ur5e + shadow ee_link orientation

File: robots/assembly/ur5e_shadow/ur5e_shadow_left_hand_glb.urdf (robot description, URDF)
Before this commit: robot ur5e_shadow_left, 41 links, 40 joints
Joints:
- joint mount_joint: origin xyz=0.0 -0.01 0.0 rpy=-1.5707926 0 0 -> xyz=0.0 0.0 -0.01 rpy=0 0 0; parent ee_link -> wrist_3_link
- joint wrist_3-flange: origin xyz=0 0 0 rpy=1.5707926 0 0 -> xyz=0 0 0 rpy=0 0 -1.5707926

File: robots/assembly/ur5e_shadow/ur5e_shadow_right_hand_glb.urdf (robot description, URDF)
Before this commit: robot ur5e_shadow_right, 41 links, 40 joints
Joints:
- joint mount_joint: origin xyz=0.0 -0.01 0.0 rpy=-1.5707926 0 0 -> xyz=0.0 0.0 -0.01 rpy=0 0 0; parent ee_link -> wrist_3_link
- joint wrist_3-flange: origin xyz=0 0 0 rpy=1.5707926 0 0 -> xyz=0 0 0 rpy=0 0 1.5707926

Commit message: Ur shadow (#20)
* [fix] fix shadow hand mesh reference

* [add] add UR5e + left shadow hand model

* [fix] fix ur5e + shadow ee_link orientation

* [fix] fix ur5e + shadow ee_link orientation

File: robots/assembly/ur5e_shadow/ur5e_shadow_left_hand_glb.urdf (robot description, URDF)
Before this commit: robot shadow_right, 33 links, 32 joints
Links:
- removed link world
- added link base
- added link base_link
- added link base_link_inertia, mass 4.0; collision mesh filename=../../arms/ur5e/meshes/collision/base.obj; visual mesh filename=../../arms/ur5e/meshes/visual/base.glb
- added link forearm_link, mass 2.275; collision mesh filename=../../arms/ur5e/meshes/collision/forearm.obj; visual mesh filename=../../arms/ur5e/meshes/visual/forearm.glb
- added link shoulder_link, mass 3.7; collision mesh filename=../../arms/ur5e/meshes/collision/shoulder.obj; visual mesh filename=../../arms/ur5e/meshes/visual/shoulder.glb
- added link upper_arm_link, mass 8.393; collision mesh filename=../../arms/ur5e/meshes/collision/upperarm.obj; visual mesh filename=../../arms/ur5e/meshes/visual/upperarm.glb
- added link wrist_1_link, mass 1.219; collision mesh filename=../../arms/ur5e/meshes/collision/wrist1.obj; visual mesh filename=../../arms/ur5e/meshes/visual/wrist1.glb
- added link wrist_2_link, mass 1.219; collision mesh filename=../../arms/ur5e/meshes/collision/wrist2.obj; visual mesh filename=../../arms/ur5e/meshes/visual/wrist2.glb
- added link wrist_3_link, mass 0.1879; collision mesh filename=../../arms/ur5e/meshes/collision/wrist3.obj; visual mesh filename=../../arms/ur5e/meshes/visual/wrist3.glb
- link ffdistal: geometry collision mesh filename=../../hands/shadow_hand/meshes/collision/f_distal_pst.obj scale=0.001 0.001 0.001; visual mesh filename=../../hands/shadow_hand/meshes/visual/f_distal_pst.glb scale=0.001 0.001 0.001
- link ffknuckle: geometry collision mesh filename=../../hands/shadow_hand/meshes/collision/f_knuckle_E3M5.obj; visual mesh filename=../../hands/shadow_hand/meshes/visual/f_knuckle_E3M5.glb scale=0.001 0.001 0.001
- link ffmiddle: geometry collision cylinder length=0.025 radius=0.007; collision sphere radius=0.007
- link ffproximal: geometry collision cylinder length=0.040 radius=0.007; visual mesh filename=../../hands/shadow_hand/meshes/visual/f_proximal_E3M5.glb scale=0.001 0.001 0.001
- link forearm: geometry collision box size=0.07 0.07 0.07; collision mesh filename=../../hands/shadow_hand/meshes/collision/forearm_E3M5.obj scale=0.001 0.001 0.001
- link lfdistal: geometry collision mesh filename=../../hands/shadow_hand/meshes/collision/f_distal_pst.obj scale=0.001 0.001 0.001; visual mesh filename=../../hands/shadow_hand/meshes/visual/f_distal_pst.glb scale=0.001 0.001 0.001
- link lfknuckle: geometry collision mesh filename=../../hands/shadow_hand/meshes/collision/f_knuckle_E3M5.obj; visual mesh filename=../../hands/shadow_hand/meshes/visual/f_knuckle_E3M5.glb scale=0.001 0.001 0.001
- link lfmetacarpal: geometry collision box size=0.018 0.024 0.040; visual mesh filename=../../hands/shadow_hand/meshes/visual/lf_metacarpal_E3M5_le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 scale=0.001 0.001 0.001
- link lfmiddle: geometry collision cylinder length=0.025 radius=0.007; collision sphere radius=0.007
- link lfproximal: geometry collision cylinder length=0.040 radius=0.007; visual mesh filename=../../hands/shadow_hand/meshes/visual/f_proximal_E3M5.glb scale=0.001 0.001 0.001
- link mfdistal: geometry collision mesh filename=../../hands/shadow_hand/meshes/collision/f_distal_pst.obj scale=0.001 0.001 0.001; visual mesh filename=../../hands/shadow_hand/meshes/visual/f_distal_pst.glb scale=0.001 0.001 0.001
- link mfknuckle: geometry collision mesh filename=../../hands/shadow_hand/meshes/collision/f_knuckle_E3M5.obj; visual mesh filename=../../hands/shadow_hand/meshes/visual/f_knuckle_E3M5.glb scale=0.001 0.001 0.001
- link mfmiddle: geometry collision cylinder length=0.025 radius=0.007; collision sphere radius=0.007
- link mfproximal: geometry collision cylinder length=0.040 radius=0.007; visual mesh filename=../../hands/shadow_hand/meshes/visual/f_proximal_E3M5.glb scale=0.001 0.001 0.001
- link palm: geometry collision box size=0.018 0.024 0.004; collision box size=0.020 0.024 0.032
- link rfdistal: geometry collision mesh filename=../../hands/shadow_hand/meshes/collision/f_distal_pst.obj scale=0.001 0.001 0.001; visual mesh filename=../../hands/shadow_hand/meshes/visual/f_distal_pst.glb scale=0.001 0.001 0.001
- link rfknuckle: geometry collision mesh filename=../../hands/shadow_hand/meshes/collision/f_knuckle_E3M5.obj; visual mesh filename=../../hands/shadow_hand/meshes/visual/f_knuckle_E3M5.glb scale=0.001 0.001 0.001
- link rfmiddle: geometry collision cylinder length=0.025 radius=0.007; collision sphere radius=0.007
- link rfproximal: geometry collision cylinder length=0.040 radius=0.007; visual mesh filename=../../hands/shadow_hand/meshes/visual/f_proximal_E3M5.glb scale=0.001 0.001 0.001
- link thdistal: geometry collision mesh filename=../../hands/shadow_hand/meshes/collision/th_distal_pst.obj scale=0.001 0.001 0.001; visual mesh filename=../../hands/shadow_hand/meshes/visual/th_distal_pst.glb scale=0.001 0.001 0.001
- link thmiddle: geometry collision mesh filename=../../hands/shadow_hand/meshes/collision/th_middle_E3M5.obj scale=0.001 0.001 0.001; visual mesh filename=../../hands/shadow_hand/meshes/visual/th_middle_E3M5.glb scale=0.001 0.001 0.001
- link thproximal: geometry collision mesh filename=../../hands/shadow_hand/meshes/collision/th_proximal_E3M5.o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 scale=0.001 0.001 0.001; visual mesh filename=../../hands/shadow_hand/meshes/visual/th_proximal_E3M5.glb scale=0.001 0.001 0.001
- link wrist: geometry collision box size=0.027 0.018 0.010; collision box size=0.027 0.018 0.010
Joints:
- removed joint ee_fixed_joint
- removed joint world_joint
- added joint base_link-base_fixed_joint: type fixed, parent base_link, child base, origin xyz=0 0 0 rpy=0 0 3.14159265359
- added joint base_link-base_link_inertia: type fixed, parent base_link, child base_link_inertia, origin xyz=0 0 0 rpy=0 0 3.14159265359
- added joint elbow_joint: type revolute, parent upper_arm_link, child forearm_link, origin xyz=-0.425 0 0 rpy=0 0 0, axis 0 0 1, limit lower=-3.14159265359 upper=3.14159265359 effort=150.0 velocity=3.14159265359
- added joint mount_joint: type fixed, parent wrist_3_link, child forearm, origin xyz=0.0 0.0 -0.01 rpy=0 0 0
- added joint shoulder_lift_joint: type revolute, parent shoulder_link, child upper_arm_link, origin xyz=0 0 0 rpy=1.570796327 0 0, axis 0 0 1, limit lower=-6.28318530718 upper=6.28318530718 effort=150.0 velocity=3.14159265359
- added joint shoulder_pan_joint: type revolute, parent base_link_inertia, child shoulder_link, origin xyz=0 0 0.1625 rpy=0 0 0, axis 0 0 1, limit lower=-6.28318530718 upper=6.28318530718 effort=150.0 velocity=3.14159265359
- added joint wrist_1_joint: type revolute, parent forearm_link, child wrist_1_link, origin xyz=-0.3922 0 0.1333 rpy=0 0 0, axis 0 0 1, limit lower=-6.28318530718 upper=6.28318530718 effort=28.0 velocity=3.14159265359
- added joint wrist_2_joint: type revolute, parent wrist_1_link, child wrist_2_link, origin xyz=0 -0.0997 -2.0448811823e-11 rpy=1.570796327 0 0, axis 0 0 1, limit lower=-6.28318530718 upper=6.28318530718 effort=28.0 velocity=3.14159265359
- added joint wrist_3-flange: type fixed, parent wrist_3_link, child ee_link, origin xyz=0 0 0 rpy=0 0 -1.5707926
- added joint wrist_3_joint: type revolute, parent wrist_2_link, child wrist_3_link, origin xyz=0 0.0996 -2.04283014801e-11 rpy=1.57079632659 3.14159265359 3.14159265359, axis 0 0 1, limit lower=-6.28318530718 upper=6.28318530718 effort=28.0 velocity=3.14159265359
- joint FFJ4: axis 0 -1 0 -> 0 1 0; origin xyz=0.033 0 0.095 rpy=0 0 0 -> xyz=-0.033 0 0.095 rpy=0 0 0
- joint LFJ4: axis 0 1 0 -> 0 -1 0; origin xyz=0.05397275 0 0.03779463 rpy=0 0.9599 0 -> xyz=-0.05397275 0 0.03779463 rpy=0 -0.9599 0
- joint LFJ5: origin xyz=-0.033 0 0.02071 rpy=0 -0.9599 0 -> xyz=0.033 0 0.02071 rpy=0 0.9599 0
- joint MFJ4: axis 0 -1 0 -> 0 1 0; origin xyz=0.011 0 0.099 rpy=0 0 0 -> xyz=-0.011 0 0.099 rpy=0 0 0
- joint RFJ4: axis 0 1 0 -> 0 -1 0; origin xyz=-0.011 0 0.095 rpy=0 0 0 -> xyz=0.011 0 0.095 rpy=0 0 0
- joint THJ3: axis 0 1 0 -> 0 -1 0
- joint THJ4: axis 0 1 0 -> 0 -1 0
- joint THJ5: axis 0 0 -1 -> 0 0 1; origin xyz=0.034 -0.00858 0.029 rpy=-0.785398163397 0 -1.57079632679 -> xyz=-0.034 -0.00858 0.029 rpy=-0.785398163397 0 1.57079632679
- joint WRJ2: axis 0 1 0 -> 0 -1 0

File: robots/assembly/ur5e_shadow/ur5e_shadow_right_hand_glb.urdf (robot description, URDF)
Before this commit: robot ur5e_shadow, 41 links, 40 joints
Links:
- link ffdistal: geometry collision mesh filename=../../hands/shadow_hand/meshes/collision/f_distal_pst.obj scale=0.001 0.001 0.001; visual mesh filename=../../hands/shadow_hand/meshes/visual/f_distal_pst.glb scale=0.001 0.001 0.001
- link thdistal: geometry collision mesh filename=../../hands/shadow_hand/meshes/collision/th_distal_pst.obj scale=0.001 0.001 0.001; visual mesh filename=../../hands/shadow_hand/meshes/visual/th_distal_pst.glb scale=0.001 0.001 0.001
Joints:
- joint mount_joint: origin xyz=-0.01 0.0 0.00 rpy=1.57079 0 1.57079 -> xyz=0.0 0.0 -0.01 rpy=0 0 0; parent ee_link -> wrist_3_link
- joint wrist_3-flange: origin xyz=0 0 0 rpy=0 -1.57079632679 -1.57079632679 -> xyz=0 0 0 rpy=0 0 -1.5707926
