Commit message: [fix] fix allegro duplicated inertia tag

File: robots/hands/allegro_hand/allegro_hand_left.urdf (robot description, URDF)
Before this commit: robot allegro_left, 23 links, 22 joints
Links:
- link link_3.0: mass 0.0096 -> 0.02

File: robots/hands/allegro_hand/allegro_hand_left_glb.urdf (robot description, URDF)
Before this commit: robot allegro_left, 23 links, 22 joints
Links:
- link link_3.0: mass 0.0096 -> 0.02

File: robots/hands/allegro_hand/allegro_hand_right.urdf (robot description, URDF)
Before this commit: robot allegro_right, 23 links, 22 joints
Links:
- link link_3.0: mass 0.0096 -> 0.02

File: robots/hands/allegro_hand/allegro_hand_right_glb.urdf (robot description, URDF)
Before this commit: robot allegro_right, 23 links, 22 joints
Links:
- link link_3.0: mass 0.0096 -> 0.02

File: robots/hands/allegro_hand/variation/allegro_hand_right_fsr.urdf (robot description, URDF)
Before this commit: robot allegro_right, 39 links, 38 joints
Links:
- link link_3.0: mass 0.0096 -> 0.02

File: robots/hands/allegro_hand/variation/allegro_hand_right_fsr_glb.urdf (robot description, URDF)
Before this commit: robot allegro_right, 39 links, 38 joints
Links:
- link link_3.0: mass 0.0096 -> 0.02

File: robots/hands/allegro_hand/variation/allegro_hand_right_fsr_simple.urdf (robot description, URDF)
Before this commit: robot allegro_right, 39 links, 38 joints
Links:
- link link_3.0: mass 0.0096 -> 0.02

Commit message: [fix] fix allegro hand finger tip pos

File: robots/hands/allegro_hand/allegro_hand_left.urdf (robot description, URDF)
Before this commit: robot allegro_left, 23 links, 22 joints
Joints:
- joint joint_11.0_tip: origin xyz=0 0 0.0267 rpy=0 0 0 -> xyz=0 0 0.0387 rpy=0 0 0
- joint joint_15.0_tip: origin xyz=0 0 0.0423 rpy=0 0 0 -> xyz=0 0 0.0543 rpy=0 0 0
- joint joint_3.0_tip: origin xyz=0 0 0.0267 rpy=0 0 0 -> xyz=0 0 0.0387 rpy=0 0 0
- joint joint_7.0_tip: origin xyz=0 0 0.0267 rpy=0 0 0 -> xyz=0 0 0.0387 rpy=0 0 0

File: robots/hands/allegro_hand/allegro_hand_left_glb.urdf (robot description, URDF)
Before this commit: robot allegro_left, 23 links, 22 joints
Joints:
- joint joint_11.0_tip: origin xyz=0 0 0.0267 rpy=0 0 0 -> xyz=0 0 0.0387 rpy=0 0 0
- joint joint_15.0_tip: origin xyz=0 0 0.0423 rpy=0 0 0 -> xyz=0 0 0.0543 rpy=0 0 0
- joint joint_3.0_tip: origin xyz=0 0 0.0267 rpy=0 0 0 -> xyz=0 0 0.0387 rpy=0 0 0
- joint joint_7.0_tip: origin xyz=0 0 0.0267 rpy=0 0 0 -> xyz=0 0 0.0387 rpy=0 0 0

File: robots/hands/allegro_hand/allegro_hand_right.urdf (robot description, URDF)
Before this commit: robot allegro_right, 23 links, 22 joints
Joints:
- joint joint_11.0_tip: origin xyz=0 0 0.0267 rpy=0 0 0 -> xyz=0 0 0.0387 rpy=0 0 0
- joint joint_15.0_tip: origin xyz=0 0 0.0423 rpy=0 0 0 -> xyz=0 0 0.0543 rpy=0 0 0
- joint joint_3.0_tip: origin xyz=0 0 0.0267 rpy=0 0 0 -> xyz=0 0 0.0387 rpy=0 0 0
- joint joint_7.0_tip: origin xyz=0 0 0.0267 rpy=0 0 0 -> xyz=0 0 0.0387 rpy=0 0 0

File: robots/hands/allegro_hand/allegro_hand_right_glb.urdf (robot description, URDF)
Before this commit: robot allegro_right, 23 links, 22 joints
Joints:
- joint joint_11.0_tip: origin xyz=0 0 0.0267 rpy=0 0 0 -> xyz=0 0 0.0387 rpy=0 0 0
- joint joint_15.0_tip: origin xyz=0 0 0.0423 rpy=0 0 0 -> xyz=0 0 0.0543 rpy=0 0 0
- joint joint_3.0_tip: origin xyz=0 0 0.0267 rpy=0 0 0 -> xyz=0 0 0.0387 rpy=0 0 0
- joint joint_7.0_tip: origin xyz=0 0 0.0267 rpy=0 0 0 -> xyz=0 0 0.0387 rpy=0 0 0
